Commit message: Completed Ramp and Door obstacle

File: march_simulation/obstacles/ramp_and_door.xacro (robot description, xacro)
@@ -22,10 +22,10 @@
         <collision>
           <geometry>
-            <box size="${platform_length} ${platform_width} ${platform_height}" />
+            <box size="${platform_length} ${platform_width} 3" />
           </geometry>
         </collision>
         <visual name='visual'>
           <geometry>
-            <box size="${platform_length} ${platform_width} ${platform_height}" />
+            <box size="${platform_length} ${platform_width} 3" />
           </geometry>
         </visual>
@@ -86,18 +86,18 @@
     </gazebo>
     <!-- Joints -->
-    <joint name="hip" type="fixed">
+    <joint name="hip_1" type="fixed">
         <parent link="${parent_name}"/>
         <child link="platform"/>
-        <origin xyz="${-distance_to_origin} 0 0" rpy="0 0 0"/>
+        <origin xyz="-3.2 0 -1.02" rpy="0 0 0"/>
     </joint>
     <joint name="joint_1" type="fixed">
         <parent link="platform"/>
         <child link="ramp_up"/>
-        <origin xyz="0.9 0 0" rpy="0 0.35 0"/>
+        <origin xyz="1.875 0 0.601" rpy="0 0.35 0"/>
     </joint>
     <joint name="joint_2" type="fixed">
         <parent link="platform"/>
         <child link="ramp_down"/>
-        <origin xyz="-0.9 0 0" rpy="0 -0.26 0"/>
+        <origin xyz="-2.115 0 0.365" rpy="0 -0.26 0"/>
     </joint>
 </robot>

Commit message: Fixed the platform height

File: march_simulation/obstacles/ramp_and_door.xacro (robot description, xacro)
@@ -22,10 +22,10 @@
         <collision>
           <geometry>
-            <box size="${platform_length} ${platform_width} 3" />
+            <box size="${platform_length} ${platform_width} ${platform_height}" />
           </geometry>
         </collision>
         <visual name='visual'>
           <geometry>
-            <box size="${platform_length} ${platform_width} 3" />
+            <box size="${platform_length} ${platform_width} ${platform_height}" />
           </geometry>
         </visual>
@@ -89,15 +89,15 @@
         <parent link="${parent_name}"/>
         <child link="platform"/>
-        <origin xyz="-3.2 0 -1.02" rpy="0 0 0"/>
+        <origin xyz="-3.2 0 ${platform_height / 2}" rpy="0 0 0"/>
     </joint>
     <joint name="joint_1" type="fixed">
         <parent link="platform"/>
         <child link="ramp_up"/>
-        <origin xyz="1.875 0 0.601" rpy="0 0.35 0"/>
+        <origin xyz="1.875 0 -0.659" rpy="0 0.35 0"/>
     </joint>
     <joint name="joint_2" type="fixed">
         <parent link="platform"/>
         <child link="ramp_down"/>
-        <origin xyz="-2.115 0 0.365" rpy="0 -0.26 0"/>
+        <origin xyz="-2.115 0 -0.895" rpy="0 -0.26 0"/>
     </joint>
 </robot>

Commit message: Fix some names

File: march_simulation/obstacles/ramp_and_door.xacro (robot description, xacro)
@@ -86,5 +86,5 @@
     </gazebo>
     <!-- Joints -->
-    <joint name="hip_1" type="fixed">
+    <joint name="joint_0" type="fixed">
         <parent link="${parent_name}"/>
         <child link="platform"/>

File: march_simulation/obstacles/stairs.xacro (robot description, xacro)
@@ -142,5 +142,5 @@
     </gazebo>
     <!-- Joints -->
-    <joint name="hip" type="fixed">
+    <joint name="joint_0" type="fixed">
         <parent link="${parent_name}"/>
         <child link="step_1"/>

File: march_simulation/obstacles/tilted_path.xacro (robot description, xacro)
@@ -89,15 +89,15 @@
     </gazebo>
     <!-- Joints -->
-    <joint name="joint_1" type="fixed">
+    <joint name="joint_0" type="fixed">
         <parent link="${parent_name}"/>
         <child link="middle_block"/>
         <origin xyz="${-distance_to_origin-2.5} 0 -0.15" rpy="${- middle_block_angle} 0 0"/>
     </joint>
-    <joint name="joint_2" type="fixed">
+    <joint name="joint_1" type="fixed">
         <parent link="middle_block"/>
         <child link="side_block_1"/>
         <origin xyz="2.17 0.01 -0.135" rpy="0 ${side_blocks_angle} 0"/>
     </joint>
-    <joint name="joint_3" type="fixed">
+    <joint name="joint_2" type="fixed">
         <parent link="middle_block"/>
         <child link="side_block_2"/>
