Commit message: Some small improvements to make the pressure sole thinner

File: ros1/src/shared/march_description/urdf/march4.xacro (robot description, xacro)
@@ -324,8 +324,38 @@
             <always_on>true</always_on>
         </sensor>
-        <sensor name="left_pressure_sole" type="contact">
+    </gazebo>
+    <!-- Foot Left -->
+    <link name="foot_left">
+        <inertial>
+            <origin xyz="${foot_com_x} ${-foot_com_y} ${foot_com_z}" rpy="0 0 0"/>
+            <mass value="${foot_mass}"/>
+            <inertia
+                    ixx="${foot_Ixx}"
+                    ixy="${-foot_Ixy}"
+                    ixz="${foot_Ixz}"
+                    iyy="${foot_Iyy}"
+                    iyz="${-foot_Iyz}"
+                    izz="${foot_Izz}" />
+        </inertial>
+        <collision>
+            <origin xyz="${(-foot_height_forward+foot_height_backward)/2} 0 0" rpy="0 0 0"/>
+            <geometry>
+                <box size="${foot_height_forward+foot_height_backward} ${width} ${width}"/>
+            </geometry>
+        </collision>
+    </link>
+    <link name="pressure_sole_left">
+        <collision>
+            <origin xyz="${(-foot_height_forward+foot_height_backward)/2} 0 0" rpy="0 0 0"/>
+            <geometry>
+                <box size="${foot_height_forward+foot_height_backward} ${width} 0.001"/>
+            </geometry>
+        </collision>
+    </link>
+    <gazebo reference="pressure_sole_left">
+        <sensor name="left_pressure_sole_2" type="contact">
             <always_on>true</always_on>
             <contact>
-                <collision>ankle_plate_left_fixed_joint_lump__foot_left_collision_1</collision>
+                <collision>ankle_plate_left_fixed_joint_lump__pressure_sole_left_collision_2</collision>
             </contact>
             <plugin name="left_foot_plugin" filename="libgazebo_ros_bumper.so">
@@ -335,24 +365,4 @@
         </sensor>
     </gazebo>
-    <!-- Foot Left -->
-    <link name="foot_left">
-        <inertial>
-            <origin xyz="${foot_com_x} ${-foot_com_y} ${foot_com_z}" rpy="0 0 0"/>
-            <mass value="${foot_mass}"/>
-            <inertia
-                    ixx="${foot_Ixx}"
-                    ixy="${-foot_Ixy}"
-                    ixz="${foot_Ixz}"
-                    iyy="${foot_Iyy}"
-                    iyz="${-foot_Iyz}"
-                    izz="${foot_Izz}" />
-        </inertial>
-        <collision>
-            <origin xyz="${(-foot_height_forward+foot_height_backward)/2} 0 0" rpy="0 0 0"/>
-            <geometry>
-                <box size="${foot_height_forward+foot_height_backward} ${width} ${width}"/>
-            </geometry>
-        </collision>
-    </link>
     <gazebo reference="foot_left">
         <mu1>${foot_mu1}</mu1>
@@ -483,14 +493,4 @@
             <always_on>true</always_on>
         </sensor>
-        <sensor name="right_pressure_sole" type="contact">
-            <always_on>true</always_on>
-            <contact>
-                <collision>ankle_plate_right_fixed_joint_lump__foot_right_collision_1</collision>
-            </contact>
-            <plugin name="right_foot_pressure_plugin" filename="libgazebo_ros_bumper.so">
-                <bumperTopicName>march/sensor/right_pressure_sole</bumperTopicName>
-                <frameName>world</frameName>
-            </plugin>
-        </sensor>
     </gazebo>
     <!-- Foot Right -->
@@ -519,4 +519,24 @@
         <minDepth>${foot_min_depth}</minDepth>
         <fdir1>1 0 0</fdir1>
+    </gazebo>
+    <link name="pressure_sole_right">
+        <collision>
+            <origin xyz="${(-foot_height_forward+foot_height_backward)/2} 0 0" rpy="0 0 0"/>
+            <geometry>
+                <box size="${foot_height_forward+foot_height_backward} ${width} 0.001"/>
+            </geometry>
+        </collision>
+    </link>
+    <gazebo reference="pressure_sole_right">
+        <sensor name="right_pressure_sole" type="contact">
+            <always_on>true</always_on>
+            <contact>
+                <collision>ankle_plate_right_fixed_joint_lump__pressure_sole_right_collision_2</collision>
+            </contact>
+            <plugin name="right_foot_plugin" filename="libgazebo_ros_bumper.so">
+                <bumperTopicName>march/sensor/right_pressure_sole</bumperTopicName>
+                <frameName>world</frameName>
+            </plugin>
+        </sensor>
     </gazebo>
     <!-- Joints -->
@@ -595,4 +615,14 @@
         <child link="foot_left"/>
         <origin xyz="0 0 ${-ankle_plate_height}" rpy="0 0 0"/>
+    </joint>
+    <joint name="left_pressure_sole_joint" type="fixed">
+        <parent link="foot_left"/>
+        <child link="pressure_sole_left"/>
+        <origin xyz="0 0 ${-(width/2)}" rpy="0 0 0"/>
+    </joint>
+    <joint name="right_pressure_sole_joint" type="fixed">
+        <parent link="foot_right"/>
+        <child link="pressure_sole_right"/>
+        <origin xyz="0 0 ${-(width/2)}" rpy="0 0 0"/>
     </joint>
     <joint name="right_hip_aa" type="revolute">
