Commit message: fix ankle hight koen

File: ros1/src/march_description/urdf/march4_with_koen_lengths.xacro (robot description, xacro)
@@ -60,5 +60,5 @@
     <xacro:property name="lower_leg_mass" value="4.458"/>
     <!-- mass = Ankle actuator + Lower leg -->
-    <xacro:property name="ankle_plate_height" value="0.095"/>
+    <xacro:property name="ankle_plate_height" value="0.12"/>
     <xacro:property name="ankle_plate_offset" value="0.07"/>
     <xacro:property name="foot_height_forward" value="${0.194}"/>

Commit message: update hip base length

File: ros1/src/march_description/urdf/march4_with_koen_lengths.xacro (robot description, xacro)
@@ -46,5 +46,5 @@
     <!-- Masses determined in Catia, see https://confluence.projectmarch.nl:8443/display/51/URDF+description -->
     <xacro:property name="width" value="0.05"/> <!-- Square dimensions (widthxwidth) of beams -->
-    <xacro:property name="hip_base_height" value="0.210"/>
+    <xacro:property name="hip_base_height" value="0.20"/>
     <xacro:property name="hip_base_mass" value="8.686"/>
     <!-- mass = Hip base + HAA actuators -->
