Commit message: Add not working contact sensor to gazebo

File: ros1/src/march_description/urdf/march4.xacro (robot description, xacro)
@@ -335,4 +335,63 @@
         </collision>
     </link>
+    <link name="foot_left_bumper">
+        <inertial>
+            <mass value="0.01"/>
+            <origin xyz="0 0 0" rpy="0 0 0"/>
+            <inertia ixx="1" ixy="0" ixz="0" iyy="1" iyz="0" izz="1" />
+        </inertial>
+        <visual>
+            <origin xyz="0 0 0" rpy="0 0 0" />
+            <geometry>
+                <box size="0.01 0.01 0.01"/>
+            </geometry>
+        </visual>
+        <collision name="foot_left_bumper_collision">
+            <origin rpy="0 0 0" xyz="0.0 0.0 0.0"/>
+            <geometry name="foot_left_bumper_collision">
+                <box size="0.01 0.01 0.01"/>
+            </geometry>
+            <contact_coefficients kd="1.0" kp="1000.0" mu="0"/>
+        </collision>
+    </link>
+    <gazebo reference="foot_left_bumper">
+        <sensor name="left_foot_sensor" type="contact">
+            <always_on>true</always_on>
+            <update_rate>30.0</update_rate>
+            <contact>
+                <collison>ankle_plate_right_fixed_joint_lump__foot_right_collision_1</collison>
+            </contact>
+        </sensor>
+        <plugin name="foot_left_bumper_plugin" filename="libgazebo_ros_bumper.so">
+            <bumperTopicName>left_foot_bumper</bumperTopicName>
+            <frameName>ankle_plate</frameName>
+        </plugin>
+    </gazebo>
+<!--    <joint name="bumper_joint" type="fixed">-->
+<!--        <axis xyz="0 1 0" />-->
+<!--        <origin xyz=".2 0 0" rpy="0 0 0"/>-->
+<!--        <parent link="foot_left"/>-->
+<!--        <child link="bump_sensor"/>-->
+<!--    </joint>-->
+<!--    <link name="bump_sensor">-->
+<!--        <collision>-->
+<!--            ankle_plate_left_collision-->
+<!--            <origin xyz="0 0 0" rpy="0 0 0"/>&ndash;&gt;-->
+<!--            <geometry>-->
+<!--                <box size="0.1 0.1 0.1"/>-->
+<!--            </geometry>-->
+<!--        </collision>-->
+<!--        <visual>-->
+<!--          <origin xyz="0 0 0" rpy="0 0 0"/>-->
+<!--          <geometry>-->
+<!--             <box size="0.1 0.1 0.1"/>-->
+<!--          </geometry>-->
+<!--        </visual>-->
+<!--        <inertial>-->
+<!--          <mass value="1e-5" />-->
+<!--          <origin xyz="0 0 0" rpy="0 0 0"/>-->
+<!--          <inertia ixx="1e-6" ixy="0" ixz="0" iyy="1e-6" iyz="0" izz="1e-6" />-->
+<!--        </inertial>-->
+<!--    </link>-->
     <gazebo reference="foot_left">
         <mu1>${foot_mu1}</mu1>

Commit message: Fix working left foot sensor

File: ros1/src/march_description/urdf/march4.xacro (robot description, xacro)
@@ -315,4 +315,14 @@
         </collision>
     </link>
+    <gazebo reference="ankle_plate_left">
+        <sensor name="ankle_plate_left_contact" type="contact">
+            <plugin name="contact_plugin" filename="libcontact.so"/>
+            <contact>
+                <collision>ankle_plate_left_fixed_joint_lump__foot_left_collision_1</collision>
+            </contact>
+            <update_rate>30</update_rate>
+            <always_on>true</always_on>
+        </sensor>
+    </gazebo>
     <!-- Foot Left -->
     <link name="foot_left">
@@ -335,63 +345,4 @@
         </collision>
     </link>
-    <link name="foot_left_bumper">
-        <inertial>
-            <mass value="0.01"/>
-            <origin xyz="0 0 0" rpy="0 0 0"/>
-            <inertia ixx="1" ixy="0" ixz="0" iyy="1" iyz="0" izz="1" />
-        </inertial>
-        <visual>
-            <origin xyz="0 0 0" rpy="0 0 0" />
-            <geometry>
-                <box size="0.01 0.01 0.01"/>
-            </geometry>
-        </visual>
-        <collision name="foot_left_bumper_collision">
-            <origin rpy="0 0 0" xyz="0.0 0.0 0.0"/>
-            <geometry name="foot_left_bumper_collision">
-                <box size="0.01 0.01 0.01"/>
-            </geometry>
-            <contact_coefficients kd="1.0" kp="1000.0" mu="0"/>
-        </collision>
-    </link>
-    <gazebo reference="foot_left_bumper">
-        <sensor name="left_foot_sensor" type="contact">
-            <always_on>true</always_on>
-            <update_rate>30.0</update_rate>
-            <contact>
-                <collison>ankle_plate_right_fixed_joint_lump__foot_right_collision_1</collison>
-            </contact>
-        </sensor>
-        <plugin name="foot_left_bumper_plugin" filename="libgazebo_ros_bumper.so">
-            <bumperTopicName>left_foot_bumper</bumperTopicName>
-            <frameName>ankle_plate</frameName>
-        </plugin>
-    </gazebo>
-<!--    <joint name="bumper_joint" type="fixed">-->
-<!--        <axis xyz="0 1 0" />-->
-<!--        <origin xyz=".2 0 0" rpy="0 0 0"/>-->
-<!--        <parent link="foot_left"/>-->
-<!--        <child link="bump_sensor"/>-->
-<!--    </joint>-->
-<!--    <link name="bump_sensor">-->
-<!--        <collision>-->
-<!--            ankle_plate_left_collision-->
-<!--            <origin xyz="0 0 0" rpy="0 0 0"/>&ndash;&gt;-->
-<!--            <geometry>-->
-<!--                <box size="0.1 0.1 0.1"/>-->
-<!--            </geometry>-->
-<!--        </collision>-->
-<!--        <visual>-->
-<!--          <origin xyz="0 0 0" rpy="0 0 0"/>-->
-<!--          <geometry>-->
-<!--             <box size="0.1 0.1 0.1"/>-->
-<!--          </geometry>-->
-<!--        </visual>-->
-<!--        <inertial>-->
-<!--          <mass value="1e-5" />-->
-<!--          <origin xyz="0 0 0" rpy="0 0 0"/>-->
-<!--          <inertia ixx="1e-6" ixy="0" ixz="0" iyy="1e-6" iyz="0" izz="1e-6" />-->
-<!--        </inertial>-->
-<!--    </link>-->
     <gazebo reference="foot_left">
         <mu1>${foot_mu1}</mu1>

Commit message: Add right foot sensor

File: ros1/src/march_description/urdf/march4.xacro (robot description, xacro)
@@ -464,4 +464,14 @@
         </collision>
     </link>
+    <gazebo reference="ankle_plate_right">
+        <sensor name="ankle_plate_right_contact" type="contact">
+            <plugin name="contact_plugin" filename="libcontact.so"/>
+            <contact>
+                <collision>ankle_plate_right_fixed_joint_lump__foot_right_collision_1</collision>
+            </contact>
+            <update_rate>30</update_rate>
+            <always_on>true</always_on>
+        </sensor>
+    </gazebo>
     <!-- Foot Right -->
     <link name="foot_right">

Commit message: Fix collision name

File: ros1/src/march_description/urdf/march4.xacro (robot description, xacro)
@@ -486,5 +486,5 @@
             <always_on>true</always_on>
             <contact>
-                <collision>ankle_plate_left_fixed_joint_lump__foot_left_collision_1</collision>
+                <collision>ankle_plate_right_fixed_joint_lump__foot_right_collision_1</collision>
             </contact>
             <plugin name="right_foot_pressure_plugin" filename="libgazebo_ros_bumper.so">

Commit message: Fix left/right issue

File: ros1/src/march_description/urdf/march4.xacro (robot description, xacro)
@@ -319,5 +319,5 @@
             <plugin name="contact_plugin" filename="libcontact.so"/>
             <contact>
-                <collision>ankle_plate_left_fixed_joint_lump__foot_right_collision_1</collision>
+                <collision>ankle_plate_left_fixed_joint_lump__foot_left_collision_1</collision>
             </contact>
             <update_rate>30</update_rate>

Commit message: Add basic working version of realsense camera

File: ros1/src/march_description/urdf/march4.xacro (robot description, xacro)
@@ -642,4 +642,11 @@
         <origin xyz="0 0 ${-ankle_plate_height}" rpy="0 0 0"/>
     </joint>
+<!--    <gazebo>-->
+<!--        <plugin name="realsense_plugin" filename="librealsense_gazebo_plugin.so"/>-->
+<!--    </gazebo>-->
+    <xacro:include filename="$(find realsense2_description)/urdf/_d435.urdf.xacro" />
+    <xacro:sensor_d435 parent="upper_leg_left">
+        <origin xyz="0 0 0" rpy="0 0 3.1416"/>
+    </xacro:sensor_d435>
     <!-- ROS Control plugin for Gazebo -->
     <transmission name="left_hip_aa">
