Commit message: Add progress from melodic version

File: ros2/src/shared/march_description/urdf/march4_old.xacro (robot description, xacro)
@@ -7,11 +7,4 @@
     the hover_height to 0.0. Set ground_gait to true to ground gait in simulation.-->
     <xacro:arg name="ground_gait" default="false"/>
-<!--    Switch between using the physical camera and the simulation camera -->
-<!--    If set to 'true', no physical camera is needed -->
-<!--    If this value is set to 'false', the plugin will not be started and the topics -->
-<!--    published by the real camera will be used. -->
-<!--    In both these situations the camera will still be visible and placed in the urdf,-->
-<!--    to be used for the transformations.-->
-    <xacro:arg name="realsense_simulation" default="false"/>
     <xacro:unless value="$(arg ground_gait)">
         <xacro:property name="parent_name" value="world"/>
@@ -25,35 +18,4 @@
         </gazebo>
     </xacro:if>
-<!-- Include all macro files    -->
-    <xacro:include filename="macros/pressure_sole.xacro"/>
-    <xacro:include filename="macros/frame_part.xacro"/>
-    <xacro:include filename="macros/rotational_joint.xacro"/>
-<!-- Add yaml file with inertia properties -->
-    <xacro:property name="yaml_file" value="properties/inertia_march4.yaml"/>
-    <xacro:property name="all_inertias" value="${load_yaml(yaml_file)}"/>
-    <xacro:property name="hip_aa_Ixx" value="0.013"/>
-    <xacro:property name="hip_aa_Ixy" value="0.008"/>
-    <xacro:property name="hip_aa_Ixz" value="0.005"/>
-    <xacro:property name="hip_aa_Iyy" value="0.023"/>
-    <xacro:property name="hip_aa_Iyz" value="-0.001"/>
-    <xacro:property name="hip_aa_Izz" value="0.028"/>
-    <xacro:property name="upper_leg_Ixx" value="0.127"/>
-    <xacro:property name="upper_leg_Ixy" value="0.0001291"/>
-    <xacro:property name="upper_leg_Ixz" value="-0.0002056"/>
-    <xacro:property name="upper_leg_Iyy" value="0.122"/>
-    <xacro:property name="upper_leg_Iyz" value="0.016"/>
-    <xacro:property name="upper_leg_Izz" value="0.015"/>
-    <xacro:property name="lower_leg_Ixx" value="0.075"/>
-    <xacro:property name="lower_leg_Ixy" value="-0.027"/>
-    <xacro:property name="lower_leg_Ixz" value="-0.008"/>
-    <xacro:property name="lower_leg_Iyy" value="0.11"/>
-    <xacro:property name="lower_leg_Iyz" value="-0.002"/>
-    <xacro:property name="lower_leg_Izz" value="0.071" />
-    <xacro:property name="foot_Ixx" value="0.021"/>
-    <xacro:property name="foot_Ixy" value="-0.002"/>
-    <xacro:property name="foot_Ixz" value="0.02"/>
-    <xacro:property name="foot_Iyy" value="0.027"/>
-    <xacro:property name="foot_Iyz" value="0.004"/>
-    <xacro:property name="foot_Izz" value="0.01" />
     <!-- The max effort of the rotary joints is lower then the value corresponding to 25A, because short-circuit errors
     have occured while applying the theoretical max effort for a long time. -->
@@ -116,23 +78,15 @@
     <xacro:property name="hip_base_com_y" value="0.016341"/>
     <xacro:property name="hip_base_com_z" value="0.147761"/>
-    <xacro:property name="hip_base_com" value="${hip_base_com_x} ${hip_base_com_y} ${hip_base_com_z}"/>
     <xacro:property name="hip_aa_com_x" value="${-hip_aa_frame_width + 0.108094}"/>
     <xacro:property name="hip_aa_com_y" value="${-hip_base_height/2 - hip_aa_frame_height + 0.197758}"/>
     <xacro:property name="hip_aa_com_z" value="0.029507"/>
-<!-- CHECKED BASED ON LEFT HIP AA< VERIFY RIGHT IS SAME!!    -->
-    <xacro:property name="left_hip_aa_com" value="${hip_aa_com_x} ${-hip_aa_com_y} ${hip_aa_com_z}"/>
-    <xacro:property name="right_hip_aa_com" value="${hip_aa_com_x} ${hip_aa_com_y} ${hip_aa_com_z}"/>
     <xacro:property name="upper_leg_com_x" value="0.000709"/>
     <xacro:property name="upper_leg_com_y" value="${-hip_base_height/2 - hip_aa_frame_height +
                                                     upper_leg_offset + 0.215254}"/>
     <xacro:property name="upper_leg_com_z" value="-0.19205"/>
-    <xacro:property name="left_upper_leg_com" value="${upper_leg_com_x} ${-upper_leg_com_y} ${upper_leg_com_z}"/>
-    <xacro:property name="right_upper_leg_com" value="${upper_leg_com_x} ${upper_leg_com_y} ${upper_leg_com_z}"/>
     <xacro:property name="lower_leg_com_x" value="-0.00321"/>
     <xacro:property name="lower_leg_com_y" value="${-hip_base_height/2 - hip_aa_frame_height +
                                                     upper_leg_offset + 0.184081}"/>
     <xacro:property name="lower_leg_com_z" value="${upper_leg_height - 0.527082}"/>
-    <xacro:property name="left_lower_leg_com" value="${lower_leg_com_x} ${-lower_leg_com_y} ${lower_leg_com_z}"/>
-    <xacro:property name="right_lower_leg_com" value="${lower_leg_com_x} ${lower_leg_com_y} ${lower_leg_com_z}"/>
     <xacro:property name="foot_com_x" value="-0.028926"/>
     <xacro:property name="foot_com_y" value="${-hip_base_height/2 - hip_aa_frame_height +
@@ -146,4 +100,34 @@
          axis is the negative URDF x axis, see confluence for the impact. The given inertia's are for the right leg,
          Ixy and Iyz will be inverted for the left leg. -->
+    <xacro:property name="hip_base_Ixx" value="0.141"/>
+    <xacro:property name="hip_base_Ixy" value="0.0000336"/>
+    <xacro:property name="hip_base_Ixz" value="-0.007"/>
+    <xacro:property name="hip_base_Iyy" value="0.087"/>
+    <xacro:property name="hip_base_Iyz" value="0.0005089"/>
+    <xacro:property name="hip_base_Izz" value="0.091"/>
+    <xacro:property name="hip_aa_Ixx" value="0.013"/>
+    <xacro:property name="hip_aa_Ixy" value="0.008"/>
+    <xacro:property name="hip_aa_Ixz" value="0.005"/>
+    <xacro:property name="hip_aa_Iyy" value="0.023"/>
+    <xacro:property name="hip_aa_Iyz" value="-0.001"/>
+    <xacro:property name="hip_aa_Izz" value="0.028"/>
+    <xacro:property name="upper_leg_Ixx" value="0.127"/>
+    <xacro:property name="upper_leg_Ixy" value="0.0001291"/>
+    <xacro:property name="upper_leg_Ixz" value="-0.0002056"/>
+    <xacro:property name="upper_leg_Iyy" value="0.122"/>
+    <xacro:property name="upper_leg_Iyz" value="0.016"/>
+    <xacro:property name="upper_leg_Izz" value="0.015"/>
+    <xacro:property name="lower_leg_Ixx" value="0.075"/>
+    <xacro:property name="lower_leg_Ixy" value="-0.027"/>
+    <xacro:property name="lower_leg_Ixz" value="-0.008"/>
+    <xacro:property name="lower_leg_Iyy" value="0.11"/>
+    <xacro:property name="lower_leg_Iyz" value="-0.002"/>
+    <xacro:property name="lower_leg_Izz" value="0.071" />
+    <xacro:property name="foot_Ixx" value="0.021"/>
+    <xacro:property name="foot_Ixy" value="-0.002"/>
+    <xacro:property name="foot_Ixz" value="0.02"/>
+    <xacro:property name="foot_Iyy" value="0.027"/>
+    <xacro:property name="foot_Iyz" value="0.004"/>
+    <xacro:property name="foot_Izz" value="0.01" />
     <!-- Joint properties -->
     <!-- For limit calculations, see https://confluence.projectmarch.nl:8443/pages/viewpage.action?pageId=268697604 -->
@@ -189,83 +173,176 @@
     <!-- Parts -->
     <!-- Hip-->
-    <xacro:frame_part name="hip_base"
-                      side="right"
-                      length="${hip_base_height}"
-                      width="${width}"
-                      direction="y"
-                      visual_origin="${-hip_aa_frame_width} 0 0"
-                      collision_origin="0 0 0"
-                      mesh="HipBase.stl"
-                      com="${hip_base_com}"
-                      mass="${hip_base_mass}"
-                      inertia="${all_inertias['hip_base']}"
-    />
+    <link name="hip_base">
+        <visual>
+            <origin xyz="${-hip_aa_frame_width} 0 0" rpy="0 0 ${pi}"/>
+            <geometry>
+                <mesh filename="package://march_description/urdf/stl-files/HipBase.stl" scale="1 1 1"/>
+            </geometry>
+            <material name="blue"/>
+        </visual>
+        <inertial>
+            <origin xyz="${hip_base_com_x} ${hip_base_com_y} ${hip_base_com_z}" rpy="0 0 0"/>
+            <mass value="${hip_base_mass}"/>
+            <inertia
+                    ixx="${hip_base_Ixx}"
+                    ixy="${hip_base_Ixy}"
+                    ixz="${hip_base_Ixz}"
+                    iyy="${hip_base_Iyy}"
+                    iyz="${hip_base_Iyz}"
+                    izz="${hip_base_Izz}" />
+        </inertial>
+        <collision>
+            <origin xyz="0 0 0" rpy="0 0 0"/>
+            <geometry>
+                <box size="${width} ${hip_base_height} ${width}"/>
+            </geometry>
+        </collision>
+    </link>
     <!-- IMU-->
     <link name="imu_link">
     </link>
-    <xacro:frame_part name="hip_aa_frame_left_side"
-                      side="left"
-                      length="${hip_aa_frame_height}"
-                      width="${width}"
-                      direction="y"
-                      visual_origin="${-hip_aa_frame_width} ${hip_base_height/2} 0"
-                      collision_origin="0 ${-hip_aa_frame_height/2} 0"
-                      mesh="LeftHAA.stl"
-    />
-    <xacro:frame_part name="hip_aa_frame_left_front"
-                      side="left"
-                      length="${hip_aa_frame_width}"
-                      width="${width}"
-                      direction="x"
-                      collision_origin="${-hip_aa_frame_width/2} 0 0"
-                      com="${left_hip_aa_com}"
-                      mass="${hip_aa_mass}"
-                      inertia="${all_inertias['hip_aa']}"
-                      />
-    <xacro:frame_part name="upper_leg_left"
-                      side="left"
-                      length="${upper_leg_height}"
-                      width="${width}"
-                      direction="z"
-                      collision_origin="0 0 ${-upper_leg_height/2}"
-                      visual_origin="0 ${hip_base_height/2 + hip_aa_frame_height - upper_leg_offset} 0"
-                      mesh="UpperLeftLeg.stl"
-                      com="${left_upper_leg_com}"
-                      mass="${upper_leg_mass}"
-                      inertia="${all_inertias['upper_leg']}"
-                    />
-    <xacro:frame_part name="lower_leg_left"
-                      side="left"
-                      length="${lower_leg_height}"
-                      width="${width}"
-                      direction="z"
-                      collision_origin="0 0 ${-lower_leg_height/2}"
-                      visual_origin="0 ${hip_base_height/2 + hip_aa_frame_height - upper_leg_offset} ${upper_leg_height}"
-                      mesh="LowerLeftLeg.stl"
-                      com="${left_lower_leg_com}"
-                      mass="${lower_leg_mass}"
-                      inertia="${all_inertias['lower_leg']}"
-                      />
-    <xacro:frame_part name="ankle_plate_left"
-                      side="left"
-                      length="${ankle_plate_height}"
-                      width="${width}"
-                      direction="z"
-                      mesh="LeftFoot.stl"
-                      visual_origin="0
-                                     ${hip_base_height/2 + hip_aa_frame_height - upper_leg_offset - ankle_plate_offset}
-                                     ${foot_scale * (upper_leg_height + lower_leg_height)}"
-                      collision_origin="0 0 ${-ankle_plate_height/2}"
-    />
-    <xacro:pressure_sole side="left" parent="ankle_plate_left"/>
-    <xacro:frame_part name="foot_left"
-                      side="left"
-                      length="${foot_height_forward+foot_height_backward}"
-                      width="${width}"
-                      direction="x"
-                      inertia="${all_inertias['foot']}"
-                      collision_origin="${(-foot_height_forward+foot_height_backward)/2} 0 0"
-                      com="${foot_com_x} ${-foot_com_y} ${foot_com_z}"
-                      mass="${foot_mass}"/>
+    <!-- Left Moving Hip-->
+    <link name="hip_aa_frame_left_side">
+        <visual>
+            <origin xyz="${-hip_aa_frame_width} ${hip_base_height/2} 0" rpy="0 0 ${pi}"/>
+            <geometry>
+                <mesh filename="package://march_description/urdf/stl-files/LeftHAA.stl" scale="1 1 1"/>
+            </geometry>
+            <material name="blue"/>
+        </visual>
+        <collision>
+            <origin xyz="0 ${-hip_aa_frame_height/2} 0" rpy="0 0 0"/>
+            <geometry>
+                <box size="${width} ${hip_aa_frame_height} ${width}"/>
+            </geometry>
+        </collision>
+    </link>
+    <link name="hip_aa_frame_left_front">
+        <inertial>
+            <origin xyz="${hip_aa_com_x} ${-hip_aa_com_y} ${hip_aa_com_z}" rpy="0 0 0"/>
+            <mass value="${hip_aa_mass}"/>
+            <inertia
+                    ixx="${hip_aa_Ixx}"
+                    ixy="${-hip_aa_Ixy}"
+                    ixz="${hip_aa_Ixz}"
+                    iyy="${hip_aa_Iyy}"
+                    iyz="${-hip_aa_Iyz}"
+                    izz="${hip_aa_Izz}" />
+        </inertial>
+        <collision>
+            <origin xyz="${-hip_aa_frame_width/2} 0 0" rpy="0 0 0"/>
+            <geometry>
+                <box size="${hip_aa_frame_width} ${width} ${width}"/>
+            </geometry>
+        </collision>
+    </link>
+    <!-- Upper Leg Left-->
+    <link name="upper_leg_left">
+        <visual>
+            <origin xyz="0 ${hip_base_height/2 + hip_aa_frame_height - upper_leg_offset} 0" rpy="0 0 ${pi}"/>
+            <geometry>
+                <mesh filename="package://march_description/urdf/stl-files/UpperLeftLeg.stl" scale="1 1 1"/>
+            </geometry>
+            <material name="blue"/>
+        </visual>
+        <inertial>
+            <origin xyz="${upper_leg_com_x} ${-upper_leg_com_y} ${upper_leg_com_z}" rpy="0 0 0"/>
+            <mass value="${upper_leg_mass}"/>
+            <inertia
+                    ixx="${upper_leg_Ixx}"
+                    ixy="${-upper_leg_Ixy}"
+                    ixz="${upper_leg_Ixz}"
+                    iyy="${upper_leg_Iyy}"
+                    iyz="${-upper_leg_Iyz}"
+                    izz="${upper_leg_Izz}" />
+        </inertial>
+        <collision>
+            <origin xyz="0 0 ${-upper_leg_height/2}" rpy="0 0 0"/>
+            <geometry>
+                <box size="${width} ${width} ${upper_leg_height}"/>
+            </geometry>
+        </collision>
+    </link>
+    <!-- Lower Leg Left -->
+    <link name="lower_leg_left">
+        <visual>
+            <origin
+                xyz="0 ${hip_base_height/2 + hip_aa_frame_height - upper_leg_offset} ${upper_leg_height}"
+                rpy="0 0 ${pi}"
+            />
+            <geometry>
+                <mesh filename="package://march_description/urdf/stl-files/LowerLeftLeg.stl" scale="1 1 1"/>
+            </geometry>
+            <material name="blue"/>
+        </visual>
+        <inertial>
+            <origin xyz="${lower_leg_com_x} ${-lower_leg_com_y} ${lower_leg_com_z}" rpy="0 0 0"/>
+            <mass value="${lower_leg_mass}"/>
+            <inertia
+                    ixx="${lower_leg_Ixx}"
+                    ixy="${-lower_leg_Ixy}"
+                    ixz="${lower_leg_Ixz}"
+                    iyy="${lower_leg_Iyy}"
+                    iyz="${-lower_leg_Iyz}"
+                    izz="${lower_leg_Izz}" />
+        </inertial>
+        <collision>
+            <origin xyz="0 0 ${-lower_leg_height/2}" rpy="0 0 0"/>
+            <geometry>
+                <box size="${width} ${width} ${lower_leg_height}"/>
+            </geometry>
+        </collision>
+    </link>
+    <!-- Ankle plate Left -->
+    <link name="ankle_plate_left">
+        <visual>
+            <origin
+                xyz="0
+                     ${hip_base_height/2 + hip_aa_frame_height - upper_leg_offset - ankle_plate_offset}
+                     ${foot_scale * (upper_leg_height + lower_leg_height)}"
+                rpy="0 0 ${pi}"
+            />
+            <geometry>
+                <mesh filename="package://march_description/urdf/stl-files/LeftFoot.stl" scale="1 1 ${foot_scale}"/>
+            </geometry>
+            <material name="blue"/>
+        </visual>
+        <collision>
+            <origin xyz="0 0 ${-ankle_plate_height/2}" rpy="0 0 0"/>
+            <geometry>
+                <box size="${width} ${width} ${ankle_plate_height}"/>
+            </geometry>
+        </collision>
+    </link>
+    <gazebo reference="ankle_plate_left">
+        <sensor name="ankle_plate_left_contact" type="contact">
+            <plugin name="contact_plugin" filename="libcontact.so"/>
+            <contact>
+                <collision>ankle_plate_left_fixed_joint_lump__foot_left_collision_1</collision>
+            </contact>
+            <update_rate>30</update_rate>
+            <always_on>true</always_on>
+        </sensor>
+    </gazebo>
+    <!-- Foot Left -->
+    <link name="foot_left">
+        <inertial>
+            <origin xyz="${foot_com_x} ${-foot_com_y} ${foot_com_z}" rpy="0 0 0"/>
+            <mass value="${foot_mass}"/>
+            <inertia
+                    ixx="${foot_Ixx}"
+                    ixy="${-foot_Ixy}"
+                    ixz="${foot_Ixz}"
+                    iyy="${foot_Iyy}"
+                    iyz="${-foot_Iyz}"
+                    izz="${foot_Izz}" />
+        </inertial>
+        <collision>
+            <origin xyz="${(-foot_height_forward+foot_height_backward)/2} 0 0" rpy="0 0 0"/>
+            <geometry>
+                <box size="${foot_height_forward+foot_height_backward} ${width} ${width}"/>
+            </geometry>
+        </collision>
+    </link>
     <link name="pressure_sole_left">
         <collision>
@@ -294,51 +371,104 @@
         <fdir1>1 0 0</fdir1>
     </gazebo>
-    <xacro:frame_part name="hip_aa_frame_right_side"
-                      side="right"
-                      direction="y"
-                      length="${hip_aa_frame_height}"
-                      visual_origin="${-hip_aa_frame_width} ${-hip_base_height/2} 0"
-                      collision_origin="0 ${hip_aa_frame_height/2} 0"
-                      mesh="RightHAA.stl"
-    />
-    <xacro:frame_part name="hip_aa_frame_right_front"
-                      width="${width}"
-                      length="${hip_aa_frame_width}"
-                      collision_origin="${-hip_aa_frame_width/2} 0 0"
-                      side="right"
-                      com="${hip_aa_com_x} ${hip_aa_com_y} ${hip_aa_com_z}"
-                      mass="${hip_aa_mass}"
-                      inertia="${all_inertias['hip_aa']}"
-    />
-    <xacro:frame_part name="upper_leg_right"
-                      side="right"
-                      width="${width}"
-                      length="${upper_leg_height}"
-                      collision_origin="0 0 ${-upper_leg_height/2}"
-                      visual_origin="0 ${-hip_base_height/2 - hip_aa_frame_height + upper_leg_offset} 0"
-                      mesh="UpperRightLeg.stl"
-                      com="${upper_leg_com_x} ${upper_leg_com_y} ${upper_leg_com_z}"
-                      inertia="${all_inertias['upper_leg']}"
-                      mass="${upper_leg_mass}"
-    />
-    <xacro:frame_part name="lower_leg_right"
-                      side="right"
-                      length="${lower_leg_height}"
-                      width="${width}"
-                      visual_origin="0 ${-hip_base_height/2 - hip_aa_frame_height + upper_leg_offset} ${upper_leg_height}"
-                      mesh="LowerRightLeg.stl"
-                      com="${lower_leg_com_x} ${lower_leg_com_y} ${lower_leg_com_z}"
-                      mass="${lower_leg_mass}"
-                      inertia="${all_inertias['lower_leg']}"
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