Commit message: Adding new urdf file for mpc testing

File: ros2/src/shared/march_description/urdf/test_joint_rotational_mpc.xacro (robot description, xacro)
@@ -9,8 +9,8 @@
     <xacro:property name="bar_width" value="0.05"/>
     <xacro:property name="joint_buffer" value="${3*(pi/180)}"/> <!-- rad -->
-    <xacro:property name="joint_lower_limit" value="-0.5363"/> <!-- rad -->
-    <xacro:property name="joint_upper_limit" value="0.5363"/> <!-- rad -->
+    <xacro:property name="joint_lower_limit" value="${-pi}"/> <!-- rad -->
+    <xacro:property name="joint_upper_limit" value="${pi}"/> <!-- rad -->
     <xacro:property name="joint_effort_limit" value="21840"/> <!-- IU = 20 A -->
-    <xacro:property name="joint_velocity_limit" value="2.0"/> <!-- rad/s -->
+    <xacro:property name="joint_velocity_limit" value="20.0"/> <!-- rad/s -->
     <xacro:property name="hover_height" value="0.5"/>
     <xacro:include filename="march.gazebo"/>
@@ -28,5 +28,5 @@
         <axis xyz="0 1 0"/>
         <limit velocity="${joint_velocity_limit}" effort="${joint_effort_limit}" lower="${joint_lower_limit}" upper="${joint_upper_limit}"/>
-        <safety_controller soft_lower_limit="${joint_lower_limit + joint_buffer}" soft_upper_limit="${joint_upper_limit - joint_buffer}" k_position="5" k_velocity="20000" />
+<!--        <safety_controller soft_lower_limit="${joint_lower_limit + joint_buffer}" soft_upper_limit="${joint_upper_limit - joint_buffer}" k_position="5" k_velocity="20000" />-->
     </joint>
     <!-- give colors to some links in gazebo -->
