Commit message: More debug changes

File: ros2/src/shared/march_description/urdf/test_joint_rotational_odrive.xacro (robot description, xacro)
@@ -11,6 +11,6 @@
     <xacro:property name="joint_lower_limit"    value="${-45*(pi/180)}"/>   <!-- rad -->
     <xacro:property name="joint_upper_limit"    value="${45*(pi/180)}"/>     <!-- rad -->
-    <xacro:property name="joint_effort_limit"   value="10"/>                <!-- IU -->
-    <xacro:property name="joint_velocity_limit" value="2.0"/>               <!-- rad/s -->
+    <xacro:property name="joint_effort_limit"   value="30"/>                <!-- IU -->
+    <xacro:property name="joint_velocity_limit" value="3.0"/>               <!-- rad/s -->
     <xacro:property name="hover_height" value="0.5"/>
     <xacro:include filename="march.gazebo"/>

Commit message: Clean up code

File: ros2/src/shared/march_description/urdf/test_joint_rotational_odrive.xacro (robot description, xacro)
@@ -11,5 +11,5 @@
     <xacro:property name="joint_lower_limit"    value="${-45*(pi/180)}"/>   <!-- rad -->
     <xacro:property name="joint_upper_limit"    value="${45*(pi/180)}"/>     <!-- rad -->
-    <xacro:property name="joint_effort_limit"   value="30"/>                <!-- IU -->
+    <xacro:property name="joint_effort_limit"   value="20"/>                <!-- IU -->
     <xacro:property name="joint_velocity_limit" value="3.0"/>               <!-- rad/s -->
     <xacro:property name="hover_height" value="0.5"/>

Commit message: Airgaitgit status

File: ros2/src/shared/march_description/urdf/test_joint_rotational_odrive.xacro (robot description, xacro)
@@ -9,6 +9,6 @@
     <xacro:property name="bar_width" value="0.05"/>
     <xacro:property name="joint_buffer"         value="${3*(pi/180)}"/>     <!-- rad -->
-    <xacro:property name="joint_lower_limit"    value="${-45*(pi/180)}"/>   <!-- rad -->
-    <xacro:property name="joint_upper_limit"    value="${45*(pi/180)}"/>     <!-- rad -->
+    <xacro:property name="joint_lower_limit"    value="-0.4395"/>   <!-- rad -->
+    <xacro:property name="joint_upper_limit"    value="1.7857"/>     <!-- rad -->
     <xacro:property name="joint_effort_limit"   value="20"/>                <!-- IU -->
     <xacro:property name="joint_velocity_limit" value="3.0"/>               <!-- rad/s -->
@@ -75,5 +75,5 @@
         </joint>
         <actuator name="rotational_joint_motor">
-            <mechanicalReduction>101</mechanicalReduction>
+            <mechanicalReduction>121</mechanicalReduction>
         </actuator>
     </transmission>
