Commit message: All joints activated again but structure to turn them off is kept

File: ros2/src/shared/march_description/urdf/march6_debug.xacro (robot description, xacro)
@@ -293,19 +293,19 @@
         <origin xyz="0 0 ${lower_leg_height+upper_leg_height+ankle_plate_height+width/2.0+hover_height}" rpy="0 0 0"/>
     </joint>
-    <!--    <xacro:march_joint-->
-    <!--            name="left_hip_aa"-->
-    <!--            parent="hip_base"-->
-    <!--            child="hip_aa_frame_left_side"-->
-    <!--            origin="0 ${-hip_base_height/2} 0"-->
-    <!--            axis="-1 0 0"-->
-    <!--            safety="${safety_values['haa']}"-->
-    <!--            limits="${joint_limits['left_haa']}"-->
-    <!--            reduction="${linear_reduction_hip}"-->
-    <!--    />-->
-    <joint name="left_hip_aa" type="fixed">
-        <parent link="hip_base"/>
-        <child link="hip_aa_frame_left_side"/>
-        <origin xyz="0 ${-hip_base_height/2} 0"/>
-    </joint>
+        <xacro:march_joint
+                name="left_hip_aa"
+                parent="hip_base"
+                child="hip_aa_frame_left_side"
+                origin="0 ${-hip_base_height/2} 0"
+                axis="-1 0 0"
+                safety="${safety_values['haa']}"
+                limits="${joint_limits['left_haa']}"
+                reduction="${linear_reduction_hip}"
+        />
+<!--    <joint name="left_hip_aa" type="fixed">-->
+<!--        <parent link="hip_base"/>-->
+<!--        <child link="hip_aa_frame_left_side"/>-->
+<!--        <origin xyz="0 ${-hip_base_height/2} 0"/>-->
+<!--    </joint>-->
     <joint name="left_hip_angle" type="fixed">
         <parent link="hip_aa_frame_left_side"/>
@@ -338,9 +338,9 @@
             limits="${joint_limits['left_knee']}"
     />
-    <!--    <joint name="left_knee" type="fixed">-->
-    <!--        <parent link="upper_leg_left"/>-->
-    <!--        <child link="lower_leg_left"/>-->
-    <!--        <origin xyz="0 ${knee_offset} ${-upper_leg_height}"/>-->
-    <!--    </joint>-->
+<!--        <joint name="left_knee" type="fixed">-->
+<!--            <parent link="upper_leg_left"/>-->
+<!--            <child link="lower_leg_left"/>-->
+<!--            <origin xyz="0 ${knee_offset} ${-upper_leg_height}"/>-->
+<!--        </joint>-->
     <xacro:march_joint
             name="left_ankle"
@@ -353,9 +353,9 @@
             limits="${joint_limits['left_ankle']}"
     />
-    <!--    <joint name="left_ankle" type="fixed">-->
-    <!--        <parent link="lower_leg_left"/>-->
-    <!--        <child link=""/>-->
-    <!--        <origin xyz=""/>-->
-    <!--    </joint>-->
+<!--        <joint name="left_ankle" type="fixed">-->
+<!--            <parent link="lower_leg_left"/>-->
+<!--            <child link="ankle_plate_left"/>-->
+<!--            <origin xyz="0 ${ankle_plate_offset} ${-lower_leg_height}"/>-->
+<!--        </joint>-->
     <joint name="left_foot_angle" type="fixed">
         <parent link="ankle_plate_left"/>
@@ -363,19 +363,19 @@
         <origin xyz="0 0 ${-ankle_plate_height-width/2}" rpy="0 0 0"/>
     </joint>
-    <!--    <xacro:march_joint-->
-    <!--            name="right_hip_aa"-->
-    <!--            parent="hip_base"-->
-    <!--            child="hip_aa_frame_right_side"-->
-    <!--            origin="0 ${hip_base_height/2} 0"-->
-    <!--            axis="1 0 0"-->
-    <!--            safety="${safety_values['haa']}"-->
-    <!--            reduction="${linear_reduction_ankle}"-->
-    <!--            limits="${joint_limits['right_haa']}"-->
-    <!--    />-->
-    <joint name="right_hip_aa" type="fixed">
-        <parent link="hip_base"/>
-        <child link="hip_aa_frame_right_side"/>
-        <origin xyz="0 ${hip_base_height/2} 0"/>
-    </joint>
+        <xacro:march_joint
+                name="right_hip_aa"
+                parent="hip_base"
+                child="hip_aa_frame_right_side"
+                origin="0 ${hip_base_height/2} 0"
+                axis="1 0 0"
+                safety="${safety_values['haa']}"
+                reduction="${linear_reduction_ankle}"
+                limits="${joint_limits['right_haa']}"
+        />
+<!--    <joint name="right_hip_aa" type="fixed">-->
+<!--        <parent link="hip_base"/>-->
+<!--        <child link="hip_aa_frame_right_side"/>-->
+<!--        <origin xyz="0 ${hip_base_height/2} 0"/>-->
+<!--    </joint>-->
     <joint name="right_hip_angle" type="fixed">
         <parent link="hip_aa_frame_right_side"/>
@@ -383,49 +383,49 @@
         <origin xyz="0 ${hip_aa_frame_height} 0" rpy="0 0 0"/>
     </joint>
-    <!--    <xacro:march_joint-->
-    <!--            name="right_hip_fe"-->
-    <!--            parent="hip_aa_frame_right_front"-->
-    <!--            child="upper_leg_right"-->
-    <!--            origin="${-hip_aa_frame_width} ${-upper_leg_offset} 0"-->
-    <!--            axis="0 1 0"-->
-    <!--            safety="${safety_values['hfe']}"-->
-    <!--            reduction="${rotary_reduction}"-->
-    <!--            limits="${joint_limits['right_hfe']}"-->
-    <!--    />-->
-    <joint name="right_hip_fe" type="fixed">
-        <parent link="hip_aa_frame_right_front"/>
-        <child link="upper_leg_right"/>
-        <origin xyz="${-hip_aa_frame_width} ${-upper_leg_offset} 0"/>
-    </joint>
-    <!--    <xacro:march_joint-->
-    <!--            name="right_knee"-->
-    <!--            parent="upper_leg_right"-->
-    <!--            child="lower_leg_right"-->
-    <!--            origin="0 ${-knee_offset} ${-upper_leg_height}"-->
-    <!--            axis="0 -1 0"-->
-    <!--            safety="${safety_values['knee']}"-->
-    <!--            limits="${joint_limits['right_knee']}"-->
-    <!--            reduction="${rotary_reduction}"-->
-    <!--    />-->
-    <joint name="right_knee" type="fixed">
-        <parent link="upper_leg_right"/>
-        <child link="lower_leg_right"/>
-        <origin xyz="0 ${-knee_offset} ${-upper_leg_height}"/>
-    </joint>
-    <!--        <xacro:march_joint-->
-    <!--                name="right_ankle"-->
-    <!--                parent="lower_leg_right"-->
-    <!--                child="ankle_plate_right"-->
-    <!--                safety="${safety_values['ankle']}"-->
-    <!--                origin="0 ${-ankle_plate_offset} ${-lower_leg_height}"-->
-    <!--                axis="0 1 0"-->
-    <!--                reduction="${linear_reduction_ankle}"-->
-    <!--                limits="${joint_limits['right_ankle']}"-->
-    <!--        />-->
-    <joint name="right_ankle" type="fixed">
-        <parent link="lower_leg_right"/>
-        <child link="ankle_plate_right"/>
-        <origin xyz="0 ${-ankle_plate_offset} ${-lower_leg_height}"/>
-    </joint>
+        <xacro:march_joint
+                name="right_hip_fe"
+                parent="hip_aa_frame_right_front"
+                child="upper_leg_right"
+                origin="${-hip_aa_frame_width} ${-upper_leg_offset} 0"
+                axis="0 1 0"
+                safety="${safety_values['hfe']}"
+                reduction="${rotary_reduction}"
+                limits="${joint_limits['right_hfe']}"
+        />
+<!--    <joint name="right_hip_fe" type="fixed">-->
+<!--        <parent link="hip_aa_frame_right_front"/>-->
+<!--        <child link="upper_leg_right"/>-->
+<!--        <origin xyz="${-hip_aa_frame_width} ${-upper_leg_offset} 0"/>-->
+<!--    </joint>-->
+        <xacro:march_joint
+                name="right_knee"
+                parent="upper_leg_right"
+                child="lower_leg_right"
+                origin="0 ${-knee_offset} ${-upper_leg_height}"
+                axis="0 -1 0"
+                safety="${safety_values['knee']}"
+                limits="${joint_limits['right_knee']}"
+                reduction="${rotary_reduction}"
+        />
+<!--    <joint name="right_knee" type="fixed">-->
+<!--        <parent link="upper_leg_right"/>-->
+<!--        <child link="lower_leg_right"/>-->
+<!--        <origin xyz="0 ${-knee_offset} ${-upper_leg_height}"/>-->
+<!--    </joint>-->
+            <xacro:march_joint
+                    name="right_ankle"
+                    parent="lower_leg_right"
+                    child="ankle_plate_right"
+                    safety="${safety_values['ankle']}"
+                    origin="0 ${-ankle_plate_offset} ${-lower_leg_height}"
+                    axis="0 1 0"
+                    reduction="${linear_reduction_ankle}"
+                    limits="${joint_limits['right_ankle']}"
+            />
+<!--    <joint name="right_ankle" type="fixed">-->
+<!--        <parent link="lower_leg_right"/>-->
+<!--        <child link="ankle_plate_right"/>-->
+<!--        <origin xyz="0 ${-ankle_plate_offset} ${-lower_leg_height}"/>-->
+<!--    </joint>-->
     <joint name="right_foot_angle" type="fixed">
         <parent link="ankle_plate_right"/>
