Commit message: Re-add camera to xacro

File: ros2/src/shared/march_description/urdf/march4.xacro (robot description, xacro)
@@ -692,4 +692,8 @@
         <origin xyz="0 0 ${-ankle_plate_height}" rpy="0 0 0"/>
     </joint>
+    <xacro:include filename="$(find realsense2_description)/urdf/_d435.urdf.xacro" />
+    <xacro:sensor_d435 parent="upper_leg_left">
+        <origin xyz="0 0 0" rpy="0 0 3.1416"/>
+    </xacro:sensor_d435>
     <!-- ROS Control plugin for Gazebo -->
     <transmission name="left_hip_aa">

Commit message: Fix the safety values for simulation working correctly (imperfect solution)

File: ros2/src/shared/march_description/urdf/march4.xacro (robot description, xacro)
@@ -25,27 +25,22 @@
         </gazebo>
     </xacro:if>
-    <!-- The max effort of the rotary joints is lower then the value corresponding to 25A, because short-circuit errors
-    have occured while applying the theoretical max effort for a long time. -->
-    <xacro:arg name="max_effort_rotary" default="18000.0" />
-    <xacro:arg name="max_effort_linear" default="22932.0" />  <!-- = 28 A -->
-    <xacro:property name="max_effort_rotary" value="$(arg max_effort_rotary)" />
-    <xacro:property name="max_effort_linear" value="$(arg max_effort_linear)" />
-    <!-- Values for the safety limits, see https://wiki.ros.org/pr2_controller_manager/safety_limits -->
-    <xacro:arg name="k_velocity_value_hfe" default="20000.0" />
-    <xacro:arg name="k_velocity_value_kfe" default="20000.0" />
-    <xacro:arg name="k_velocity_value_haa" default="20000.0" />
-    <xacro:arg name="k_velocity_value_adpf" default="20000.0" />
-    <xacro:property name="k_velocity_value_hfe" value="$(arg k_velocity_value_hfe)" />
-    <xacro:property name="k_velocity_value_kfe" value="$(arg k_velocity_value_kfe)" />
-    <xacro:property name="k_velocity_value_haa" value="$(arg k_velocity_value_haa)" />
-    <xacro:property name="k_velocity_value_adpf" value="$(arg k_velocity_value_adpf)" />
-    <xacro:arg name="k_position_value_hfe" default="14.88" />
-    <xacro:arg name="k_position_value_kfe" default="14.88" />
-    <xacro:arg name="k_position_value_haa" default="4.0" />
-    <xacro:arg name="k_position_value_adpf" default="5.0" />
-    <xacro:property name="k_position_value_hfe" value="$(arg k_position_value_hfe)" />
-    <xacro:property name="k_position_value_kfe" value="$(arg k_position_value_kfe)" />
-    <xacro:property name="k_position_value_haa" value="$(arg k_position_value_haa)" />
-    <xacro:property name="k_position_value_adpf" value="$(arg k_position_value_adpf)" />
+    <xacro:arg name="configuration" default="exoskeleton"/>
+    <xacro:property name="configuration" value="$(arg configuration)"/>
+<!-- Include all macro files    -->
+    <xacro:include filename="macros/safety_limits.xacro" />
+    <xacro:include filename="macros/pressure_sole.xacro"/>
+    <xacro:include filename="macros/frame_part.xacro"/>
+    <xacro:include filename="macros/joint.xacro"/>
+<!-- Add yaml files with properties -->
+    <xacro:property name="joint_limits_yaml_file" value="properties/march4_joint_limits.yaml"/>
+    <xacro:property name="joint_limits" value="${load_yaml(joint_limits_yaml_file)}"/>
+    <xacro:property name="safety_yaml_file" value="properties/march4_safety_${configuration}.yaml"/>
+    <xacro:property name="safety_values" value="${load_yaml(safety_yaml_file)}"/>
+    <xacro:property name="inertia_yaml_file" value="properties/march4_inertia.yaml"/>
+    <xacro:property name="inertia" value="${load_yaml(inertia_yaml_file)}"/>
+    <xacro:property name="dimensions_yaml_file" value="properties/march4_dimensions.yaml"/>
+    <xacro:property name="dimensions" value="${load_yaml(dimensions_yaml_file)}"/>
+    <xacro:property name="rotary_reduction" value="101"/>
+    <xacro:property name="linear_reduction" value="200"/>
     <!-- Constants for robot dimensions -->
     <!-- Masses determined in Catia, see https://confluence.projectmarch.nl:8443/display/51/URDF+description -->
@@ -101,74 +96,4 @@
     <xacro:property name="foot_com_z" value="${upper_leg_height + lower_leg_height + ankle_plate_height - 0.789788}"/>
     <xacro:property name="foot_scale" value="1.35"/>
-    <!-- Inertia of the parts -->
-    <!-- Inertia's have been determined in Catia, see
-         https://confluence.projectmarch.nl:8443/display/51/URDF+description -->
-    <!-- The inertia's were defined around the CoM. Note that in the Catia x axis is the URDF y axis and the Catia y
-         axis is the negative URDF x axis, see confluence for the impact. The given inertia's are for the right leg,
-         Ixy and Iyz will be inverted for the left leg. -->
-    <xacro:property name="hip_base_Ixx" value="0.141"/>
-    <xacro:property name="hip_base_Ixy" value="0.0000336"/>
-    <xacro:property name="hip_base_Ixz" value="-0.007"/>
-    <xacro:property name="hip_base_Iyy" value="0.087"/>
-    <xacro:property name="hip_base_Iyz" value="0.0005089"/>
-    <xacro:property name="hip_base_Izz" value="0.091"/>
-    <xacro:property name="hip_aa_Ixx" value="0.013"/>
-    <xacro:property name="hip_aa_Ixy" value="0.008"/>
-    <xacro:property name="hip_aa_Ixz" value="0.005"/>
-    <xacro:property name="hip_aa_Iyy" value="0.023"/>
-    <xacro:property name="hip_aa_Iyz" value="-0.001"/>
-    <xacro:property name="hip_aa_Izz" value="0.028"/>
-    <xacro:property name="upper_leg_Ixx" value="0.127"/>
-    <xacro:property name="upper_leg_Ixy" value="0.0001291"/>
-    <xacro:property name="upper_leg_Ixz" value="-0.0002056"/>
-    <xacro:property name="upper_leg_Iyy" value="0.122"/>
-    <xacro:property name="upper_leg_Iyz" value="0.016"/>
-    <xacro:property name="upper_leg_Izz" value="0.015"/>
-    <xacro:property name="lower_leg_Ixx" value="0.075"/>
-    <xacro:property name="lower_leg_Ixy" value="-0.027"/>
-    <xacro:property name="lower_leg_Ixz" value="-0.008"/>
-    <xacro:property name="lower_leg_Iyy" value="0.11"/>
-    <xacro:property name="lower_leg_Iyz" value="-0.002"/>
-    <xacro:property name="lower_leg_Izz" value="0.071" />
-    <xacro:property name="foot_Ixx" value="0.021"/>
-    <xacro:property name="foot_Ixy" value="-0.002"/>
-    <xacro:property name="foot_Ixz" value="0.02"/>
-    <xacro:property name="foot_Iyy" value="0.027"/>
-    <xacro:property name="foot_Iyz" value="0.004"/>
-    <xacro:property name="foot_Izz" value="0.01" />
-    <!-- Joint properties -->
-    <!-- For limit calculations, see https://confluence.projectmarch.nl:8443/pages/viewpage.action?pageId=268697604 -->
-    <xacro:property name="left_hip_fe_rotation_lower_limit" value="${-21.04431152*pi/180}"/> <!-- rad -->
-    <xacro:property name="left_hip_fe_rotation_upper_limit" value="${98.97033691*pi/180}"/> <!-- rad -->
-    <xacro:property name="right_hip_fe_rotation_lower_limit" value="${-20.23406982*pi/180}"/> <!-- rad -->
-    <xacro:property name="right_hip_fe_rotation_upper_limit" value="${99.48120117*pi/180}"/> <!-- rad -->
-    <xacro:property name="hip_fe_soft_buffer" value="${3*pi/180}"/> <!-- rad -->
-    <xacro:property name="hip_fe_effort_limit" value="${max_effort_rotary}"/> <!-- IU -->
-    <xacro:property name="hip_fe_velocity_limit" value="2.0"/> <!-- rad/s -->
-    <xacro:property name="left_hip_aa_rotation_lower_limit" value="${-18.54492188*pi/180}"/> <!-- rad -->
-    <xacro:property name="left_hip_aa_rotation_upper_limit" value="${16.34765625*pi/180}"/> <!-- rad -->
-    <xacro:property name="right_hip_aa_rotation_lower_limit" value="${-18.10546875*pi/180}"/> <!-- rad -->
-    <xacro:property name="right_hip_aa_rotation_upper_limit" value="${15.99609375*pi/180}"/> <!-- rad -->
-    <xacro:property name="hip_aa_soft_buffer" value="${3.5*pi/180}"/> <!-- rad -->
-    <xacro:property name="hip_aa_effort_limit" value="${max_effort_linear}"/> <!-- IU -->
-    <xacro:property name="hip_aa_velocity_limit" value="1.0"/> <!-- rad/s -->
-    <xacro:property name="left_knee_rotation_lower_limit" value="${-5.012512207*pi/180}"/>
-    <xacro:property name="left_knee_rotation_upper_limit" value="${112.4230957*pi/180}"/>
-    <xacro:property name="right_knee_rotation_lower_limit" value="${-4.89440918*pi/180}"/>
-    <xacro:property name="right_knee_rotation_upper_limit" value="${115.3097534*pi/180}"/>
-    <xacro:property name="knee_extension_soft_buffer" value="${3.5*pi/180}"/> <!-- rad -->
-    <xacro:property name="knee_flexion_soft_buffer" value="${3*pi/180}"/> <!-- rad -->
-    <xacro:property name="knee_effort_limit" value="${max_effort_rotary}"/> <!-- IU -->
-    <xacro:property name="knee_velocity_limit" value="2.5"/>
-    <xacro:property name="left_ankle_rotation_lower_limit" value="${-26.30401611*pi/180}"/>
-    <xacro:property name="left_ankle_rotation_upper_limit" value="${15.88348389*pi/180}"/>
-    <xacro:property name="right_ankle_rotation_lower_limit" value="${-23.203125*pi/180}"/>
-    <xacro:property name="right_ankle_rotation_upper_limit" value="${14.23828125*pi/180}"/>
-    <xacro:property name="ankle_dorsalflexion_soft_buffer" value="${5*pi/180}"/> <!-- rad -->
-    <xacro:property name="ankle_plantarflexion_soft_buffer" value="${3*pi/180}"/> <!-- rad -->
-    <xacro:property name="ankle_effort_limit" value="${max_effort_linear}"/> <!-- IU -->
-    <xacro:property name="ankle_velocity_limit" value="1.0"/>
-    <xacro:property name="camera_link" value="0.05"/> <!-- Size of square 'camera' box -->
-    <xacro:property name="axel_offset" value="0.05"/> <!-- Space btw top of beam and the each joint -->
     <!-- Import all Gazebo-customization elements, including Gazebo colors -->
     <xacro:include filename="march.gazebo"/>
@@ -180,196 +105,76 @@
     <!-- Parts -->
     <!-- Hip-->
-    <link name="hip_base">
-        <visual>
-            <origin xyz="${-hip_aa_frame_width} 0 0" rpy="0 0 ${pi}"/>
-            <geometry>
-                <mesh filename="package://march_description/urdf/stl-files/HipBase.stl" scale="1 1 1"/>
-            </geometry>
-            <material name="blue"/>
-        </visual>
-        <inertial>
-            <origin xyz="${hip_base_com_x} ${hip_base_com_y} ${hip_base_com_z}" rpy="0 0 0"/>
-            <mass value="${hip_base_mass}"/>
-            <inertia
-                    ixx="${hip_base_Ixx}"
-                    ixy="${hip_base_Ixy}"
-                    ixz="${hip_base_Ixz}"
-                    iyy="${hip_base_Iyy}"
-                    iyz="${hip_base_Iyz}"
-                    izz="${hip_base_Izz}" />
-        </inertial>
-        <collision>
-            <origin xyz="0 0 0" rpy="0 0 0"/>
-            <geometry>
-                <box size="${width} ${hip_base_height} ${width}"/>
-            </geometry>
-        </collision>
-    </link>
+    <xacro:frame_part name="hip_base"
+                      reflect="1"
+                      length="${hip_base_height}"
+                      direction="y"
+                      visual_origin="${-hip_aa_frame_width} 0 0"
+                      collision_origin="0 0 0"
+                      mesh="HipBase.stl"
+                      com="${hip_base_com_x} ${hip_base_com_y} ${hip_base_com_z}"
+                      mass="${hip_base_mass}"
+                      inertia="${inertia['hip_base']}"
+    />
     <!-- IMU-->
     <link name="imu_link">
     </link>
-    <!-- Left Moving Hip-->
-    <link name="hip_aa_frame_left_side">
-        <visual>
-            <origin xyz="${-hip_aa_frame_width} ${hip_base_height/2} 0" rpy="0 0 ${pi}"/>
-            <geometry>
-                <mesh filename="package://march_description/urdf/stl-files/LeftHAA.stl" scale="1 1 1"/>
-            </geometry>
-            <material name="blue"/>
-        </visual>
-        <collision>
-            <origin xyz="0 ${-hip_aa_frame_height/2} 0" rpy="0 0 0"/>
-            <geometry>
-                <box size="${width} ${hip_aa_frame_height} ${width}"/>
-            </geometry>
-        </collision>
-    </link>
-    <link name="hip_aa_frame_left_front">
-        <inertial>
-            <origin xyz="${hip_aa_com_x} ${-hip_aa_com_y} ${hip_aa_com_z}" rpy="0 0 0"/>
-            <mass value="${hip_aa_mass}"/>
-            <inertia
-                    ixx="${hip_aa_Ixx}"
-                    ixy="${-hip_aa_Ixy}"
-                    ixz="${hip_aa_Ixz}"
-                    iyy="${hip_aa_Iyy}"
-                    iyz="${-hip_aa_Iyz}"
-                    izz="${hip_aa_Izz}" />
-        </inertial>
-        <collision>
-            <origin xyz="${-hip_aa_frame_width/2} 0 0" rpy="0 0 0"/>
-            <geometry>
-                <box size="${hip_aa_frame_width} ${width} ${width}"/>
-            </geometry>
-        </collision>
-    </link>
-    <!-- Upper Leg Left-->
-    <link name="upper_leg_left">
-        <visual>
-            <origin xyz="0 ${hip_base_height/2 + hip_aa_frame_height - upper_leg_offset} 0" rpy="0 0 ${pi}"/>
-            <geometry>
-                <mesh filename="package://march_description/urdf/stl-files/UpperLeftLeg.stl" scale="1 1 1"/>
-            </geometry>
-            <material name="blue"/>
-        </visual>
-        <inertial>
-            <origin xyz="${upper_leg_com_x} ${-upper_leg_com_y} ${upper_leg_com_z}" rpy="0 0 0"/>
-            <mass value="${upper_leg_mass}"/>
-            <inertia
-                    ixx="${upper_leg_Ixx}"
-                    ixy="${-upper_leg_Ixy}"
-                    ixz="${upper_leg_Ixz}"
-                    iyy="${upper_leg_Iyy}"
-                    iyz="${-upper_leg_Iyz}"
-                    izz="${upper_leg_Izz}" />
-        </inertial>
-        <collision>
-            <origin xyz="0 0 ${-upper_leg_height/2}" rpy="0 0 0"/>
-            <geometry>
-                <box size="${width} ${width} ${upper_leg_height}"/>
-            </geometry>
-        </collision>
-    </link>
-    <!-- Lower Leg Left -->
-    <link name="lower_leg_left">
-        <visual>
-            <origin
-                xyz="0 ${hip_base_height/2 + hip_aa_frame_height - upper_leg_offset} ${upper_leg_height}"
-                rpy="0 0 ${pi}"
-            />
-            <geometry>
-                <mesh filename="package://march_description/urdf/stl-files/LowerLeftLeg.stl" scale="1 1 1"/>
-            </geometry>
-            <material name="blue"/>
-        </visual>
-        <inertial>
-            <origin xyz="${lower_leg_com_x} ${-lower_leg_com_y} ${lower_leg_com_z}" rpy="0 0 0"/>
-            <mass value="${lower_leg_mass}"/>
-            <inertia
-                    ixx="${lower_leg_Ixx}"
-                    ixy="${-lower_leg_Ixy}"
-                    ixz="${lower_leg_Ixz}"
-                    iyy="${lower_leg_Iyy}"
-                    iyz="${-lower_leg_Iyz}"
-                    izz="${lower_leg_Izz}" />
-        </inertial>
-        <collision>
-            <origin xyz="0 0 ${-lower_leg_height/2}" rpy="0 0 0"/>
-            <geometry>
-                <box size="${width} ${width} ${lower_leg_height}"/>
-            </geometry>
-        </collision>
-    </link>
-    <!-- Ankle plate Left -->
-    <link name="ankle_plate_left">
-        <visual>
-            <origin
-                xyz="0
-                     ${hip_base_height/2 + hip_aa_frame_height - upper_leg_offset - ankle_plate_offset}
-                     ${foot_scale * (upper_leg_height + lower_leg_height)}"
-                rpy="0 0 ${pi}"
-            />
-            <geometry>
-                <mesh filename="package://march_description/urdf/stl-files/LeftFoot.stl" scale="1 1 ${foot_scale}"/>
-            </geometry>
-            <material name="blue"/>
-        </visual>
-        <collision>
-            <origin xyz="0 0 ${-ankle_plate_height/2}" rpy="0 0 0"/>
-            <geometry>
-                <box size="${width} ${width} ${ankle_plate_height}"/>
-            </geometry>
-        </collision>
-    </link>
-    <gazebo reference="ankle_plate_left">
-        <sensor name="ankle_plate_left_contact" type="contact">
-            <plugin name="contact_plugin" filename="libcontact.so"/>
-            <contact>
-                <collision>ankle_plate_left_fixed_joint_lump__foot_left_collision_1</collision>
-            </contact>
-            <update_rate>30</update_rate>
-            <always_on>true</always_on>
-        </sensor>
-    </gazebo>
-    <!-- Foot Left -->
-    <link name="foot_left">
-        <inertial>
-            <origin xyz="${foot_com_x} ${-foot_com_y} ${foot_com_z}" rpy="0 0 0"/>
-            <mass value="${foot_mass}"/>
-            <inertia
-                    ixx="${foot_Ixx}"
-                    ixy="${-foot_Ixy}"
-                    ixz="${foot_Ixz}"
-                    iyy="${foot_Iyy}"
-                    iyz="${-foot_Iyz}"
-                    izz="${foot_Izz}" />
-        </inertial>
-        <collision>
-            <origin xyz="${(-foot_height_forward+foot_height_backward)/2} 0 0" rpy="0 0 0"/>
-            <geometry>
-                <box size="${foot_height_forward+foot_height_backward} ${width} ${width}"/>
-            </geometry>
-        </collision>
-    </link>
-    <link name="pressure_sole_left">
-        <collision>
-            <origin xyz="${(-foot_height_forward+foot_height_backward)/2} 0 0" rpy="0 0 0"/>
-            <geometry>
-                <box size="${foot_height_forward+foot_height_backward} ${width} 0.001"/>
-            </geometry>
-        </collision>
-    </link>
-    <gazebo reference="pressure_sole_left">
-        <sensor name="left_pressure_sole" type="contact">
-            <always_on>true</always_on>
-            <contact>
-                <collision>ankle_plate_left_fixed_joint_lump__pressure_sole_left_collision_2</collision>
-            </contact>
-            <plugin name="left_foot_plugin" filename="libgazebo_ros_bumper.so">
-                <bumperTopicName>march/sensor/left_pressure_sole</bumperTopicName>
-                <frameName>world</frameName>
-            </plugin>
-        </sensor>
-    </gazebo>
+    <xacro:frame_part name="hip_aa_frame_left_side"
+                      reflect="-1"
+                      length="${hip_aa_frame_height}"
+                      direction="y"
+                      collision_origin="0 ${-hip_aa_frame_height/2} 0"
+                      visual_origin="${-hip_aa_frame_width} ${hip_base_height/2} 0"
+                      mesh="LeftHAA.stl"
+    />
+    <xacro:frame_part name="hip_aa_frame_left_front"
+                      reflect="-1"
+                      length="${hip_aa_frame_width}"
+                      direction="x"
+                      collision_origin="${-hip_aa_frame_width/2} 0 0"
+                      com="${hip_aa_com_x} ${-hip_aa_com_y} ${hip_aa_com_z}"
+                      mass="${hip_aa_mass}"
+                      inertia="${inertia['hip_aa']}"
+                      />
+    <xacro:frame_part name="upper_leg_left"
+                      reflect="-1"
+                      length="${upper_leg_height}"
+                      direction="z"
+                      collision_origin="0 0 ${-upper_leg_height/2}"
+                      visual_origin="0 ${hip_base_height/2 + hip_aa_frame_height - upper_leg_offset} 0"
+                      mesh="UpperLeftLeg.stl"
+                      com="${upper_leg_com_x} ${-upper_leg_com_y} ${upper_leg_com_z}"
+                      mass="${upper_leg_mass}"
+                      inertia="${inertia['upper_leg']}"
+                    />
+    <xacro:frame_part name="lower_leg_left"
+                      reflect="-1"
+                      length="${lower_leg_height}"
+                      direction="z"
+                      collision_origin="0 0 ${-lower_leg_height/2}"
+                      visual_origin="0 ${hip_base_height/2 + hip_aa_frame_height - upper_leg_offset} ${upper_leg_height}"
+                      mesh="LowerLeftLeg.stl"
+                      com="${lower_leg_com_x} ${-lower_leg_com_y} ${lower_leg_com_z}"
+                      mass="${lower_leg_mass}"
+                      inertia="${inertia['lower_leg']}"
+                      />
+    <xacro:frame_part name="ankle_plate_left"
+                      reflect="-1"
+                      length="${ankle_plate_height}"
+                      direction="z"
+                      mesh="LeftFoot.stl"
+                      visual_origin="0
+                                     ${hip_base_height/2 + hip_aa_frame_height - upper_leg_offset - ankle_plate_offset}
+                                     ${foot_scale * (upper_leg_height + lower_leg_height)}"
+                      scale="1 1 ${foot_scale}"
+                      collision_origin="0 0 ${-ankle_plate_height/2}"
+    />
+    <xacro:frame_part name="foot_left"
+                      reflect="-1"
+                      length="${foot_height_forward+foot_height_backward}"
+                      direction="x"
+                      inertia="${inertia['foot']}"
+                      collision_origin="${-(foot_height_forward+foot_height_backward)/2} 0 0"
+                      com="${foot_com_x} ${-foot_com_y} ${foot_com_z}"
+                      mass="${foot_mass}"/>
     <gazebo reference="foot_left">
         <mu1>${foot_mu1}</mu1>
@@ -378,147 +183,65 @@
         <fdir1>1 0 0</fdir1>
     </gazebo>
-    <!-- Right Moving Hip-->
-    <link name="hip_aa_frame_right_side">
-        <visual>
-            <origin xyz="${-hip_aa_frame_width} ${-hip_base_height/2} 0" rpy="0 0 ${pi}"/>
-            <geometry>
-                <mesh filename="package://march_description/urdf/stl-files/RightHAA.stl" scale="1 1 1"/>
-            </geometry>
-            <material name="blue"/>
-        </visual>
-        <collision>
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
Commit message: Fix placement of the camera

File: ros2/src/shared/march_description/urdf/march4.xacro (robot description, xacro)
@@ -693,6 +693,9 @@
     </joint>
     <xacro:include filename="camera/_d435.urdf.xacro" />
-    <xacro:sensor_d435 parent="upper_leg_left">
-        <origin xyz="0 0 0" rpy="0 0 3.1416"/>
+    <xacro:sensor_d435 parent="hip_base">
+<!--    Attached to the hip_base, since this is most comparable to the backpack -->
+<!--    in amount of movement-->
+        <origin xyz="-0.15 0.18 0.18" rpy="${0.5 * pi} ${0.25 * pi} ${pi}"/>
+        <!-- Rotate to be vertical and pointing down 45 degrees -->
     </xacro:sensor_d435>
     <!-- ROS Control plugin for Gazebo -->

File: ros2/src/shared/march_description/urdf/march4_with_koen_lengths.xacro (robot description, xacro)
@@ -645,6 +645,9 @@
     </joint>
     <xacro:include filename="camera/_d435.urdf.xacro" />
-    <xacro:sensor_d435 parent="upper_leg_left">
-        <origin xyz="0 0 0" rpy="0 0 3.1416"/>
+    <xacro:sensor_d435 parent="hip_base">
+        <!--    Attached to the hip_base, since this is most comparable to the backpack -->
+        <!--    in amount of movement-->
+        <origin xyz="-0.15 0.18 0.18" rpy="${0.5 * pi} ${0.25 * pi} ${pi}"/>
+        <!-- Rotate to be vertical and pointing down 45 degrees -->
     </xacro:sensor_d435>
     <!-- ROS Control plugin for Gazebo -->
