Commit message: Small change to move to dimensions of first design by Martiny

File: ros2/src/shared/march_description/urdf/march4.xacro (robot description, xacro)
@@ -695,6 +695,6 @@
     <xacro:sensor_d435 parent="hip_base">
 <!--    Attached to the hip_base, since this is most comparable to the backpack -->
-<!--    in amount of movement-->
-        <origin xyz="-0.15 0.18 0.18" rpy="${0.5 * pi} ${0.25 * pi} ${pi}"/>
+<!--    in amount of movement, the distance from hip base is based on first design.-->
+        <origin xyz="-0.17 0.195 0.215" rpy="${0.5 * pi} ${0.25 * pi} ${pi}"/>
         <!-- Rotate to be vertical and pointing down 45 degrees -->
     </xacro:sensor_d435>

File: ros2/src/shared/march_description/urdf/march4_with_koen_lengths.xacro (robot description, xacro)
@@ -647,6 +647,6 @@
     <xacro:sensor_d435 parent="hip_base">
         <!--    Attached to the hip_base, since this is most comparable to the backpack -->
-        <!--    in amount of movement-->
-        <origin xyz="-0.15 0.18 0.18" rpy="${0.5 * pi} ${0.25 * pi} ${pi}"/>
+        <!--    in amount of movement, the distance from hip base is based on first design.-->
+        <origin xyz="-0.17 0.195 0.215" rpy="${0.5 * pi} ${0.25 * pi} ${pi}"/>
         <!-- Rotate to be vertical and pointing down 45 degrees -->
     </xacro:sensor_d435>

Commit message: Fix pointer problems to stop random shutting down

File: ros2/src/shared/march_description/urdf/march4.xacro (robot description, xacro)
@@ -7,4 +7,5 @@
     the hover_height to 0.0. Set ground_gait to true to ground gait in simulation.-->
     <xacro:arg name="ground_gait" default="false"/>
+    <xacro:property name="ground_gait" value="$(arg ground_gait)"/>
 <!--    Switch between using the physical camera and the simulation camera -->
 <!--    If set to 'true', no physical camera is needed -->

Commit message: Clean up code

File: ros2/src/shared/march_description/urdf/march4.xacro (robot description, xacro)
@@ -7,5 +7,4 @@
     the hover_height to 0.0. Set ground_gait to true to ground gait in simulation.-->
     <xacro:arg name="ground_gait" default="false"/>
-    <xacro:property name="ground_gait" value="$(arg ground_gait)"/>
 <!--    Switch between using the physical camera and the simulation camera -->
 <!--    If set to 'true', no physical camera is needed -->

Commit message: First attempt to add dual camera

File: ros2/src/shared/march_description/urdf/march4.xacro (robot description, xacro)
@@ -700,8 +700,16 @@
     </joint>
     <xacro:include filename="camera/_d435.urdf.xacro" />
-    <xacro:sensor_d435 parent="hip_base" plugin="$(arg realsense_simulation)">
+    <xacro:sensor_d435 name="camera_front" parent="hip_base"
+                       plugin="$(arg realsense_simulation)">
 <!--    Attached to the hip_base, since this is most comparable to the backpack -->
 <!--    in amount of movement, the distance from hip base is based on first design.-->
         <origin xyz="-0.17 0.195 0.215" rpy="${0.5 * pi} ${0.25 * pi} ${pi}"/>
+        <!-- Rotate to be vertical and pointing down 45 degrees -->
+    </xacro:sensor_d435>
+    <xacro:sensor_d435 name="camera_back" parent="hip_base"
+                       plugin="$(arg realsense_simulation)">
+        <!--    Attached to the hip_base, since this is most comparable to the backpack -->
+        <!--    in amount of movement, the distance from hip base is based on first design.-->
+        <origin xyz="0 0 0" rpy="0 0 0"/>
         <!-- Rotate to be vertical and pointing down 45 degrees -->
     </xacro:sensor_d435>

Commit message: Update mar robot state publisher

File: ros2/src/shared/march_description/urdf/march4.xacro (robot description, xacro)
@@ -709,5 +709,5 @@
     <xacro:sensor_d435 name="camera_back" parent="hip_base"
                        plugin="$(arg realsense_simulation)">
-        <origin xyz="0 0 0" rpy="0 0 0"/>
+        <origin xyz="0 22 0" rpy="0 0 ${0.5 * pi}"/>
     </xacro:sensor_d435>
     <!-- ROS Control plugin for Gazebo -->

Commit message: Fix rotation of back camera

File: ros2/src/shared/march_description/urdf/march4.xacro (robot description, xacro)
@@ -700,5 +700,5 @@
     </joint>
     <xacro:include filename="camera/_d435.urdf.xacro" />
-    <xacro:sensor_d435 name="camera_front" parent="hip_base"
+    <xacro:sensor_d435 name="camera_front" topics_ns="camera_front" parent="hip_base"
                        plugin="$(arg realsense_simulation)">
 <!--    Attached to the hip_base, since this is most comparable to the backpack -->
@@ -707,7 +707,7 @@
         <!-- Rotate to be vertical and pointing down 45 degrees -->
     </xacro:sensor_d435>
-    <xacro:sensor_d435 name="camera_back" parent="hip_base"
+    <xacro:sensor_d435 name="camera_back" topics_ns="camera_back" parent="hip_base"
                        plugin="$(arg realsense_simulation)">
-        <origin xyz="0 22 0" rpy="0 0 ${0.5 * pi}"/>
+        <origin xyz="0 0.22 0" rpy="0 ${0.3 * pi} 0"/>
     </xacro:sensor_d435>
     <!-- ROS Control plugin for Gazebo -->

Commit message: Fix safety controller problem

File: ros2/src/shared/march_description/urdf/march4.xacro (robot description, xacro)
@@ -7,10 +7,10 @@
     the hover_height to 0.0. Set ground_gait to true to ground gait in simulation.-->
     <xacro:arg name="ground_gait" default="false"/>
-<!--    Switch between using the physical camera and the simulation camera -->
-<!--    If set to 'true', no physical camera is needed -->
-<!--    If this value is set to 'false', the plugin will not be started and the topics -->
-<!--    published by the real camera will be used. -->
-<!--    In both these situations the camera will still be visible and placed in the urdf,-->
-<!--    to be used for the transformations.-->
+    <!--    Switch between using the physical camera and the simulation camera -->
+    <!--    If set to 'true', no physical camera is needed -->
+    <!--    If this value is set to 'false', the plugin will not be started and the topics -->
+    <!--    published by the real camera will be used. -->
+    <!--    In both these situations the camera will still be visible and placed in the urdf,-->
+    <!--    to be used for the transformations.-->
     <xacro:arg name="realsense_simulation" default="false"/>
     <xacro:unless value="$(arg ground_gait)">
@@ -27,17 +27,20 @@
     <xacro:arg name="configuration" default="exoskeleton"/>
     <xacro:property name="configuration" value="$(arg configuration)"/>
-<!-- Include all macro files    -->
-    <xacro:include filename="macros/safety_limits.xacro" />
+    <!-- Include all macro files    -->
+    <xacro:include filename="macros/safety_limits.xacro"/>
     <xacro:include filename="macros/pressure_sole.xacro"/>
     <xacro:include filename="macros/frame_part.xacro"/>
     <xacro:include filename="macros/joint.xacro"/>
-<!-- Add yaml files with properties -->
-    <xacro:property name="joint_limits_yaml_file" value="properties/march4_joint_limits.yaml"/>
+    <!-- Add yaml files with properties -->
+    <xacro:property name="joint_limits_yaml_file"
+                    value="properties/march4_joint_limits.yaml"/>
     <xacro:property name="joint_limits" value="${load_yaml(joint_limits_yaml_file)}"/>
-    <xacro:property name="safety_yaml_file" value="properties/march4_safety_${configuration}.yaml"/>
+    <xacro:property name="safety_yaml_file"
+                    value="properties/march4_safety_${configuration}.yaml"/>
     <xacro:property name="safety_values" value="${load_yaml(safety_yaml_file)}"/>
     <xacro:property name="inertia_yaml_file" value="properties/march4_inertia.yaml"/>
     <xacro:property name="inertia" value="${load_yaml(inertia_yaml_file)}"/>
-    <xacro:property name="dimensions_yaml_file" value="properties/march4_dimensions.yaml"/>
+    <xacro:property name="dimensions_yaml_file"
+                    value="properties/march4_dimensions.yaml"/>
     <xacro:property name="dimensions" value="${load_yaml(dimensions_yaml_file)}"/>
     <xacro:property name="rotary_reduction" value="101"/>
@@ -45,5 +48,6 @@
     <!-- Constants for robot dimensions -->
     <!-- Masses determined in Catia, see https://confluence.projectmarch.nl:8443/display/51/URDF+description -->
-    <xacro:property name="width" value="0.05"/> <!-- Square dimensions (widthxwidth) of beams -->
+    <xacro:property name="width"
+                    value="0.05"/> <!-- Square dimensions (widthxwidth) of beams -->
     <xacro:property name="hip_base_height" value="0.160"/>
     <xacro:property name="hip_base_mass" value="8.686"/>
@@ -81,5 +85,6 @@
     <xacro:property name="hip_base_com_z" value="0.147761"/>
     <xacro:property name="hip_aa_com_x" value="${-hip_aa_frame_width + 0.108094}"/>
-    <xacro:property name="hip_aa_com_y" value="${-hip_base_height/2 - hip_aa_frame_height + 0.197758}"/>
+    <xacro:property name="hip_aa_com_y"
+                    value="${-hip_base_height/2 - hip_aa_frame_height + 0.197758}"/>
     <xacro:property name="hip_aa_com_z" value="0.029507"/>
     <xacro:property name="upper_leg_com_x" value="0.000709"/>
@@ -94,5 +99,6 @@
     <xacro:property name="foot_com_y" value="${-hip_base_height/2 - hip_aa_frame_height +
                                                upper_leg_offset + ankle_plate_offset + 0.155916}"/>
-    <xacro:property name="foot_com_z" value="${upper_leg_height + lower_leg_height + ankle_plate_height - 0.789788}"/>
+    <xacro:property name="foot_com_z"
+                    value="${upper_leg_height + lower_leg_height + ankle_plate_height - 0.789788}"/>
     <xacro:property name="foot_scale" value="1.35"/>
     <!-- Import all Gazebo-customization elements, including Gazebo colors -->
@@ -135,5 +141,5 @@
                       mass="${hip_aa_mass}"
                       inertia="${inertia['hip_aa']}"
-                      />
+    />
     <xacro:frame_part name="upper_leg_left"
                       reflect="-1"
@@ -146,5 +152,5 @@
                       mass="${upper_leg_mass}"
                       inertia="${inertia['upper_leg']}"
-                    />
+    />
     <xacro:frame_part name="lower_leg_left"
                       reflect="-1"
@@ -157,5 +163,5 @@
                       mass="${lower_leg_mass}"
                       inertia="${inertia['lower_leg']}"
-                      />
+    />
     <xacro:frame_part name="ankle_plate_left"
                       reflect="-1"
@@ -261,12 +267,12 @@
     </joint>
     <xacro:march_joint
-        name="left_hip_aa"
-        parent="hip_base"
-        child="hip_aa_frame_left_side"
-        origin="0 ${-hip_base_height/2} 0"
-        axis="-1 0 0"
-        safety="${safety_values['haa']}"
-        limits="${joint_limits['left_haa']}"
-        reduction="${linear_reduction}"
+            name="left_hip_aa"
+            parent="hip_base"
+            child="hip_aa_frame_left_side"
+            origin="0 ${-hip_base_height/2} 0"
+            axis="-1 0 0"
+            safety="${safety_values['haa']}"
+            limits="${joint_limits['left_haa']}"
+            reduction="${linear_reduction}"
     />
     <joint name="left_hip_angle" type="fixed">
@@ -276,32 +282,32 @@
     </joint>
     <xacro:march_joint
-        name="left_hip_fe"
-        parent="hip_aa_frame_left_front"
-        child="upper_leg_left"
-        axis="0 1 0"
-        safety="${safety_values['hfe']}"
-        origin="${-hip_aa_frame_width} ${upper_leg_offset} 0"
-        reduction="${rotary_reduction}"
-        limits="${joint_limits['left_hfe']}"
-        />
-    <xacro:march_joint
-        name="left_knee"
-        parent="upper_leg_left"
-        child="lower_leg_left"
-        safety="${safety_values['knee']}"
-        origin="0 0 ${-upper_leg_height}"
-        axis="0 -1 0"
-        reduction="${rotary_reduction}"
-        limits="${joint_limits['left_knee']}"
-    />
-    <xacro:march_joint
-        name="left_ankle"
-        parent="lower_leg_left"
-        child="ankle_plate_left"
-        safety="${safety_values['ankle']}"
-        origin="0 ${ankle_plate_offset} ${-lower_leg_height}"
-        axis="0 1 0"
-        reduction="${linear_reduction}"
-        limits="${joint_limits['left_ankle']}"
+            name="left_hip_fe"
+            parent="hip_aa_frame_left_front"
+            child="upper_leg_left"
+            axis="0 1 0"
+            safety="${safety_values['hfe']}"
+            origin="${-hip_aa_frame_width} ${upper_leg_offset} 0"
+            reduction="${rotary_reduction}"
+            limits="${joint_limits['left_hfe']}"
+    />
+    <xacro:march_joint
+            name="left_knee"
+            parent="upper_leg_left"
+            child="lower_leg_left"
+            safety="${safety_values['knee']}"
+            origin="0 0 ${-upper_leg_height}"
+            axis="0 -1 0"
+            reduction="${rotary_reduction}"
+            limits="${joint_limits['left_knee']}"
+    />
+    <xacro:march_joint
+            name="left_ankle"
+            parent="lower_leg_left"
+            child="ankle_plate_left"
+            safety="${safety_values['ankle']}"
+            origin="0 ${ankle_plate_offset} ${-lower_leg_height}"
+            axis="0 1 0"
+            reduction="${linear_reduction}"
+            limits="${joint_limits['left_ankle']}"
     />
     <joint name="left_foot_angle" type="fixed">
@@ -311,12 +317,12 @@
     </joint>
     <xacro:march_joint
-        name="right_hip_aa"
-        parent="hip_base"
-        child="hip_aa_frame_right_side"
-        origin="0 ${hip_base_height/2} 0"
-        axis="1 0 0"
-        safety="${safety_values['haa']}"
-        reduction="${linear_reduction}"
-        limits="${joint_limits['right_haa']}"
+            name="right_hip_aa"
+            parent="hip_base"
+            child="hip_aa_frame_right_side"
+            origin="0 ${hip_base_height/2} 0"
+            axis="1 0 0"
+            safety="${safety_values['haa']}"
+            reduction="${linear_reduction}"
+            limits="${joint_limits['right_haa']}"
     />
     <joint name="right_hip_angle" type="fixed">
@@ -326,32 +332,32 @@
     </joint>
     <xacro:march_joint
-        name="right_hip_fe"
-        parent="hip_aa_frame_right_front"
-        child="upper_leg_right"
-        origin="${-hip_aa_frame_width} ${-upper_leg_offset} 0"
-        axis="0 1 0"
-        safety="${safety_values['hfe']}"
-        reduction="${rotary_reduction}"
-        limits="${joint_limits['right_hfe']}"
-    />
-    <xacro:march_joint
-        name="right_knee"
-        parent="upper_leg_right"
-        child="lower_leg_right"
-        origin="0 0 ${-upper_leg_height}"
-        axis="0 -1 0"
-        safety="${safety_values['knee']}"
-        limits="${joint_limits['right_knee']}"
-        reduction="${rotary_reduction}"
-    />
-    <xacro:march_joint
-        name="right_ankle"
-        parent="lower_leg_right"
-        child="ankle_plate_right"
-        safety="${safety_values['ankle']}"
-        origin="0 ${-ankle_plate_offset} ${-lower_leg_height}"
-        axis="0 1 0"
-        reduction="${linear_reduction}"
-        limits="${joint_limits['left_ankle']}"
+            name="right_hip_fe"
+            parent="hip_aa_frame_right_front"
+            child="upper_leg_right"
+            origin="${-hip_aa_frame_width} ${-upper_leg_offset} 0"
+            axis="0 1 0"
+            safety="${safety_values['hfe']}"
+            reduction="${rotary_reduction}"
+            limits="${joint_limits['right_hfe']}"
+    />
+    <xacro:march_joint
+            name="right_knee"
+            parent="upper_leg_right"
+            child="lower_leg_right"
+            origin="0 0 ${-upper_leg_height}"
+            axis="0 -1 0"
+            safety="${safety_values['knee']}"
+            limits="${joint_limits['right_knee']}"
+            reduction="${rotary_reduction}"
+    />
+    <xacro:march_joint
+            name="right_ankle"
+            parent="lower_leg_right"
+            child="ankle_plate_right"
+            safety="${safety_values['ankle']}"
+            origin="0 ${-ankle_plate_offset} ${-lower_leg_height}"
+            axis="0 1 0"
+            reduction="${linear_reduction}"
+            limits="${joint_limits['left_ankle']}"
     />
     <joint name="right_foot_angle" type="fixed">
@@ -360,11 +366,15 @@
         <origin xyz="0 0 ${-ankle_plate_height}" rpy="0 0 0"/>
     </joint>
-    <xacro:include filename="camera/_d435.urdf.xacro" />
+    <xacro:include filename="camera/_d435.urdf.xacro"/>
     <xacro:sensor_d435 name="camera_front" topics_ns="camera_front" parent="hip_base"
                        plugin="$(arg realsense_simulation)">
-<!--    Attached to the hip_base, since this is most comparable to the backpack -->
-<!--    in amount of movement, the distance from hip base is based on first design.-->
+        <!--    Attached to the hip_base, since this is most comparable to the backpack -->
+        <!--    in amount of movement, the distance from hip base is based on first design.-->
         <origin xyz="-0.17 0.195 0.215" rpy="${0.5 * pi} ${0.25 * pi} ${pi}"/>
         <!-- Rotate to be vertical and pointing down 45 degrees -->
     </xacro:sensor_d435>
+    <xacro:sensor_d435 name="camera_back" topics_ns="camera_back" parent="hip_base"
+                       plugin="$(arg realsense_simulation)">
+        <origin xyz="0 0.22 0" rpy="0 ${0.3 * pi} 0"/>
+    </xacro:sensor_d435>
 </robot>

Commit message: Change to use 1 yaml file

File: ros2/src/shared/march_description/urdf/march4.xacro (robot description, xacro)
@@ -33,15 +33,12 @@
     <xacro:include filename="macros/joint.xacro"/>
     <!-- Add yaml files with properties -->
-    <xacro:property name="joint_limits_yaml_file"
-                    value="properties/march4_joint_limits.yaml"/>
-    <xacro:property name="joint_limits" value="${load_yaml(joint_limits_yaml_file)}"/>
-    <xacro:property name="safety_yaml_file"
-                    value="properties/march4_safety_${configuration}.yaml"/>
-    <xacro:property name="safety_values" value="${load_yaml(safety_yaml_file)}"/>
-    <xacro:property name="inertia_yaml_file" value="properties/march4_inertia.yaml"/>
-    <xacro:property name="inertia" value="${load_yaml(inertia_yaml_file)}"/>
-    <xacro:property name="dimensions_yaml_file"
-                    value="properties/march4_dimensions.yaml"/>
-    <xacro:property name="dimensions" value="${load_yaml(dimensions_yaml_file)}"/>
+    <xacro:property name="config_yaml_file"
+                    value="properties/march4.yaml"/>
+    <xacro:property name="properties" value="${load_yaml(config_yaml_file)}"/>
+    <xacro:property name="joint_limits" value="${properties['joint_limits']}"/>
+    <xacro:property name="safety_values"
+                    value="${properties['safety'][configuration]}"/>
+    <xacro:property name="inertia" value="${properties['inertia']}"/>
+    <xacro:property name="dimensions" value="${properties['dimensions']}"/>
     <xacro:property name="rotary_reduction" value="101"/>
     <xacro:property name="linear_reduction" value="200"/>

Commit message: Add pressure sole heel

File: ros2/src/shared/march_description/urdf/march4.xacro (robot description, xacro)
@@ -186,6 +186,9 @@
         <fdir1>1 0 0</fdir1>
     </gazebo>
-    <xacro:pressure_sole foot_place="left_hallux" foot_name="foot_left">
-        <origin xyz="${(-foot_height_forward+foot_height_backward)/8} ${width/2} 0" rpy="0 0 0"/>
+    <xacro:pressure_sole foot_place="left_heel_1" foot_name="foot_left">
+        <origin xyz="${(-foot_height_forward+foot_height_backward)/8} ${width/4} 0" rpy="0 0 0"/>
+    </xacro:pressure_sole>
+    <xacro:pressure_sole foot_place="left_heel_2" foot_name="foot_left">
+        <origin xyz="${(-foot_height_forward+foot_height_backward)/8} ${-width/4} 0" rpy="0 0 0"/>
     </xacro:pressure_sole>
     <xacro:frame_part name="hip_aa_frame_right_side"
@@ -240,6 +243,9 @@
     />
     <!-- Foot Right -->
-    <xacro:pressure_sole foot_place="right_toe" foot_name="foot_right">
-        <origin xyz="${(-foot_height_forward+foot_height_backward)/2} 0 0" rpy="0 0 0"/>
+    <xacro:pressure_sole foot_place="right_heel_1" foot_name="foot_right">
+        <origin xyz="${(-foot_height_forward+foot_height_backward)/8} ${width/4} 0" rpy="0 0 0"/>
+    </xacro:pressure_sole>
+    <xacro:pressure_sole foot_place="right_heel_2" foot_name="foot_right">
+        <origin xyz="${(-foot_height_forward+foot_height_backward)/8} ${-width/4} 0" rpy="0 0 0"/>
     </xacro:pressure_sole>
     <xacro:frame_part name="foot_right"

Commit message: Beunfixes

File: ros2/src/shared/march_description/urdf/march4.xacro (robot description, xacro)
@@ -15,5 +15,5 @@
     <xacro:arg name="realsense_simulation" default="false"/>
     <xacro:unless value="$(arg ground_gait)">
-        <xacro:property name="parent_name" value="world"/>
+        <xacro:property name="parent_name" value="base_link"/>
         <xacro:property name="hover_height" value="0.3"/>
     </xacro:unless>
@@ -117,5 +117,5 @@
     </material>
     <!-- Used for fixing robot to Gazebo 'base_link' -->
-    <link name="${parent_name}"/>
+<!--    <link name="${parent_name}"/>-->
     <!-- Parts -->
     <!-- Hip-->
@@ -132,5 +132,5 @@
     />
     <!-- IMU-->
-    <link name="imu_link">
+    <link name="base_link">
     </link>
     <xacro:frame_part name="hip_aa_frame_left_side"
@@ -254,12 +254,12 @@
                       mass="${foot_mass}"/>
     <!-- Joints -->
-    <joint name="imu_joint" type="fixed">
-        <parent link="${parent_name}"/>
-        <child link="imu_link"/>
-    </joint>
+<!--    <joint name="imu_joint" type="fixed">-->
+<!--        <parent link="${parent_name}"/>-->
+<!--        <child link="imu_link"/>-->
+<!--    </joint>-->
     <joint name="hip" type="fixed">
-        <parent link="imu_link"/>
+        <parent link="base_link"/>
         <child link="hip_base"/>
-        <origin xyz="0 0 ${lower_leg_height+upper_leg_height+ankle_plate_height+width/2.0+hover_height}" rpy="0 0 0"/>
+        <origin xyz="0 0 0" rpy="0 0 0"/>
     </joint>
     <xacro:march_joint

Commit message: March4.xacro camera loc update

File: ros2/src/shared/march_description/urdf/march4.xacro (robot description, xacro)
@@ -368,5 +368,5 @@
         <!--    Attached to the hip_base, since this is most comparable to the backpack -->
         <!--    in amount of movement, the distance from hip base is based on first design.-->
-        <origin xyz="-0.17 0.195 0.215" rpy="${0.5 * pi} ${0.25 * pi} ${pi}"/>
+        <origin xyz="-0.15 0.18 0.10" rpy="${0.5 * pi} ${0.25 * pi} ${pi}"/>
         <!-- Rotate to be vertical and pointing down 45 degrees -->
     </xacro:sensor_d435>
