Commit message: Turn off safety controller for rotational joint

File: ros2/src/shared/march_description/urdf/test_joint_rotational.xacro (robot description, xacro)
@@ -8,7 +8,10 @@
     <xacro:property name="bar_mass" value="1.080"/>
     <xacro:property name="bar_width" value="0.05"/>
-    <xacro:property name="joint_buffer" value="${3*pi/180}"/> <!-- rad -->
-    <xacro:property name="joint_lower_limit" value="-0.5363"/> <!-- rad -->
-    <xacro:property name="joint_upper_limit" value="0.5363"/> <!-- rad -->
+    <!--<xacro:property name="joint_buffer" value="${3*pi/180}"/> --><!-- rad -->
+    <xacro:property name="joint_buffer" value="0"/> <!-- rad -->
+    <!--<xacro:property name="joint_lower_limit" value="-0.5363"/> --> <!-- rad -->
+    <xacro:property name="joint_lower_limit" value="${-pi}"/> <!-- rad -->
+    <xacro:property name="joint_upper_limit" value="${pi}"/> <!-- rad -->
+    <!-- <xacro:property name="joint_upper_limit" value="0.5363"/> --> <!-- rad -->
     <xacro:property name="joint_effort_limit" value="21840"/> <!-- IU = 20 A -->
     <xacro:property name="joint_velocity_limit" value="2.0"/> <!-- rad/s -->
@@ -28,5 +31,5 @@
         <axis xyz="0 1 0"/>
         <limit velocity="${joint_velocity_limit}" effort="${joint_effort_limit}" lower="${joint_lower_limit}" upper="${joint_upper_limit}"/>
-        <safety_controller soft_lower_limit="${joint_lower_limit + joint_buffer}" soft_upper_limit="${joint_upper_limit - joint_buffer}" k_position="5" k_velocity="20000" />
+        <!-- <safety_controller soft_lower_limit="${joint_lower_limit + joint_buffer}" soft_upper_limit="${joint_upper_limit - joint_buffer}" k_position="5" k_velocity="20000" /> -->
     </joint>
     <!-- give colors to some links in gazebo -->

Commit message: Restoring xacro file and adding some last finishing touches

File: ros2/src/shared/march_description/urdf/test_joint_rotational.xacro (robot description, xacro)
@@ -5,13 +5,10 @@
     <xacro:property name="joint_base_mass" value="1"/> <!-- arbitrary value for joint_base_mass -->
     <xacro:property name="joint_base_width" value="0.05"/> <!-- Cube dimensions (width x width x width) of joint base -->
-    <xacro:property name="bar_length" value="${0.39}"/>
+    <xacro:property name="bar_length" value="0.39"/>
     <xacro:property name="bar_mass" value="1.080"/>
     <xacro:property name="bar_width" value="0.05"/>
-    <!--<xacro:property name="joint_buffer" value="${3*pi/180}"/> --><!-- rad -->
-    <xacro:property name="joint_buffer" value="0"/> <!-- rad -->
-    <!--<xacro:property name="joint_lower_limit" value="-0.5363"/> --> <!-- rad -->
-    <xacro:property name="joint_lower_limit" value="${-pi}"/> <!-- rad -->
-    <xacro:property name="joint_upper_limit" value="${pi}"/> <!-- rad -->
-    <!-- <xacro:property name="joint_upper_limit" value="0.5363"/> --> <!-- rad -->
+    <xacro:property name="joint_buffer" value="${3*(pi/180)}"/> <!-- rad -->
+    <xacro:property name="joint_lower_limit" value="-0.5363"/> <!-- rad -->
+    <xacro:property name="joint_upper_limit" value="0.5363"/> <!-- rad -->
     <xacro:property name="joint_effort_limit" value="21840"/> <!-- IU = 20 A -->
     <xacro:property name="joint_velocity_limit" value="2.0"/> <!-- rad/s -->
@@ -31,5 +28,5 @@
         <axis xyz="0 1 0"/>
         <limit velocity="${joint_velocity_limit}" effort="${joint_effort_limit}" lower="${joint_lower_limit}" upper="${joint_upper_limit}"/>
-        <!-- <safety_controller soft_lower_limit="${joint_lower_limit + joint_buffer}" soft_upper_limit="${joint_upper_limit - joint_buffer}" k_position="5" k_velocity="20000" /> -->
+        <safety_controller soft_lower_limit="${joint_lower_limit + joint_buffer}" soft_upper_limit="${joint_upper_limit - joint_buffer}" k_position="5" k_velocity="20000" />
     </joint>
     <!-- give colors to some links in gazebo -->

Commit message: WIP reference system

File: ros2/src/shared/march_description/urdf/test_joint_rotational.xacro (robot description, xacro)
@@ -9,6 +9,6 @@
     <xacro:property name="bar_width" value="0.05"/>
     <xacro:property name="joint_buffer" value="${3*(pi/180)}"/> <!-- rad -->
-    <xacro:property name="joint_lower_limit" value="-0.5363"/> <!-- rad -->
-    <xacro:property name="joint_upper_limit" value="0.5363"/> <!-- rad -->
+    <xacro:property name="joint_lower_limit" value="${-pi}"/> <!-- rad -->
+    <xacro:property name="joint_upper_limit" value="${pi}"/> <!-- rad -->
     <xacro:property name="joint_effort_limit" value="21840"/> <!-- IU = 20 A -->
     <xacro:property name="joint_velocity_limit" value="2.0"/> <!-- rad/s -->
@@ -28,5 +28,5 @@
         <axis xyz="0 1 0"/>
         <limit velocity="${joint_velocity_limit}" effort="${joint_effort_limit}" lower="${joint_lower_limit}" upper="${joint_upper_limit}"/>
-<!--        <safety_controller soft_lower_limit="${joint_lower_limit + joint_buffer}" soft_upper_limit="${joint_upper_limit - joint_buffer}" k_position="5" k_velocity="20000" />-->
+        <safety_controller soft_lower_limit="${joint_lower_limit + joint_buffer}" soft_upper_limit="${joint_upper_limit - joint_buffer}" k_position="0" k_velocity="0" />
     </joint>
     <!-- give colors to some links in gazebo -->

Commit message: WIP reference system

File: ros2/src/shared/march_description/urdf/test_joint_rotational.xacro (robot description, xacro)
@@ -9,6 +9,6 @@
     <xacro:property name="bar_width" value="0.05"/>
     <xacro:property name="joint_buffer" value="${3*(pi/180)}"/> <!-- rad -->
-    <xacro:property name="joint_lower_limit" value="-0.5363"/> <!-- rad -->
-    <xacro:property name="joint_upper_limit" value="0.5363"/> <!-- rad -->
+    <xacro:property name="joint_lower_limit" value="${-pi}"/> <!-- rad -->
+    <xacro:property name="joint_upper_limit" value="${pi}"/> <!-- rad -->
     <xacro:property name="joint_effort_limit" value="21840"/> <!-- IU = 20 A -->
     <xacro:property name="joint_velocity_limit" value="2.0"/> <!-- rad/s -->

Commit message: Creating MPC test branch

File: ros2/src/shared/march_description/urdf/test_joint_rotational.xacro (robot description, xacro)
@@ -9,6 +9,6 @@
     <xacro:property name="bar_width" value="0.05"/>
     <xacro:property name="joint_buffer" value="${3*(pi/180)}"/> <!-- rad -->
-    <xacro:property name="joint_lower_limit" value="-0.5363"/> <!-- rad -->
-    <xacro:property name="joint_upper_limit" value="0.5363"/> <!-- rad -->
+    <xacro:property name="joint_lower_limit" value="${-pi}"/> <!-- rad -->
+    <xacro:property name="joint_upper_limit" value="${pi}"/> <!-- rad -->
     <xacro:property name="joint_effort_limit" value="21840"/> <!-- IU = 20 A -->
     <xacro:property name="joint_velocity_limit" value="2.0"/> <!-- rad/s -->
@@ -28,5 +28,5 @@
         <axis xyz="0 1 0"/>
         <limit velocity="${joint_velocity_limit}" effort="${joint_effort_limit}" lower="${joint_lower_limit}" upper="${joint_upper_limit}"/>
-        <safety_controller soft_lower_limit="${joint_lower_limit + joint_buffer}" soft_upper_limit="${joint_upper_limit - joint_buffer}" k_position="5" k_velocity="20000" />
+        <safety_controller soft_lower_limit="${joint_lower_limit + joint_buffer}" soft_upper_limit="${joint_upper_limit - joint_buffer}" k_position="1" k_velocity="1" />
     </joint>
     <!-- give colors to some links in gazebo -->

File: ros2/src/shared/march_description/urdf/test_joint_rotational_mpc.xacro (robot description, xacro)
@@ -12,5 +12,5 @@
     <xacro:property name="joint_upper_limit" value="${pi}"/> <!-- rad -->
     <xacro:property name="joint_effort_limit" value="21840"/> <!-- IU = 20 A -->
-    <xacro:property name="joint_velocity_limit" value="20.0"/> <!-- rad/s -->
+    <xacro:property name="joint_velocity_limit" value="2.0"/> <!-- rad/s -->
     <xacro:property name="hover_height" value="0.5"/>
     <xacro:include filename="march.gazebo"/>
@@ -31,5 +31,5 @@
         with the internal workings of the model predictive controller.
         It will be enabled again once a solution has been found -->
-        <!-- <safety_controller soft_lower_limit="${joint_lower_limit + joint_buffer}" soft_upper_limit="${joint_upper_limit - joint_buffer}" k_position="5" k_velocity="20000" /> -->
+         <safety_controller soft_lower_limit="${joint_lower_limit + joint_buffer}" soft_upper_limit="${joint_upper_limit - joint_buffer}" k_position="1" k_velocity="1" />
     </joint>
     <!-- give colors to some links in gazebo -->

Commit message: MPC Tweaks

File: ros2/src/shared/march_description/urdf/test_joint_rotational.xacro (robot description, xacro)
@@ -12,5 +12,5 @@
     <xacro:property name="joint_upper_limit" value="${pi}"/> <!-- rad -->
     <xacro:property name="joint_effort_limit" value="21840"/> <!-- IU = 20 A -->
-    <xacro:property name="joint_velocity_limit" value="2.0"/> <!-- rad/s -->
+    <xacro:property name="joint_velocity_limit" value="20.0"/> <!-- rad/s -->
     <xacro:property name="hover_height" value="0.5"/>
     <xacro:include filename="march.gazebo"/>
@@ -28,5 +28,5 @@
         <axis xyz="0 1 0"/>
         <limit velocity="${joint_velocity_limit}" effort="${joint_effort_limit}" lower="${joint_lower_limit}" upper="${joint_upper_limit}"/>
-        <safety_controller soft_lower_limit="${joint_lower_limit + joint_buffer}" soft_upper_limit="${joint_upper_limit - joint_buffer}" k_position="1" k_velocity="1" />
+        <safety_controller soft_lower_limit="${joint_lower_limit + joint_buffer}" soft_upper_limit="${joint_upper_limit - joint_buffer}" k_position="5" k_velocity="20000" />
     </joint>
     <!-- give colors to some links in gazebo -->

Commit message: Changes made during testing 02022021

File: ros2/src/shared/march_description/urdf/test_joint_rotational.xacro (robot description, xacro)
@@ -11,6 +11,6 @@
     <xacro:property name="joint_lower_limit" value="-0.5363"/> <!-- rad -->
     <xacro:property name="joint_upper_limit" value="0.5363"/> <!-- rad -->
-    <xacro:property name="joint_effort_limit" value="21840"/> <!-- IU = 20 A -->
-    <xacro:property name="joint_velocity_limit" value="2.0"/> <!-- rad/s -->
+    <xacro:property name="joint_effort_limit" value="218400"/> <!-- IU = 20 A -->
+    <xacro:property name="joint_velocity_limit" value="20.0"/> <!-- rad/s -->
     <xacro:property name="hover_height" value="0.5"/>
     <xacro:include filename="march.gazebo"/>

Commit message: Reverting joint limits to old values

File: ros2/src/shared/march_description/urdf/test_joint_rotational.xacro (robot description, xacro)
@@ -9,6 +9,6 @@
     <xacro:property name="bar_width" value="0.05"/>
     <xacro:property name="joint_buffer" value="${3*(pi/180)}"/> <!-- rad -->
-    <xacro:property name="joint_lower_limit" value="${-pi}"/> <!-- rad -->
-    <xacro:property name="joint_upper_limit" value="${pi}"/> <!-- rad -->
+    <xacro:property name="joint_lower_limit" value="-0.5363"/> <!-- rad -->
+    <xacro:property name="joint_upper_limit" value="0.5363"/> <!-- rad -->
     <xacro:property name="joint_effort_limit" value="21840"/> <!-- IU = 20 A -->
     <xacro:property name="joint_velocity_limit" value="2.0"/> <!-- rad/s -->

Commit message: Reverting joint limits to old values

File: ros2/src/shared/march_description/urdf/test_joint_rotational.xacro (robot description, xacro)
@@ -9,6 +9,6 @@
     <xacro:property name="bar_width" value="0.05"/>
     <xacro:property name="joint_buffer" value="${3*(pi/180)}"/> <!-- rad -->
-    <xacro:property name="joint_lower_limit" value="${-pi}"/> <!-- rad -->
-    <xacro:property name="joint_upper_limit" value="${pi}"/> <!-- rad -->
+    <xacro:property name="joint_lower_limit" value="-0.5363"/> <!-- rad -->
+    <xacro:property name="joint_upper_limit" value="0.5363"/> <!-- rad -->
     <xacro:property name="joint_effort_limit" value="21840"/> <!-- IU = 20 A -->
     <xacro:property name="joint_velocity_limit" value="2.0"/> <!-- rad/s -->

File: ros2/src/shared/march_description/urdf/test_joint_rotational_mpc.xacro (robot description, xacro)
@@ -9,6 +9,6 @@
     <xacro:property name="bar_width" value="0.05"/>
     <xacro:property name="joint_buffer" value="${3*(pi/180)}"/> <!-- rad -->
-    <xacro:property name="joint_lower_limit" value="${-pi}"/> <!-- rad -->
-    <xacro:property name="joint_upper_limit" value="${pi}"/> <!-- rad -->
+    <xacro:property name="joint_lower_limit" value="-0.5363"/> <!-- rad -->
+    <xacro:property name="joint_upper_limit" value="0.5363"/> <!-- rad -->
     <xacro:property name="joint_effort_limit" value="21840"/> <!-- IU = 20 A -->
     <xacro:property name="joint_velocity_limit" value="20.0"/> <!-- rad/s -->

Commit message: Adjusting test_joint_rotational.xacro joint limits and turning off safety_controller

File: ros2/src/shared/march_description/urdf/test_joint_rotational.xacro (robot description, xacro)
@@ -9,8 +9,8 @@
     <xacro:property name="bar_width" value="0.05"/>
     <xacro:property name="joint_buffer" value="${3*(pi/180)}"/> <!-- rad -->
-    <xacro:property name="joint_lower_limit" value="-0.5363"/> <!-- rad -->
-    <xacro:property name="joint_upper_limit" value="0.5363"/> <!-- rad -->
-    <xacro:property name="joint_effort_limit" value="21840"/> <!-- IU = 20 A -->
-    <xacro:property name="joint_velocity_limit" value="2.0"/> <!-- rad/s -->
+    <xacro:property name="joint_lower_limit" value="-0.7"/> <!-- rad -->
+    <xacro:property name="joint_upper_limit" value="0.7"/> <!-- rad -->
+    <xacro:property name="joint_effort_limit" value="30"/> <!-- 30 A -->
+    <xacro:property name="joint_velocity_limit" value="3.0"/> <!-- rad/s -->
     <xacro:property name="hover_height" value="0.5"/>
     <xacro:include filename="march.gazebo"/>
@@ -28,5 +28,5 @@
         <axis xyz="0 1 0"/>
         <limit velocity="${joint_velocity_limit}" effort="${joint_effort_limit}" lower="${joint_lower_limit}" upper="${joint_upper_limit}"/>
-        <safety_controller soft_lower_limit="${joint_lower_limit + joint_buffer}" soft_upper_limit="${joint_upper_limit - joint_buffer}" k_position="5" k_velocity="20000" />
+        <safety_controller soft_lower_limit="${joint_lower_limit + joint_buffer}" soft_upper_limit="${joint_upper_limit - joint_buffer}" k_position="20000" k_velocity="20000" />
     </joint>
     <!-- give colors to some links in gazebo -->

Commit message: Changed knee gait to more tranquilo version. fixed typo in controllers yaml file. changed joint limits to allow for gait

File: ros2/src/shared/march_description/urdf/test_joint_rotational.xacro (robot description, xacro)
@@ -9,6 +9,6 @@
     <xacro:property name="bar_width" value="0.05"/>
     <xacro:property name="joint_buffer" value="${3*(pi/180)}"/> <!-- rad -->
-    <xacro:property name="joint_lower_limit" value="-0.7"/> <!-- rad -->
-    <xacro:property name="joint_upper_limit" value="0.7"/> <!-- rad -->
+    <xacro:property name="joint_lower_limit" value="-1.05"/> <!-- rad -->
+    <xacro:property name="joint_upper_limit" value="1.05"/> <!-- rad -->
     <xacro:property name="joint_effort_limit" value="30"/> <!-- 30 A -->
     <xacro:property name="joint_velocity_limit" value="3.0"/> <!-- rad/s -->

Commit message: Add necessary files for using DieBOSlave with test joint

File: ros2/src/shared/march_description/urdf/test_joint_rotational.xacro (robot description, xacro)
@@ -8,11 +8,26 @@
     <xacro:property name="bar_mass" value="1.080"/>
     <xacro:property name="bar_width" value="0.05"/>
-    <xacro:property name="joint_buffer"         value="${3*(pi/180)}"/>     <!-- rad -->
-    <xacro:property name="joint_lower_limit"    value="-0.4395"/>   <!-- rad -->
-    <xacro:property name="joint_upper_limit"    value="1.7857"/>     <!-- rad -->
-    <xacro:property name="joint_effort_limit"   value="20"/>                <!-- IU -->
-    <xacro:property name="joint_velocity_limit" value="3.0"/>               <!-- rad/s -->
     <xacro:property name="hover_height" value="0.5"/>
     <xacro:include filename="march.gazebo"/>
+    <xacro:arg name="configuration" default="exoskeleton"/>
+    <xacro:property name="configuration" value="$(arg configuration)"/>
+    <!-- Include all macro files    -->
+    <xacro:include filename="macros/safety_limits.xacro"/>
+    <xacro:include filename="macros/pressure_sole.xacro"/>
+    <xacro:include filename="macros/frame_part.xacro"/>
+    <xacro:include filename="macros/joint.xacro"/>
+    <xacro:include filename="macros/configurable_joint.xacro"/>
+    <!-- Add yaml files with properties -->
+    <xacro:property name="config_yaml_file"
+                    value="properties/test_joints.yaml"/>
+    <xacro:property name="properties" value="${load_yaml(config_yaml_file)}"/>
+    <xacro:property name="joint_limits" value="${properties['joint_limits']}"/>
+    <xacro:property name="safety_values"
+                    value="${properties['safety'][configuration]}"/>
+    <xacro:property name="inertia" value="${properties['inertia']}"/>
+    <xacro:property name="dimensions" value="${properties['dimensions']}"/>
+    <!-- Harmonic Drive: 101, Belt: 1,2-->
+    <xacro:property name="rotary_reduction" value="${101 * 1.2}"/>
+    <xacro:property name="actuating_joints" value="${(properties['actuating_joints'])}"/>
     <!-- Used for fixing robot to Gazebo 'base_link' -->
     <link name="world"/>
@@ -22,12 +37,14 @@
         <origin xyz="0 0 ${hover_height}" rpy="0 0 0"/>
     </joint>
-    <joint name="rotational_joint" type="revolute">
-        <parent link="joint_base"/>
-        <child link="bar"/>
-        <origin xyz="0 ${-joint_base_width} 0" rpy="0 0 0"/>
-        <axis xyz="0 1 0"/>
-        <limit velocity="${joint_velocity_limit}" effort="${joint_effort_limit}" lower="${joint_lower_limit}" upper="${joint_upper_limit}"/>
-        <safety_controller soft_lower_limit="${joint_lower_limit + joint_buffer}" soft_upper_limit="${joint_upper_limit - joint_buffer}" k_position="20000" k_velocity="20000" />
-    </joint>
+    <xacro:march_configurable_joint
+            name="rotational_joint"
+            parent="joint_base"
+            child="bar"
+            safety="${safety_values['rotational_joint']}"
+            origin="0 ${-joint_base_width} 0"
+            axis="0 1 0"
+            reduction="${rotary_reduction}"
+            limits="${joint_limits['rotational_joint']}"
+    />
     <!-- give colors to some links in gazebo -->
     <gazebo reference="joint_base">
@@ -68,13 +85,3 @@
         </inertial>
     </link>
-    <!-- ROS Control plugin for Gazebo -->
-    <transmission name="rotational_joint_transmission">
-        <type>transmission_interface/SimpleTransmission</type>
-        <joint name="rotational_joint">
-            <hardwareInterface>hardware_interface/EffortJointInterface</hardwareInterface>
-        </joint>
-        <actuator name="rotational_joint_motor">
-            <mechanicalReduction>121</mechanicalReduction>
-        </actuator>
-    </transmission>
 </robot>
