Commit message: Adding required files for actuating linear joint with odrive

File: ros2/src/shared/march_description/urdf/test_joint_linear.xacro (robot description, xacro)
@@ -14,8 +14,8 @@
     <xacro:property name="bar_width" value="0.05"/>
     <xacro:property name="joint_buffer" value="${3*pi/180}"/> <!-- rad -->
-    <xacro:property name="joint_lower_limit" value="${-8.5*pi/180}"/> <!-- rad -->
-    <xacro:property name="joint_upper_limit" value="${8.5*pi/180}"/> <!-- rad -->
+    <xacro:property name="joint_lower_limit" value="${-223*pi/360}"/> <!-- rad -->
+    <xacro:property name="joint_upper_limit" value="${223*pi/360}"/> <!-- rad -->
     <xacro:property name="joint_effort_limit" value="10927.0"/>
-    <xacro:property name="joint_velocity_limit" value="1.0"/> <!-- rad/s -->
+    <xacro:property name="joint_velocity_limit" value="10.0"/> <!-- rad/s -->
     <xacro:property name="hover_height" value="0.5"/>
     <xacro:include filename="march.gazebo"/>
@@ -85,5 +85,5 @@
         <actuator name="linear_joint_motor">
             <hardwareInterface>hardware_interface/EffortJointInterface</hardwareInterface>
-            <mechanicalReduction>1</mechanicalReduction>
+            <mechanicalReduction>223</mechanicalReduction>
         </actuator>
     </transmission>

Commit message: Adding up to date mpc code from main

File: ros2/src/shared/march_description/urdf/test_joint_linear.xacro (robot description, xacro)
@@ -2,8 +2,8 @@
 <!-- Revolute-Revolute Manipulator -->
 <robot name="march" xmlns:xacro="http://www.ros.org/wiki/xacro">
-    <!-- Switch between airgaiting or standing on the ground -->
-    <!-- Value set to 'world' fixes the robot to the world -->
-    <!-- Value set to 'base_link' makes the robot stand on the ground -->
-    <!-- Important note when changing value make sure rviz fixed frame is set to the same value (moveit.rviz) -->
+    <!-- Switch between airgaiting or standing on the ground-->
+    <!--Value set to: 'world' fixes the robot to the world-->
+    <!--Value set to: 'base_link' makes the robot stand on the ground-->
+    <!--Important note: when changing value make sure rviz fixed frame is set to the same value (moveit.rviz)-->
     <!-- Constants for robot dimensions -->
     <xacro:property name="PI" value="3.1415926535897931"/>
@@ -14,8 +14,8 @@
     <xacro:property name="bar_width" value="0.05"/>
     <xacro:property name="joint_buffer" value="${3*pi/180}"/> <!-- rad -->
-    <xacro:property name="joint_lower_limit" value="${-223*pi/360}"/> <!-- rad -->
-    <xacro:property name="joint_upper_limit" value="${223*pi/360}"/> <!-- rad -->
+    <xacro:property name="joint_lower_limit" value="${-8.5*pi/180}"/> <!-- rad -->
+    <xacro:property name="joint_upper_limit" value="${8.5*pi/180}"/> <!-- rad -->
     <xacro:property name="joint_effort_limit" value="10927.0"/>
-    <xacro:property name="joint_velocity_limit" value="10.0"/> <!-- rad/s -->
+    <xacro:property name="joint_velocity_limit" value="1.0"/> <!-- rad/s -->
     <xacro:property name="hover_height" value="0.5"/>
     <xacro:include filename="march.gazebo"/>
@@ -84,5 +84,6 @@
         </joint>
         <actuator name="linear_joint_motor">
-            <mechanicalReduction>3.14159265</mechanicalReduction>
+            <hardwareInterface>hardware_interface/EffortJointInterface</hardwareInterface>
+            <mechanicalReduction>1</mechanicalReduction>
         </actuator>
     </transmission>

Commit message: Linear test joint settings and xacro update

File: ros2/src/shared/march_description/urdf/test_joint_linear.xacro (robot description, xacro)
@@ -13,9 +13,9 @@
     <xacro:property name="bar_mass" value="1.080"/>
     <xacro:property name="bar_width" value="0.05"/>
-    <xacro:property name="joint_buffer" value="${3*pi/180}"/> <!-- rad -->
-    <xacro:property name="joint_lower_limit" value="${-223*pi/360}"/> <!-- rad -->
-    <xacro:property name="joint_upper_limit" value="${223*pi/360}"/> <!-- rad -->
+    <xacro:property name="joint_buffer" value="1"/> <!-- rad -->
+    <xacro:property name="joint_lower_limit" value="-10"/> <!-- rad -->
+    <xacro:property name="joint_upper_limit" value="10"/> <!-- rad -->
     <xacro:property name="joint_effort_limit" value="10927.0"/>
-    <xacro:property name="joint_velocity_limit" value="10.0"/> <!-- rad/s -->
+    <xacro:property name="joint_velocity_limit" value="5.0"/> <!-- rad/s -->
     <xacro:property name="hover_height" value="0.5"/>
     <xacro:include filename="march.gazebo"/>
@@ -30,5 +30,5 @@
         <origin xyz="0 0 ${hover_height}" rpy="0 0 0"/>
     </joint>
-    <joint name="linear_joint" type="revolute">
+    <joint name="linear_joint" type="prismatic">
         <parent link="joint_base"/>
         <child link="bar"/>
@@ -67,5 +67,5 @@
                 <box size="${bar_width} ${bar_width} ${bar_length}"/>
             </geometry>
-        </visual>
+        </visual>pi
         <inertial>
             <origin xyz="0 0 ${-bar_length/2}" rpy="0 0 0"/>

Commit message: Prepare files for running gaits on linear joints

File: ros2/src/shared/march_description/urdf/test_joint_linear.xacro (robot description, xacro)
@@ -14,8 +14,8 @@
     <xacro:property name="bar_width" value="0.05"/>
     <xacro:property name="joint_buffer" value="1"/> <!-- rad -->
-    <xacro:property name="joint_lower_limit" value="-10"/> <!-- rad -->
-    <xacro:property name="joint_upper_limit" value="10"/> <!-- rad -->
-    <xacro:property name="joint_effort_limit" value="10927.0"/>
-    <xacro:property name="joint_velocity_limit" value="5.0"/> <!-- rad/s -->
+    <xacro:property name="joint_lower_limit" value="-20"/> <!-- rad -->
+    <xacro:property name="joint_upper_limit" value="20"/> <!-- rad -->
+    <xacro:property name="joint_effort_limit" value="10"/>
+    <xacro:property name="joint_velocity_limit" value="10.0"/> <!-- rad/s -->
     <xacro:property name="hover_height" value="0.5"/>
     <xacro:include filename="march.gazebo"/>
@@ -36,5 +36,5 @@
         <axis xyz="0 1 0"/>
         <limit velocity="${joint_velocity_limit}" effort="${joint_effort_limit}" lower="${joint_lower_limit}" upper="${joint_upper_limit}"/>
-        <safety_controller soft_lower_limit="${joint_lower_limit + joint_buffer}" soft_upper_limit="${joint_upper_limit - joint_buffer}" k_position="10" k_velocity="10" />
+        <safety_controller soft_lower_limit="${joint_lower_limit + joint_buffer}" soft_upper_limit="${joint_upper_limit - joint_buffer}" k_position="1000" k_velocity="1000" />
     </joint>
     <!-- give colors to some links in gazebo -->

Commit message: Move direction to encoder class

File: ros2/src/shared/march_description/urdf/test_joint_linear.xacro (robot description, xacro)
@@ -16,6 +16,6 @@
     <xacro:property name="joint_lower_limit" value="${-8.5*pi/180}"/> <!-- rad -->
     <xacro:property name="joint_upper_limit" value="${8.5*pi/180}"/> <!-- rad -->
-    <xacro:property name="joint_effort_limit" value="10927.0"/>
-    <xacro:property name="joint_velocity_limit" value="1.0"/> <!-- rad/s -->
+    <xacro:property name="joint_effort_limit" value="20.0"/>
+    <xacro:property name="joint_velocity_limit" value="2.0"/> <!-- rad/s -->
     <xacro:property name="hover_height" value="0.5"/>
     <xacro:include filename="march.gazebo"/>
@@ -85,5 +85,5 @@
         <actuator name="linear_joint_motor">
             <hardwareInterface>hardware_interface/EffortJointInterface</hardwareInterface>
-            <mechanicalReduction>1</mechanicalReduction>
+            <mechanicalReduction>236</mechanicalReduction>
         </actuator>
     </transmission>

Commit message: Remove old test_joint files

File: ros2/src/shared/march_description/urdf/test_joint_linear.xacro (robot description, xacro)
@@ -3,7 +3,7 @@
 <robot name="march" xmlns:xacro="http://www.ros.org/wiki/xacro">
     <!-- Switch between airgaiting or standing on the ground-->
-    <!--Value set to: 'world' fixes the robot to the world-->
-    <!--Value set to: 'base_link' makes the robot stand on the ground-->
-    <!--Important note: when changing value make sure rviz fixed frame is set to the same value (moveit.rviz)-->
+    <!--Value set to 'world' fixes the robot to the world-->
+    <!--Value set to 'base_link' makes the robot stand on the ground-->
+    <!--Important note when changing value make sure rviz fixed frame is set to the same value (moveit.rviz)-->
     <!-- Constants for robot dimensions -->
     <xacro:property name="PI" value="3.1415926535897931"/>
@@ -13,7 +13,7 @@
     <xacro:property name="bar_mass" value="1.080"/>
     <xacro:property name="bar_width" value="0.05"/>
-    <xacro:property name="joint_buffer" value="${3*pi/180}"/> <!-- rad -->
-    <xacro:property name="joint_lower_limit" value="${-8.5*pi/180}"/> <!-- rad -->
-    <xacro:property name="joint_upper_limit" value="${8.5*pi/180}"/> <!-- rad -->
+    <xacro:property name="joint_buffer" value="${0*pi/180}"/> <!-- rad -->
+    <xacro:property name="joint_lower_limit" value="-0.2013"/> <!-- rad -->
+    <xacro:property name="joint_upper_limit" value="0.1477"/> <!-- rad -->
     <xacro:property name="joint_effort_limit" value="20.0"/>
     <xacro:property name="joint_velocity_limit" value="2.0"/> <!-- rad/s -->
@@ -36,5 +36,5 @@
         <axis xyz="0 1 0"/>
         <limit velocity="${joint_velocity_limit}" effort="${joint_effort_limit}" lower="${joint_lower_limit}" upper="${joint_upper_limit}"/>
-        <safety_controller soft_lower_limit="${joint_lower_limit + joint_buffer}" soft_upper_limit="${joint_upper_limit - joint_buffer}" k_position="10" k_velocity="10" />
+        <safety_controller soft_lower_limit="${joint_lower_limit + joint_buffer}" soft_upper_limit="${joint_upper_limit - joint_buffer}" k_position="20000" k_velocity="20000" />
     </joint>
     <!-- give colors to some links in gazebo -->
@@ -85,5 +85,5 @@
         <actuator name="linear_joint_motor">
             <hardwareInterface>hardware_interface/EffortJointInterface</hardwareInterface>
-            <mechanicalReduction>236</mechanicalReduction>
+            <mechanicalReduction>240</mechanicalReduction>
         </actuator>
     </transmission>

File: ros2/src/shared/march_description/urdf/test_joint_rotational.xacro (robot description, xacro)
@@ -8,9 +8,9 @@
     <xacro:property name="bar_mass" value="1.080"/>
     <xacro:property name="bar_width" value="0.05"/>
-    <xacro:property name="joint_buffer" value="${3*(pi/180)}"/> <!-- rad -->
-    <xacro:property name="joint_lower_limit" value="-0.5363"/> <!-- rad -->
-    <xacro:property name="joint_upper_limit" value="0.5363"/> <!-- rad -->
-    <xacro:property name="joint_effort_limit" value="21840"/> <!-- IU = 20 A -->
-    <xacro:property name="joint_velocity_limit" value="2.0"/> <!-- rad/s -->
+    <xacro:property name="joint_buffer"         value="${3*(pi/180)}"/>     <!-- rad -->
+    <xacro:property name="joint_lower_limit"    value="-0.4395"/>   <!-- rad -->
+    <xacro:property name="joint_upper_limit"    value="1.7857"/>     <!-- rad -->
+    <xacro:property name="joint_effort_limit"   value="20"/>                <!-- IU -->
+    <xacro:property name="joint_velocity_limit" value="3.0"/>               <!-- rad/s -->
     <xacro:property name="hover_height" value="0.5"/>
     <xacro:include filename="march.gazebo"/>
@@ -28,5 +28,5 @@
         <axis xyz="0 1 0"/>
         <limit velocity="${joint_velocity_limit}" effort="${joint_effort_limit}" lower="${joint_lower_limit}" upper="${joint_upper_limit}"/>
-        <safety_controller soft_lower_limit="${joint_lower_limit + joint_buffer}" soft_upper_limit="${joint_upper_limit - joint_buffer}" k_position="5" k_velocity="20000" />
+        <safety_controller soft_lower_limit="${joint_lower_limit + joint_buffer}" soft_upper_limit="${joint_upper_limit - joint_buffer}" k_position="20000" k_velocity="20000" />
     </joint>
     <!-- give colors to some links in gazebo -->
@@ -75,5 +75,5 @@
         </joint>
         <actuator name="rotational_joint_motor">
-            <mechanicalReduction>101</mechanicalReduction>
+            <mechanicalReduction>121</mechanicalReduction>
         </actuator>
     </transmission>

Commit message: Update .xacro file for linear test joint

File: ros2/src/shared/march_description/urdf/test_joint_linear.xacro (robot description, xacro)
@@ -20,7 +20,22 @@
     <xacro:property name="hover_height" value="0.5"/>
     <xacro:include filename="march.gazebo"/>
-    <plugin name="gazebo_ros_control" filename="libgazebo_ros_control.so">
-        <robotNamespace>/march</robotNamespace>
-    </plugin>
+    <xacro:arg name="configuration" default="exoskeleton"/>
+    <xacro:property name="configuration" value="$(arg configuration)"/>
+    <!-- Include all macro files    -->
+    <xacro:include filename="macros/safety_limits.xacro"/>
+    <xacro:include filename="macros/pressure_sole.xacro"/>
+    <xacro:include filename="macros/frame_part.xacro"/>
+    <xacro:include filename="macros/joint.xacro"/>
+    <xacro:include filename="macros/configurable_joint.xacro"/>
+    <!-- Add yaml files with properties -->
+    <xacro:property name="config_yaml_file"
+                    value="properties/test_joints.yaml"/>
+    <xacro:property name="properties" value="${load_yaml(config_yaml_file)}"/>
+    <xacro:property name="joint_limits" value="${properties['joint_limits']}"/>
+    <xacro:property name="safety_values"
+                    value="${properties['safety'][configuration]}"/>
+    <xacro:property name="inertia" value="${properties['inertia']}"/>
+    <xacro:property name="dimensions" value="${properties['dimensions']}"/>
+    <xacro:property name="linear_reduction_ankle" value="236"/>
     <!-- Used for fixing robot to Gazebo 'base_link' -->
     <link name="world"/>
@@ -30,12 +45,14 @@
         <origin xyz="0 0 ${hover_height}" rpy="0 0 0"/>
     </joint>
-    <joint name="linear_joint" type="revolute">
-        <parent link="joint_base"/>
-        <child link="bar"/>
-        <origin xyz="0 ${-joint_base_width} 0" rpy="0 0 0"/>
-        <axis xyz="0 1 0"/>
-        <limit velocity="${joint_velocity_limit}" effort="${joint_effort_limit}" lower="${joint_lower_limit}" upper="${joint_upper_limit}"/>
-        <safety_controller soft_lower_limit="${joint_lower_limit + joint_buffer}" soft_upper_limit="${joint_upper_limit - joint_buffer}" k_position="20000" k_velocity="20000" />
-    </joint>
+    <xacro:march_configurable_joint
+            name="linear_joint"
+            parent="joint_base"
+            child="bar"
+            safety="${safety_values['linear_joint']}"
+            origin="0 ${-joint_base_width} 0"
+            axis="0 1 0"
+            reduction="${linear_reduction_ankle}"
+            limits="${joint_limits['linear_joint']}"
+    />
     <!-- give colors to some links in gazebo -->
     <gazebo reference="joint_base">
@@ -77,14 +94,3 @@
         </inertial>
     </link>
-    <!-- ROS Control plugin for Gazebo -->
-    <transmission name="linear_joint_transmission">
-        <type>transmission_interface/SimpleTransmission</type>
-        <joint name="linear_joint">
-            <hardwareInterface>hardware_interface/EffortJointInterface</hardwareInterface>
-        </joint>
-        <actuator name="linear_joint_motor">
-            <hardwareInterface>hardware_interface/EffortJointInterface</hardwareInterface>
-            <mechanicalReduction>240</mechanicalReduction>
-        </actuator>
-    </transmission>
 </robot>

File: ros2/src/shared/march_description/urdf/test_joint_rotational.xacro (robot description, xacro)
@@ -29,5 +29,4 @@
     <!-- Harmonic Drive: 101, Belt: 1,2-->
     <xacro:property name="rotary_reduction" value="${101 * 1.2}"/>
-    <xacro:property name="actuating_joints" value="${(properties['actuating_joints'])}"/>
     <!-- Used for fixing robot to Gazebo 'base_link' -->
     <link name="world"/>

Commit message: Updating limits in the test_joint_linear xacro file and converting them to meters

File: ros2/src/shared/march_description/urdf/test_joint_linear.xacro (robot description, xacro)
@@ -13,9 +13,9 @@
     <xacro:property name="bar_mass" value="1.080"/>
     <xacro:property name="bar_width" value="0.05"/>
-    <xacro:property name="joint_buffer" value="1"/> <!-- rad -->
-    <xacro:property name="joint_lower_limit" value="-20"/> <!-- rad -->
-    <xacro:property name="joint_upper_limit" value="20"/> <!-- rad -->
-    <xacro:property name="joint_effort_limit" value="10"/>
-    <xacro:property name="joint_velocity_limit" value="10.0"/> <!-- rad/s -->
+    <xacro:property name="joint_buffer" value="0.001"/> <!-- m -->
+    <xacro:property name="joint_lower_limit" value="-0.021"/> <!-- m -->
+    <xacro:property name="joint_upper_limit" value="0.021"/> <!-- m -->
+    <xacro:property name="joint_effort_limit" value="28"/>
+    <xacro:property name="joint_velocity_limit" value="0.10"/> <!-- m/s -->
     <xacro:property name="hover_height" value="0.5"/>
     <xacro:include filename="march.gazebo"/>
