Commit message: Upper left leg

File: ros2/src/shared/march_description/urdf/march6.xacro (robot description, xacro)
@@ -186,5 +186,5 @@
     <xacro:include filename="march.gazebo"/>
     <material name="blue">
-        <color rgba="0 0.35 0.52"/> <!-- TODO nieuwe huisstijl -->
+        <color rgba="0 0 0.6 1"/> <!-- TODO nieuwe huisstijl -->
     </material>
     <!-- Used for fixing robot to Gazebo 'base_link' -->
@@ -259,7 +259,7 @@
     <link name="upper_leg_left">
         <visual>
-            <origin xyz="0 ${hip_base_height/2 + hip_aa_frame_height - upper_leg_offset} 0" rpy="0 0 ${pi}"/>
-            <geometry>
-                <mesh filename="package://march_description/urdf/stl-files/UpperLeftLeg.stl" scale="1 1 1"/>
+            <origin xyz="0 0 0" rpy="0 0 ${pi}"/>
+            <geometry>
+                <mesh filename="package://march_description/urdf/stl-files/march6/UpperLegTest.stl" scale="0.001 0.001 0.001"/>
             </geometry>
             <material name="blue"/>

Commit message: Right leg and temporary .gitignore

File: ros2/src/shared/march_description/urdf/march6.xacro (robot description, xacro)
@@ -194,7 +194,7 @@
     <link name="hip_base">
         <visual>
-            <origin xyz="${-hip_aa_frame_width} 0 0" rpy="0 0 ${pi}"/>
-            <geometry>
-                <mesh filename="package://march_description/urdf/stl-files/HipBase.stl" scale="1 1 1"/>
+            <origin xyz="${hip_aa_frame_width} ${-hip_base_height/2} ${-width}" rpy="0 0 0"/>
+            <geometry>
+                <mesh filename="package://march_description/urdf/stl-files/march6/HipBase.stl" scale="0.001 0.001 0.001"/>
             </geometry>
             <material name="blue"/>
@@ -261,5 +261,5 @@
             <origin xyz="0 0 0" rpy="0 0 ${pi}"/>
             <geometry>
-                <mesh filename="package://march_description/urdf/stl-files/march6/UpperLegTest.stl" scale="0.001 0.001 0.001"/>
+                <mesh filename="package://march_description/urdf/stl-files/UpperLeftLeg.stl" scale="0.001 0.001 0.001"/>
             </geometry>
             <material name="blue"/>
@@ -428,7 +428,7 @@
     <link name="upper_leg_right">
         <visual>
-            <origin xyz="0 ${-hip_base_height/2 - hip_aa_frame_height + upper_leg_offset} 0" rpy="0 0 ${pi}"/>
-            <geometry>
-                <mesh filename="package://march_description/urdf/stl-files/UpperRightLeg.stl" scale="1 1 1"/>
+            <origin xyz="0 0 ${-upper_leg_height-width}" rpy="0 0 0"/>
+            <geometry>
+                <mesh filename="package://march_description/urdf/stl-files/march6/UpperRightLeg.stl" scale="0.001 0.001 0.001"/>
             </geometry>
             <material name="blue"/>
@@ -456,9 +456,9 @@
         <visual>
             <origin
-                xyz="0 ${-hip_base_height/2 - hip_aa_frame_height + upper_leg_offset} ${upper_leg_height}"
-                rpy="0 0 ${pi}"
+                xyz="0 ${0} ${-lower_leg_height}"
+                rpy="0 0 0"
             />
             <geometry>
-                <mesh filename="package://march_description/urdf/stl-files/LowerRightLeg.stl" scale="1 1 1"/>
+                <mesh filename="package://march_description/urdf/stl-files/march6/LowerRightLeg.stl" scale="0.001 0.001 0.001"/>
             </geometry>
             <material name="blue"/>

Commit message: Update mechanical reduction joint

File: ros2/src/shared/march_description/urdf/march6.xacro (robot description, xacro)
@@ -41,6 +41,9 @@
     <xacro:property name="inertia" value="${properties['inertia']}"/>
     <xacro:property name="dimensions" value="${properties['dimensions']}"/>
-    <xacro:property name="rotary_reduction" value="101"/>
-    <xacro:property name="linear_reduction" value="200"/>
+    <!-- Harmonic Drive: 101, Belt: 1,2-->
+    <xacro:property name="rotary_reduction" value="${101 * 1.2}"/>
+    <!-- Linearised around 0 -->
+    <xacro:property name="linear_reduction_hip" value="240"/>
+    <xacro:property name="linear_reduction_ankle" value="236"/>
     <!-- Constants for robot dimensions -->
     <!-- Masses determined in Catia, see https://confluence.projectmarch.nl:8443/display/51/URDF+description -->
@@ -296,5 +299,5 @@
             safety="${safety_values['haa']}"
             limits="${joint_limits['left_haa']}"
-            reduction="${linear_reduction}"
+            reduction="${linear_reduction_hip}"
     />
     <joint name="left_hip_angle" type="fixed">
@@ -330,5 +333,5 @@
             origin="0 ${ankle_plate_offset} ${-lower_leg_height}"
             axis="0 1 0"
-            reduction="${linear_reduction}"
+            reduction="${linear_reduction_ankle}"
             limits="${joint_limits['left_ankle']}"
     />
@@ -345,5 +348,5 @@
             axis="1 0 0"
             safety="${safety_values['haa']}"
-            reduction="${linear_reduction}"
+            reduction="${linear_reduction_ankle}"
             limits="${joint_limits['right_haa']}"
     />
@@ -380,5 +383,5 @@
             origin="0 ${-ankle_plate_offset} ${-lower_leg_height}"
             axis="0 1 0"
-            reduction="${linear_reduction}"
+            reduction="${linear_reduction_ankle}"
             limits="${joint_limits['right_ankle']}"
     />

Commit message: Remove redundant scale arguments

File: ros2/src/shared/march_description/urdf/march6.xacro (robot description, xacro)
@@ -115,5 +115,4 @@
     <xacro:property name="foot_com_z"
                     value="${upper_leg_height + lower_leg_height + ankle_plate_height - 0.789788}"/>
-    <xacro:property name="foot_scale" value="1.35"/>
     <!-- Import all Gazebo-customization elements, including Gazebo colors -->
     <xacro:include filename="march.gazebo"/>
@@ -135,5 +134,4 @@
                       mass="${dimensions['hip_base']['mass']}"
                       inertia="${inertia['hip_base']}"
-                      scale="1 1 1"
                       visual_rpy="0 0 0"
     />
@@ -148,5 +146,4 @@
                       visual_origin="${width/2} ${width/2} ${-width}"
                       mesh="march6/HipLeft.stl"
-                      scale="1 1 1"
                       visual_rpy="0 0 0"
     />
@@ -172,5 +169,4 @@
                       mass="${upper_leg_mass}"
                       inertia="${inertia['upper_leg']}"
-                      scale="1 1 1"
     />
     <xacro:frame_part name="lower_leg_left"
@@ -184,5 +180,4 @@
                       mass="${lower_leg_mass}"
                       inertia="${inertia['lower_leg']}"
-                      scale="1 1 1"
     />
 <!-- Left Foot -->
@@ -194,5 +189,4 @@
                       visual_origin="${-foot_height_forward+0.005} ${-ankle_plate_offset+knee_offset-width/2} ${-ankle_plate_height-width+0.01}"
                       collision_origin="0 0 ${-ankle_plate_height/2}"
-                      scale="1 1 1"
                       visual_rpy="0 0 ${pi}"
     />
@@ -220,5 +214,4 @@
                       collision_origin="0 ${hip_aa_frame_height/2} 0"
                       mesh="march6/HipRight.stl"
-                      scale="1 1 1"
                       visual_rpy="0 0 ${pi}"
     />
@@ -243,5 +236,4 @@
                       inertia="${inertia['upper_leg']}"
                       mass="${upper_leg_mass}"
-                      scale="1 1 1"
                       visual_rpy="0 0 0"
     />
@@ -256,5 +248,4 @@
                       inertia="${inertia['lower_leg']}"
                       collision_origin="0 0 ${-lower_leg_height/2}"
-                      scale="1 1 1"
                       visual_rpy="0 0 0"
     />
@@ -267,5 +258,4 @@
                       visual_origin="0 ${ankle_plate_offset-knee_offset+width/2} ${-ankle_plate_height-width+0.01}"
                       collision_origin="0 0 ${-ankle_plate_height/2}"
-                      scale="1 1 1"
                       visual_rpy="0 0 0"
     />

Commit message: Fix working with part of joint in simulation

File: ros2/src/shared/march_description/urdf/march6.xacro (robot description, xacro)
@@ -32,4 +32,5 @@
     <xacro:include filename="macros/frame_part.xacro"/>
     <xacro:include filename="macros/joint.xacro"/>
+    <xacro:include filename="macros/configurable_joint.xacro"/>
     <!-- Add yaml files with properties -->
     <xacro:property name="config_yaml_file"
@@ -46,4 +47,5 @@
     <xacro:property name="linear_reduction_hip" value="240"/>
     <xacro:property name="linear_reduction_ankle" value="236"/>
+    <xacro:property name="moving_joints" value="${(properties['moving_joints'])}"/>
     <!-- Constants for robot dimensions -->
     <!-- Masses determined in Catia, see https://confluence.projectmarch.nl:8443/display/51/URDF+description -->
@@ -273,5 +275,5 @@
         <origin xyz="0 0 ${lower_leg_height+upper_leg_height+ankle_plate_height+width/2.0+hover_height}" rpy="0 0 0"/>
     </joint>
-    <xacro:march_joint
+    <xacro:march_configurable_joint
             name="left_hip_aa"
             parent="hip_base"
@@ -288,5 +290,5 @@
         <origin xyz="0 ${-hip_aa_frame_height} 0" rpy="0 0 0"/>
     </joint>
-    <xacro:march_joint
+    <xacro:march_configurable_joint
             name="left_hip_fe"
             parent="hip_aa_frame_left_front"
@@ -298,5 +300,5 @@
             limits="${joint_limits['left_hfe']}"
     />
-    <xacro:march_joint
+    <xacro:march_configurable_joint
             name="left_knee"
             parent="upper_leg_left"
@@ -308,5 +310,5 @@
             limits="${joint_limits['left_knee']}"
     />
-    <xacro:march_joint
+    <xacro:march_configurable_joint
             name="left_ankle"
             parent="lower_leg_left"
@@ -323,5 +325,5 @@
         <origin xyz="0 0 ${-ankle_plate_height-width/2}" rpy="0 0 0"/>
     </joint>
-    <xacro:march_joint
+    <xacro:march_configurable_joint
             name="right_hip_aa"
             parent="hip_base"
@@ -338,5 +340,5 @@
         <origin xyz="0 ${hip_aa_frame_height} 0" rpy="0 0 0"/>
     </joint>
-    <xacro:march_joint
+    <xacro:march_configurable_joint
             name="right_hip_fe"
             parent="hip_aa_frame_right_front"
@@ -348,5 +350,5 @@
             limits="${joint_limits['right_hfe']}"
     />
-    <xacro:march_joint
+    <xacro:march_configurable_joint
             name="right_knee"
             parent="upper_leg_right"
@@ -358,5 +360,5 @@
             reduction="${rotary_reduction}"
     />
-    <xacro:march_joint
+    <xacro:march_configurable_joint
             name="right_ankle"
             parent="lower_leg_right"

Commit message: Rename moving to actuating

File: ros2/src/shared/march_description/urdf/march6.xacro (robot description, xacro)
@@ -47,5 +47,5 @@
     <xacro:property name="linear_reduction_hip" value="240"/>
     <xacro:property name="linear_reduction_ankle" value="236"/>
-    <xacro:property name="moving_joints" value="${(properties['moving_joints'])}"/>
+    <xacro:property name="actuating_joints" value="${(properties['actuating_joints'])}"/>
     <!-- Constants for robot dimensions -->
     <!-- Masses determined in Catia, see https://confluence.projectmarch.nl:8443/display/51/URDF+description -->

Commit message: Debug changes

File: ros2/src/shared/march_description/urdf/march6.xacro (robot description, xacro)
@@ -273,14 +273,19 @@
         <origin xyz="0 0 ${lower_leg_height+upper_leg_height+ankle_plate_height+width/2.0+hover_height}" rpy="0 0 0"/>
     </joint>
-    <xacro:march_joint
-            name="left_hip_aa"
-            parent="hip_base"
-            child="hip_aa_frame_left_side"
-            origin="0 ${-hip_base_height/2} 0"
-            axis="-1 0 0"
-            safety="${safety_values['haa']}"
-            limits="${joint_limits['left_haa']}"
-            reduction="${linear_reduction_hip}"
-    />
+<!--    <xacro:march_joint-->
+<!--            name="left_hip_aa"-->
+<!--            parent="hip_base"-->
+<!--            child="hip_aa_frame_left_side"-->
+<!--            origin="0 ${-hip_base_height/2} 0"-->
+<!--            axis="-1 0 0"-->
+<!--            safety="${safety_values['haa']}"-->
+<!--            limits="${joint_limits['left_haa']}"-->
+<!--            reduction="${linear_reduction_hip}"-->
+<!--    />-->
+    <joint name="left_hip_aa" type="fixed">
+        <parent link="hip_base"/>
+        <child link="hip_aa_frame_left_side"/>
+        <origin xyz="0 ${-hip_base_height/2} 0" rpy="0 0 0"/>
+    </joint>
     <joint name="left_hip_angle" type="fixed">
         <parent link="hip_aa_frame_left_side"/>
@@ -308,14 +313,19 @@
             limits="${joint_limits['left_knee']}"
     />
-    <xacro:march_joint
-            name="left_ankle"
-            parent="lower_leg_left"
-            child="ankle_plate_left"
-            safety="${safety_values['ankle']}"
-            origin="0 ${ankle_plate_offset} ${-lower_leg_height}"
-            axis="0 1 0"
-            reduction="${linear_reduction_ankle}"
-            limits="${joint_limits['left_ankle']}"
-    />
+<!--    <xacro:march_joint-->
+<!--            name="left_ankle"-->
+<!--            parent="lower_leg_left"-->
+<!--            child="ankle_plate_left"-->
+<!--            safety="${safety_values['ankle']}"-->
+<!--            origin="0 ${ankle_plate_offset} ${-lower_leg_height}"-->
+<!--            axis="0 1 0"-->
+<!--            reduction="${linear_reduction_ankle}"-->
+<!--            limits="${joint_limits['left_ankle']}"-->
+<!--    />-->
+    <joint name="left_ankle" type="fixed">
+        <parent link="lower_leg_left"/>
+        <child link="ankle_plate_left"/>
+        <origin xyz="0 ${ankle_plate_offset} ${-lower_leg_height}" rpy="0 0 0"/>
+    </joint>
     <joint name="left_foot_angle" type="fixed">
         <parent link="ankle_plate_left"/>
@@ -323,14 +333,19 @@
         <origin xyz="0 0 ${-ankle_plate_height-width/2}" rpy="0 0 0"/>
     </joint>
-    <xacro:march_joint
-            name="right_hip_aa"
-            parent="hip_base"
-            child="hip_aa_frame_right_side"
-            origin="0 ${hip_base_height/2} 0"
-            axis="1 0 0"
-            safety="${safety_values['haa']}"
-            reduction="${linear_reduction_ankle}"
-            limits="${joint_limits['right_haa']}"
-    />
+<!--    <xacro:march_joint-->
+<!--            name="right_hip_aa"-->
+<!--            parent="hip_base"-->
+<!--            child="hip_aa_frame_right_side"-->
+<!--            origin="0 ${hip_base_height/2} 0"-->
+<!--            axis="1 0 0"-->
+<!--            safety="${safety_values['haa']}"-->
+<!--            reduction="${linear_reduction_ankle}"-->
+<!--            limits="${joint_limits['right_haa']}"-->
+<!--    />-->
+    <joint name="right_hip_aa" type="fixed">
+        <parent link="hip_base"/>
+        <child link="hip_aa_frame_right_side"/>
+        <origin xyz="0 ${hip_base_height/2} 0" rpy="0 0 0"/>
+    </joint>
     <joint name="right_hip_angle" type="fixed">
         <parent link="hip_aa_frame_right_side"/>
@@ -358,14 +373,19 @@
             reduction="${rotary_reduction}"
     />
-    <xacro:march_joint
-            name="right_ankle"
-            parent="lower_leg_right"
-            child="ankle_plate_right"
-            safety="${safety_values['ankle']}"
-            origin="0 ${-ankle_plate_offset} ${-lower_leg_height}"
-            axis="0 1 0"
-            reduction="${linear_reduction_ankle}"
-            limits="${joint_limits['right_ankle']}"
-    />
+<!--    <xacro:march_joint-->
+<!--            name="right_ankle"-->
+<!--            parent="lower_leg_right"-->
+<!--            child="ankle_plate_right"-->
+<!--            safety="${safety_values['ankle']}"-->
+<!--            origin="0 ${-ankle_plate_offset} ${-lower_leg_height}"-->
+<!--            axis="0 1 0"-->
+<!--            reduction="${linear_reduction_ankle}"-->
+<!--            limits="${joint_limits['right_ankle']}"-->
+<!--    />-->
+    <joint name="right_ankle" type="fixed">
+        <parent link="lower_leg_right"/>
+        <child link="ankle_plate_right"/>
+        <origin xyz="0 ${-ankle_plate_offset} ${-lower_leg_height}" rpy="0 0 0"/>
+    </joint>
     <joint name="right_foot_angle" type="fixed">
         <parent link="ankle_plate_right"/>

Commit message: Fixing yaw problems

File: ros2/src/shared/march_description/urdf/march6.xacro (robot description, xacro)
@@ -273,5 +273,5 @@
         <parent link="imu_link"/>
         <child link="hip_base"/>
-        <origin xyz="0 0 ${lower_leg_height+upper_leg_height+ankle_plate_height+width/2.0+hover_height}" rpy="0 0 0"/>
+        <origin xyz="0 0 ${lower_leg_height+upper_leg_height+ankle_plate_height+width/2.0+hover_height}" rpy="0 0 ${0.25 * pi}"/>
     </joint>
     <xacro:march_configurable_joint

Commit message: Add final functionality

File: ros2/src/shared/march_description/urdf/march6.xacro (robot description, xacro)
@@ -273,5 +273,5 @@
         <parent link="imu_link"/>
         <child link="hip_base"/>
-        <origin xyz="0 0 ${lower_leg_height+upper_leg_height+ankle_plate_height+width/2.0+hover_height}" rpy="0 0 ${0.25 * pi}"/>
+        <origin xyz="1 2 ${lower_leg_height+upper_leg_height+ankle_plate_height+width/2.0+hover_height}" rpy="0.2 0.3 ${0.58634739845}"/>
     </joint>
     <xacro:march_configurable_joint

Commit message: Update Realsense position

File: ros2/src/shared/march_description/urdf/march6.xacro (robot description, xacro)
@@ -389,5 +389,5 @@
         <!--    Attached to the hip_base, since this is most comparable to the backpack -->
         <!--    in amount of movement, the distance from hip base is based on first design.-->
-        <origin xyz="-0.17 0.195 0.215" rpy="${0.5 * pi} ${0.25 * pi} ${pi}"/>
+        <origin xyz="-0.32 0.22 0.16" rpy="${0.5 * pi} ${0.25 * pi} ${pi}"/>
         <!-- Rotate to be vertical and pointing down 45 degrees -->
     </xacro:sensor_d435>

Commit message: Rotate backsense

File: ros2/src/shared/march_description/urdf/march6.xacro (robot description, xacro)
@@ -394,5 +394,5 @@
     <xacro:sensor_d435 name="camera_back" topics_ns="camera_back" parent="hip_base"
                        plugin="$(arg realsense_simulation)">
-        <origin xyz="0 0.22 0" rpy="0 ${0.3 * pi} 0"/>
+        <origin xyz="0 0.22 0" rpy="0 ${0.48 * pi} 0"/>
     </xacro:sensor_d435>
 </robot>

Commit message: Add jointless launch option to ros2

File: ros2/src/shared/march_description/urdf/march6.xacro (robot description, xacro)
@@ -14,4 +14,7 @@
     <!--    to be used for the transformations.-->
     <xacro:arg name="realsense_simulation" default="false"/>
+    <!--    Running the exoskeleton jointless can be usefull for testing hardware -->
+    <!-- like the camera's or the Power Distribution board -->
+    <xacro:arg name="jointless" default="false"/>
     <xacro:unless value="$(arg ground_gait)">
         <xacro:property name="parent_name" value="world"/>
@@ -47,5 +50,8 @@
     <xacro:property name="linear_reduction_hip" value="240"/>
     <xacro:property name="linear_reduction_ankle" value="236"/>
-    <xacro:property name="actuating_joints" value="${(properties['actuating_joints'])}"/>
+    <xacro:property name="actuating_joints" value="[]"/>
+    <xacro:unless value="$(arg jointless)">
+        <xacro:property name="actuating_joints" value="${(properties['actuating_joints'])}"/>
+    </xacro:unless>
     <!-- Constants for robot dimensions -->
     <!-- Masses determined in Catia, see https://confluence.projectmarch.nl:8443/display/51/URDF+description -->

Commit message: Undo change in urdf

File: ros2/src/shared/march_description/urdf/march6.xacro (robot description, xacro)
@@ -394,5 +394,5 @@
     <xacro:sensor_d435 name="camera_back" topics_ns="camera_back" parent="hip_base"
                        plugin="$(arg realsense_simulation)">
-        <origin xyz="0 0.22 0" rpy="0 ${0.48 * pi} 0"/>
+        <origin xyz="0 0.22 0" rpy="0 ${0.3 * pi} 0"/>
     </xacro:sensor_d435>
 </robot>

Commit message: Update camera position'

File: ros2/src/shared/march_description/urdf/march6.xacro (robot description, xacro)
@@ -389,5 +389,5 @@
         <!--    Attached to the hip_base, since this is most comparable to the backpack -->
         <!--    in amount of movement, the distance from hip base is based on first design.-->
-        <origin xyz="-0.32 0.22 0.16" rpy="${0.5 * pi} ${0.25 * pi} ${pi}"/>
+        <origin xyz="-0.32 0.22 0.16" rpy="${0.5 * pi} ${0.21 * pi} ${pi}"/>
         <!-- Rotate to be vertical and pointing down 45 degrees -->
     </xacro:sensor_d435>

Commit message: Update camera position in the right direction

File: ros2/src/shared/march_description/urdf/march6.xacro (robot description, xacro)
@@ -389,5 +389,5 @@
         <!--    Attached to the hip_base, since this is most comparable to the backpack -->
         <!--    in amount of movement, the distance from hip base is based on first design.-->
-        <origin xyz="-0.32 0.22 0.16" rpy="${0.5 * pi} ${0.21 * pi} ${pi}"/>
+        <origin xyz="-0.32 0.22 0.16" rpy="${0.5 * pi} ${0.29 * pi} ${pi}"/>
         <!-- Rotate to be vertical and pointing down 45 degrees -->
     </xacro:sensor_d435>

Commit message: Update to use back imu orientations do not seem correct yet

File: ros2/src/shared/march_description/urdf/march6.xacro (robot description, xacro)
@@ -389,10 +389,10 @@
         <!--    Attached to the hip_base, since this is most comparable to the backpack -->
         <!--    in amount of movement, the distance from hip base is based on first design.-->
-        <origin xyz="-0.32 0.22 0.16" rpy="${0.5 * pi} ${0.29 * pi} ${pi}"/>
+        <origin xyz="-0.32 0.22 0.16" rpy="${0.5 * pi} ${48/180 * pi} ${pi}"/>
         <!-- Rotate to be vertical and pointing down 45 degrees -->
     </xacro:sensor_d435>
     <xacro:sensor_d435 name="camera_back" topics_ns="camera_back" parent="hip_base"
                        plugin="$(arg realsense_simulation)">
-        <origin xyz="0 0.22 0" rpy="0 ${0.48 * pi} 0"/>
+        <origin xyz="0 0.22 0" rpy="0 ${75/180 * pi} 0"/>
     </xacro:sensor_d435>
 </robot>

Commit message: Change back orientation again' g

File: ros2/src/shared/march_description/urdf/march6.xacro (robot description, xacro)
@@ -394,5 +394,5 @@
     <xacro:sensor_d435 name="camera_back" topics_ns="camera_back" parent="hip_base"
                        plugin="$(arg realsense_simulation)">
-        <origin xyz="0 0.22 0" rpy="0 ${75/180 * pi} 0"/>
+        <origin xyz="0 0.22 0" rpy="${pi} ${105/180 * pi} ${pi}"/>
     </xacro:sensor_d435>
 </robot>
