Commit message: Fix back camera using the imu

File: ros2/src/shared/march_description/urdf/march6.xacro (robot description, xacro)
@@ -269,4 +269,5 @@
         <parent link="${parent_name}"/>
         <child link="imu_link"/>
+        <origin xyz="0 0 0" rpy="0 0 0"/>
     </joint>
     <xacro:if value="$(eval configuration == 'exoskeleton')">
@@ -385,5 +386,12 @@
     </joint>
     <xacro:include filename="camera/_d435.urdf.xacro"/>
-    <xacro:sensor_d435 name="camera_front" topics_ns="camera_front" parent="hip_base"
+    <xacro:sensor_d435 name="camera_back" topics_ns="camera_back" parent="hip_aa_frame_right_side"
+                       plugin="$(arg realsense_simulation)">
+        <origin xyz="0 0.06725 0" rpy="0 ${75/180 * pi} 0"/>
+    </xacro:sensor_d435>
+<!--    -->
+<!--    -->
+    <xacro:sensor_d435 name="camera_front" topics_ns="camera_front"
+                       parent="hip_base"
                        plugin="$(arg realsense_simulation)">
         <!--    Attached to the hip_base, since this is most comparable to the backpack -->
@@ -392,7 +400,3 @@
         <!-- Rotate to be vertical and pointing down 45 degrees -->
     </xacro:sensor_d435>
-    <xacro:sensor_d435 name="camera_back" topics_ns="camera_back" parent="hip_base"
-                       plugin="$(arg realsense_simulation)">
-        <origin xyz="0 0.22 0" rpy="${pi} ${105/180 * pi} ${pi}"/>
-    </xacro:sensor_d435>
 </robot>

Commit message: Add jointless argument on more locations

File: ros2/src/shared/march_description/urdf/march6.xacro (robot description, xacro)
@@ -50,5 +50,7 @@
     <xacro:property name="linear_reduction_hip" value="240"/>
     <xacro:property name="linear_reduction_ankle" value="236"/>
-    <xacro:property name="actuating_joints" value="[]"/>
+    <xacro:if value="$(arg jointless)">
+        <xacro:property name="actuating_joints" value="[]"/>
+    </xacro:if>
     <xacro:unless value="$(arg jointless)">
         <xacro:property name="actuating_joints" value="${(properties['actuating_joints'])}"/>

Commit message: Apply 1 suggestion(s) to 1 file(s)

File: ros2/src/shared/march_description/urdf/march6.xacro (robot description, xacro)
@@ -269,5 +269,4 @@
         <parent link="${parent_name}"/>
         <child link="imu_link"/>
-        <origin xyz="0 0 0" rpy="0 0 0"/>
     </joint>
     <xacro:if value="$(eval configuration == 'exoskeleton')">
