Commit message: Make different launch arguments for M6 and M7 realsense nodes

File: ros2/src/shared/march_description/urdf/march6_three_cameras.xacro (robot description, xacro)
@@ -403,3 +403,7 @@
         <origin xyz="-0.08 -0.035 -0.05 " rpy="${0 * pi} ${61/180 * pi} ${pi}"/>
     </xacro:sensor_d435>
+    <xacro:sensor_d435 name="camera_back" topics_ns="camera_back" parent="hip_aa_frame_right_side"
+                       plugin="$(arg realsense_simulation)">
+        <origin xyz="0 0.06725 0" rpy="0 ${75/180 * pi} 0"/>
+    </xacro:sensor_d435>
 </robot>
