Commit message: Resolve "Place cameras in march 7 XACRO"

File: ros2/src/shared/march_description/urdf/march7.xacro (robot description, xacro)
@@ -397,15 +397,24 @@
     </joint>
     <xacro:include filename="camera/_d435.urdf.xacro"/>
-    <xacro:sensor_d435 name="camera_right" topics_ns="camera_back" parent="upper_leg_right"
-                       plugin="$(arg realsense_simulation)">
-        <origin xyz="0.1 0 0" rpy="0 ${75/180 * pi} 0"/>
+    <xacro:sensor_d435
+            name="camera_front_right"
+            topics_ns="camera_front_right"
+            parent="upper_leg_right"
+            plugin="$(arg realsense_simulation)">
+        <origin xyz="-0.07 -0.011 -0.007 " rpy="${0 * pi} ${61/180 * pi} ${pi}"/>
     </xacro:sensor_d435>
-    <xacro:sensor_d435 name="camera_front" topics_ns="camera_front"
-                       parent="hip_base"
-                       plugin="$(arg realsense_simulation)">
-        <!--    Attached to the hip_base, since this is most comparable to the backpack -->
-        <!--    in amount of movement, the distance from hip base is based on first design.-->
-        <origin xyz="-0.32 0.20 0.20" rpy="${0.5 * pi} ${48/180 * pi} ${pi}"/>
-        <!-- Rotate to be vertical and pointing down 48 degrees -->
+    <xacro:sensor_d435
+            name="camera_front_left"
+            topics_ns="camera_front_left"
+            parent="upper_leg_left"
+            plugin="$(arg realsense_simulation)">
+        <origin xyz="-0.07 0.011 -0.007 " rpy="${0 * pi} ${61/180 * pi} ${pi}"/>
+    </xacro:sensor_d435>
+    <xacro:sensor_d435
+            name="camera_back"
+            topics_ns="camera_back"
+            parent="hip_aa_frame_right_side"
+            plugin="$(arg realsense_simulation)">
+        <origin xyz="0.018 0.126 -0.018" rpy="0 ${75/180 * pi} 0"/>
     </xacro:sensor_d435>
 </robot>

Commit message: Ankle encoder values

File: ros2/src/shared/march_description/urdf/march7.xacro (robot description, xacro)
@@ -409,5 +409,5 @@
             parent="upper_leg_left"
             plugin="$(arg realsense_simulation)">
-        <origin xyz="-0.07 0.011 -0.007 " rpy="${0 * pi} ${61/180 * pi} ${pi}"/>
+        <origin xyz="-0.094 0.011 0.005 " rpy="${0 * pi} ${(180 - 61) / 180 * pi} ${0 * pi}"/>
     </xacro:sensor_d435>
     <xacro:sensor_d435

Commit message: Camera rotations in xacro from 15-08-2022 WORKS

File: ros2/src/shared/march_description/urdf/march7.xacro (robot description, xacro)
@@ -400,5 +400,5 @@
             parent="upper_leg_right"
             plugin="$(arg realsense_simulation)">
-        <origin xyz="-0.07 -0.011 -0.007 " rpy="${0 * pi} ${61/180 * pi} ${pi}"/>
+        <origin xyz="-0.07 -0.011 -0.007 " rpy="${0 * pi} ${54/180 * pi} ${pi}"/>
     </xacro:sensor_d435>
     <xacro:sensor_d435
@@ -407,5 +407,5 @@
             parent="upper_leg_left"
             plugin="$(arg realsense_simulation)">
-        <origin xyz="-0.094 0.011 0.005 " rpy="${0 * pi} ${(180 - 61) / 180 * pi} ${0 * pi}"/>
+        <origin xyz="-0.094 0.011 0.005 " rpy="${0 * pi} ${(180 - 54) / 180 * pi} ${0 * pi}"/>
     </xacro:sensor_d435>
     <xacro:sensor_d435

Commit message: Adjust camera angles in xacro file

File: ros2/src/shared/march_description/urdf/march7.xacro (robot description, xacro)
@@ -400,5 +400,5 @@
             parent="upper_leg_right"
             plugin="$(arg realsense_simulation)">
-        <origin xyz="-0.07 -0.011 -0.007 " rpy="${0 * pi} ${54/180 * pi} ${pi}"/>
+        <origin xyz="-0.07 -0.011 -0.007 " rpy="${0 * pi} ${53.5/180 * pi} ${pi}"/>
     </xacro:sensor_d435>
     <xacro:sensor_d435
@@ -407,5 +407,5 @@
             parent="upper_leg_left"
             plugin="$(arg realsense_simulation)">
-        <origin xyz="-0.094 0.011 0.005 " rpy="${0 * pi} ${(180 - 54) / 180 * pi} ${0 * pi}"/>
+        <origin xyz="-0.094 0.011 0.005 " rpy="${0 * pi} ${(180 - 52) / 180 * pi} ${0 * pi}"/>
     </xacro:sensor_d435>
     <xacro:sensor_d435

Commit message: Works. Rehearsal.

File: ros2/src/shared/march_description/urdf/march7.xacro (robot description, xacro)
@@ -400,5 +400,5 @@
             parent="upper_leg_right"
             plugin="$(arg realsense_simulation)">
-        <origin xyz="-0.07 -0.011 -0.007 " rpy="${0 * pi} ${53.5/180 * pi} ${pi}"/>
+        <origin xyz="-0.07 -0.011 -0.007 " rpy="${0 * pi} ${54/180 * pi} ${pi}"/>
     </xacro:sensor_d435>
     <xacro:sensor_d435
@@ -407,5 +407,5 @@
             parent="upper_leg_left"
             plugin="$(arg realsense_simulation)">
-        <origin xyz="-0.094 0.011 0.005 " rpy="${0 * pi} ${(180 - 52) / 180 * pi} ${0 * pi}"/>
+        <origin xyz="-0.094 0.011 0.005 " rpy="${0 * pi} ${(180 - 54) / 180 * pi} ${0 * pi}"/>
     </xacro:sensor_d435>
     <xacro:sensor_d435
