Commit message: modify joint names in urdf

File: ros2/src/shared/march_description/urdf/hennie_v0.urdf (robot description, URDF)
Before this commit: robot Hennie, 11 links, 10 joints
Joints:
- removed joint L_ADPF
- removed joint L_HAA
- removed joint L_HFE
- removed joint L_KFE
- removed joint R_ADPF
- removed joint R_HAA
- removed joint R_HFE
- removed joint R_KFE
- added joint left_ankle: type revolute, parent L_LL, child L_foot, origin xyz=0 -0.037 -0.414 rpy=0 0 0, axis 0 1 0, limit lower=-0.0174533 upper=0.436332 effort=0.9 velocity=4.1
- added joint left_hip_aa: type revolute, parent backpack, child L_hip, origin xyz=-0.021 0.08 0.025 rpy=0 0 0, axis 1 0 0, limit lower=-0.2618 upper=0.174533 effort=280 velocity=2.6
- added joint left_hip_fe: type revolute, parent L_hip, child L_UL, origin xyz=0.182 0.182 0 rpy=0 0 0.0, axis 0 1 0, limit lower=-2.00713 upper=0.20944 effort=250 velocity=3.94
- added joint left_knee: type revolute, parent L_UL, child L_LL, origin xyz=0 -0.06 -0.413 rpy=0 0 0, axis 0 1 0, limit lower=-0.017453 upper=1.9548 effort=250 velocity=3.94
- added joint right_ankle: type revolute, parent R_LL, child R_foot, origin xyz=0 0.037 -0.414 rpy=0 0 0, axis 0 1 0, limit lower=-0.0174533 upper=0.436332 effort=0.9 velocity=4.1
- added joint right_hip_aa: type revolute, parent backpack, child R_hip, origin xyz=-0.021 -0.08 0.025 rpy=0 0 0, axis 1 0 0, limit lower=-0.174533 upper=0.0872665 effort=4.5 velocity=2.6
- added joint right_hip_fe: type revolute, parent R_hip, child R_UL, origin xyz=0.182 -0.182 0 rpy=0 0 0.0, axis 0 1 0, limit lower=-2.00713 upper=0.20944 effort=12.2 velocity=3.94
- added joint right_knee: type revolute, parent R_UL, child R_LL, origin xyz=0 0.06 -0.413 rpy=0 0 0, axis 0 1 0, limit lower=-0.017453 upper=1.9548 effort=12.2 velocity=3.94

Commit message: make that sim updates on joiint_names, and flip axis in hennie.urdf for IK

File: ros2/src/shared/march_description/urdf/hennie_v0.urdf (robot description, URDF)
Before this commit: robot Hennie, 11 links, 10 joints
Joints:
- joint left_ankle: axis 0 1 0 -> 0 -1 0
- joint left_hip_aa: axis 1 0 0 -> -1 0 0
- joint left_hip_fe: axis 0 1 0 -> 0 -1 0
- joint right_ankle: axis 0 1 0 -> 0 -1 0
- joint right_hip_fe: axis 0 1 0 -> 0 -1 0

Commit message: added scalings new urdfs to make a working airgait

File: ros2/src/shared/march_description/urdf/hennie_v0.urdf (robot description, URDF)
Before this commit: robot Hennie, 11 links, 10 joints
Joints:
- joint left_ankle: limit lower=-0.0174533 upper=0.436332 effort=0.9 velocity=4.1 -> lower=-0.436332313 upper=0.1745329252 effort=179 velocity=4.1
- joint left_hip_aa: limit lower=-0.2618 upper=0.174533 effort=280 velocity=2.6 -> lower=-0.2617993878 upper=0.1745329252 effort=280 velocity=2.6
- joint left_hip_fe: limit lower=-2.00713 upper=0.20944 effort=250 velocity=3.94 -> lower=-0.1745329252 upper=1.9634954085 effort=250 velocity=3.94
- joint left_knee: limit lower=-0.017453 upper=1.9548 effort=250 velocity=3.94 -> lower=0 upper=2.181661565 effort=250 velocity=3.94
- joint right_ankle: limit lower=-0.0174533 upper=0.436332 effort=0.9 velocity=4.1 -> lower=-0.436332313 upper=0.1745329252 effort=179 velocity=4.1
- joint right_hip_aa: limit lower=-0.174533 upper=0.0872665 effort=4.5 velocity=2.6 -> lower=-0.2617993878 upper=0.1745329252 effort=280 velocity=2.6
- joint right_hip_fe: limit lower=-2.00713 upper=0.20944 effort=12.2 velocity=3.94 -> lower=-0.1745329252 upper=1.9634954085 effort=250 velocity=3.94
- joint right_knee: limit lower=-0.017453 upper=1.9548 effort=12.2 velocity=3.94 -> lower=0 upper=2.181661565 effort=250 velocity=3.94

Commit message: add toes to the ik solver and urdf

File: ros2/src/shared/march_description/urdf/hennie_v0.urdf (robot description, URDF)
Before this commit: robot Hennie, 11 links, 10 joints
Links:
- added link L_toe
- added link R_toe
Joints:
- added joint left_toe: type fixed, parent L_ground, child L_toe, origin xyz=0.184 -0.085 0
- added joint right_toe: type fixed, parent R_ground, child R_toe, origin xyz=0.184 0.085 0
