Commit message: Add curb obstacle

File: ros1/src/march_simulation/obstacles/curb.xacro (robot description, xacro)
@@ -8,5 +8,5 @@
     <xacro:property name="step_depth" default="0.280"/>
     <xacro:property name="step_width" default="1.80"/>
-    <xacro:property name="distance_to_origin" default="0.4"/>
+    <xacro:property name="distance_to_origin" default="0.45"/>
     <link name="${parent_name}"/>
     <link name="step_1">

Commit message: Make curb obstacle longer

File: ros1/src/march_simulation/obstacles/curb.xacro (robot description, xacro)
@@ -6,5 +6,5 @@
     <xacro:property name="parent_name" value="world"/>
     <xacro:property name="step_height" default="0.170"/>
-    <xacro:property name="step_depth" default="0.280"/>
+    <xacro:property name="step_depth" default="7"/>
     <xacro:property name="step_width" default="1.80"/>
     <xacro:property name="distance_to_origin" default="0.45"/>
