Commit message: Fix working size-changing node with new feature in CoM controller for sitting

File: ros1/src/march_simulation/obstacles/bench.xacro (robot description, xacro)
@@ -2,4 +2,4 @@
 <robot name="bench" xmlns:xacro="http://www.ros.org/wiki/xacro">
     <xacro:include filename="bench_macro.xacro"/>
-    <xacro:bench bench_length="0.5" bench_width="1" bench_height="0.4"/>
+    <xacro:bench length="0.5" width="1" height="0.4"/>
 </robot>

File: ros1/src/march_simulation/obstacles/bench_macro.xacro (robot description, xacro)
@@ -1,5 +1,5 @@
 <?xml version="1.0"?>
 <robot  xmlns:xacro="http://www.ros.org/wiki/xacro">
-    <xacro:macro name="bench" params="bench_length bench_width bench_height">
+    <xacro:macro name="bench" params="length:=0.5 width:=1 height:=0.4">
         <gazebo>
             <static>true</static>
@@ -17,10 +17,10 @@
             <collision>
                 <geometry>
-                    <box size="${bench_length} ${bench_width} ${bench_height}" />
+                    <box size="${length} ${width} ${height}" />
                 </geometry>
             </collision>
             <visual name='visual'>
                 <geometry>
-                    <box size="${bench_length} ${bench_width} ${bench_height}" />
+                    <box size="${length} ${width} ${height}" />
                 </geometry>
             </visual>
@@ -46,5 +46,5 @@
             <parent link="${parent_name}"/>
             <child link="bench"/>
-            <origin xyz="${bench_length / 2} 0 ${bench_height / 2}" rpy="0 0 0"/>
+            <origin xyz="${length / 2} 0 ${height / 2}" rpy="0 0 0"/>
         </joint>
     </xacro:macro>
