Commit message: clean up left over comment

File: ros1/src/simulation/march_simulation/obstacles/ramp_and_door.xacro (robot description, xacro)
@@ -107,4 +107,2 @@
     </joint>
 </robot>
-<!--         <origin xyz="${-1 * sin(radians(45) - ramp_up_slope) * (ramp_up_length / sqrt(2)) - platform_length / 2} 0
-        ${cos(radians(45) - ramp_up_slope) * (ramp_up_length / sqrt(2)) - platform_height / 2}" rpy="0 ${-1 * ramp_up_slope} 0"/> -->

Commit message: Add _macro.xacro file and introduce new service

File: ros1/src/simulation/march_simulation/obstacles/ramp_and_door.xacro (robot description, xacro)
@@ -1,108 +1,5 @@
 <?xml version="1.0"?>
 <robot name="ramp_and_door" xmlns:xacro="http://www.ros.org/wiki/xacro">
-    <gazebo>
-        <static>true</static>
-    </gazebo>
-    <!-- Sizes from the rules of the cybathlon 2020 -->
-    <xacro:property name="platform_height" default="0.48"/>
-    <xacro:property name="platform_length" default="2.920"/>
-    <xacro:property name="platform_width" default="1.4"/>
-    <xacro:property name="ramp_up_length" default="3.0"/>
-    <xacro:property name="distance_to_origin" default="0.4"/>
-    <xacro:property name="ramp_up_slope" default="${radians(20)}"/>
-    <xacro:property name="ramp_down_slope" value="${radians(20)}"/>
-    <xacro:property name="ramp_down_length" default="${sin(ramp_up_slope) * ramp_up_length / sin(ramp_down_slope)}"/>
-    <xacro:property name="parent_name" value="world"/>
-    <xacro:property name="mu1" value="1.0"/>
-    <xacro:property name="mu2" value="1.0"/>
-    <!-- Minimum allowable depth before contact correction impulse is applied. -->
-    <xacro:property name="min_depth" value="0.0005"/>
-    <!-- Used for fixing robot to Gazebo 'base_link' -->
-    <link name="${parent_name}"/>
-    <!-- Links -->
-    <link name="platform">
-        <collision>
-          <geometry>
-            <box size="${platform_length} ${platform_width} ${platform_height}" />
-          </geometry>
-        </collision>
-        <visual name='visual'>
-          <geometry>
-            <box size="${platform_length} ${platform_width} ${platform_height}" />
-          </geometry>
-        </visual>
-        <inertial>
-            <origin xyz="0 0 0" rpy="0 0 0"/>
-            <mass value="1"/>
-            <inertia
-                    ixx="1"
-                    ixy="1"
-                    ixz="1"
-                    iyy="1"
-                    iyz="1"
-                    izz="1" />
-        </inertial>
-    </link>
-    <link name="ramp_up">
-        <collision>
-          <origin xyz="0 0 0" rpy="0 0 0"/>
-          <geometry>
-            <box size="${ramp_up_length} ${platform_width} ${ramp_up_length}" />
-          </geometry>
-        </collision>
-        <visual name='visual'>
-          <origin xyz="0 0 0" rpy="0 0 0"/>
-          <geometry>
-            <box size="${ramp_up_length} ${platform_width} ${ramp_up_length}" />
-          </geometry>
-        </visual>
-    </link>
-    <link name="ramp_down">
-        <collision>
-          <origin xyz="0 0 0" rpy="0 0 0"/>
-          <geometry>
-            <box size="${ramp_down_length} ${platform_width} ${ramp_down_length}" />
-          </geometry>
-        </collision>
-        <visual name='visual'>
-          <origin xyz="0 0 0" rpy="0 0 0"/>
-          <geometry>
-            <box size="${ramp_down_length} ${platform_width} ${ramp_down_length}" />
-          </geometry>
-        </visual>
-    </link>
-    <gazebo reference="platform">
-        <mu1>${mu1}</mu1>
-        <mu2>${mu2}</mu2>
-        <minDepth>${min_depth}</minDepth>
-    </gazebo>
-    <gazebo reference="ramp_up">
-        <mu1>${mu1}</mu1>
-        <mu2>${mu2}</mu2>
-        <minDepth>${min_depth}</minDepth>
-    </gazebo>
-    <gazebo reference="ramp_down">
-        <mu1>${mu1}</mu1>
-        <mu2>${mu2}</mu2>
-        <minDepth>${min_depth}</minDepth>
-    </gazebo>
-    <!-- Joints -->
-    <joint name="joint_0" type="fixed"> <!-- Ensure the ramp up side just above ground, and 0.4 m away from origin -->
-        <parent link="${parent_name}"/>
-        <child link="ramp_up"/>
-        <origin xyz="${-1 * cos(radians(45) - ramp_up_slope) * ramp_up_length / sqrt(2) - distance_to_origin} 0
-                     ${-1 * sin(radians(45) - ramp_up_slope) * ramp_up_length / sqrt(2)}" rpy="0 ${ramp_up_slope} 0"/>
-    </joint>
-    <joint name="joint_1" type="fixed"> <!-- Let platform be straight, and smoothly connect it to the ramp up -->
-        <parent link="ramp_up"/>
-        <child link="platform"/>
-        <origin xyz="${-1 * ramp_up_length / 2 - cos(ramp_up_slope) * platform_length / 2 + sin(ramp_up_slope) * platform_height / 2} 0
-        ${ramp_up_length / 2 - sin(ramp_up_slope) * platform_length / 2 - cos(ramp_up_slope) * platform_height / 2}" rpy="0 ${-1 * ramp_up_slope} 0"/>
-    </joint>
-    <joint name="joint_2" type="fixed">
-        <parent link="platform"/>
-        <child link="ramp_down"/>
-        <origin xyz="${-1 * platform_length / 2 - cos(radians(45) + ramp_down_slope) * ramp_down_length / sqrt(2)} 0
-        ${platform_height / 2 - sin(radians(45) + ramp_down_slope) * ramp_down_length / sqrt(2)}" rpy="0 ${-1 * ramp_down_slope} 0"/>
-    </joint>
+    <xacro:include filename="ramp_and_door_macro.xacro"/>
+    <xacro:ramp_and_door/>
 </robot>
