Commit message: Large xacro refactor, replacing all joints and pressure soles with macros, moving safety to yaml

File: ros2/src/shared/march_description/urdf/macros/frame_part.xacro (robot description, xacro)
@@ -2,5 +2,5 @@
 <robot  xmlns:xacro="http://www.ros.org/wiki/xacro">
     <xacro:macro name="frame_part"
-                 params="name side length width direction collision_origin visual_origin:=0 mesh:=0 com:=0 mass:=0 inertia:=0">
+                 params="name side length direction collision_origin visual_origin:=0 mesh:=0 com:=0 mass:=0 inertia:=0 scale:='1 1 1'">
         <xacro:if value="${direction == 'x'}">
             <xacro:property name="size" value="${length} ${width} ${width}"/>
@@ -20,5 +20,5 @@
                     <origin xyz="${visual_origin}" rpy="${rpy}"/>
                     <geometry>
-                        <mesh filename="package://march_description/urdf/stl-files/${mesh}" scale="1 1 1"/>
+                        <mesh filename="package://march_description/urdf/stl-files/${mesh}" scale="${scale}"/>
                     </geometry>
                     <material name="blue"/>

File: ros2/src/shared/march_description/urdf/macros/joint.xacro (robot description, xacro)
@@ -1,7 +1,6 @@
 <?xml version="1.0"?>
 <robot  xmlns:xacro="http://www.ros.org/wiki/xacro">
-    <xacro:macro name="rotational_joint"
-                 params="name parent child safety origin axis">
-        <xacro:include filename="safety_limits.xacro" />
+    <xacro:macro name="march_joint"
+                 params="name parent child safety origin axis reduction limits">
         <joint name="${name}" type="revolute">
             <parent link="${parent}"/>
@@ -9,5 +8,5 @@
             <origin xyz="${origin}" rpy="0 0 0"/>
             <axis xyz="${axis}"/>
-            <xacro:safety_limits safety="${safety}"/>
+            <xacro:safety_limits safety="${safety}" limits="${limits}"/>
         </joint>
         <transmission name="${name}">
@@ -17,5 +16,7 @@
             </joint>
             <actuator name="${name}_motor">
-                <mechanicalReduction>101</mechanicalReduction>
+                <mechanicalReduction>
+                    ${reduction}
+                </mechanicalReduction>
             </actuator>
         </transmission>

File: ros2/src/shared/march_description/urdf/macros/pressure_sole.xacro (robot description, xacro)
@@ -2,25 +2,28 @@
 <robot  xmlns:xacro="http://www.ros.org/wiki/xacro">
     <xacro:macro name="pressure_sole"
-                 params="side parent">
-        <gazebo reference="${parent}">
-            <sensor name="${parent}_contact" type="contact">
-                <plugin name="contact_plugin" filename="libcontact.so"/>
-                <contact>
-                    <collision name="ankle_plate_left_fixed_joint_lump__foot_left_collision_1"/>
-                </contact>
-                <update_rate>30</update_rate>
+                 params="side foot_name">
+        <link name="pressure_sole_${side}">
+            <collision>
+                <origin xyz="${(-foot_height_forward+foot_height_backward)/2} 0 0" rpy="0 0 0"/>
+                <geometry>
+                    <box size="${foot_height_forward+foot_height_backward} ${width} 0.001"/>
+                </geometry>
+            </collision>
+        </link>
+        <gazebo reference="pressure_sole_${side}">
+            <sensor name="pressure_sole_${side}" type="contact">
                 <always_on>true</always_on>
-            </sensor>
-            <sensor name="left_pressure_sole" type="contact">
-                <always_on>true</always_on>
-                <contact>
-                    <collision>ankle_plate_left_fixed_joint_lump__foot_left_collision_1</collision>
-                </contact>
-                <plugin name="left_foot_plugin" filename="libgazebo_ros_bumper.so">
-                    <bumperTopicName>march/sensor/left_pressure_sole</bumperTopicName>
+                <contact collision="ankle_plate_${side}_fixed_joint_lump__pressure_sole_${side}_collision_2"/>
+                <plugin name="pressure_sole_plugin_${side}" filename="libgazebo_ros_bumper.so">
+                    <bumperTopicName>/march/sensor/right_pressure_sole</bumperTopicName>
                     <frameName>world</frameName>
                 </plugin>
             </sensor>
-        </gazebo>
+        </gazebo>`
+        <joint name="pressure_sole_${side}_joint" type="fixed">
+            <parent link="${foot_name}"/>
+            <child link="pressure_sole_${side}"/>
+            <origin xyz="0 0 ${-(width/2)}" rpy="0 0 0"/>
+        </joint>
     </xacro:macro>
 </robot>

File: ros2/src/shared/march_description/urdf/macros/safety_limits.xacro (robot description, xacro)
@@ -1,13 +1,14 @@
 <?xml version="1.0"?>
 <robot  xmlns:xacro="http://www.ros.org/wiki/xacro">
-    <xacro:macro name="safety_limits" params="safety">
-        <limit velocity="${safety['}"
-               effort="${safety['max_effort']'}"
-               lower="${safety['lower_limit']}"
-               upper="${safety['upper_limit']}"/>
-        <safety_controller soft_lower_limit="${safety['lower_limit'] + safety['lower_soft_buffer']}"
-                   soft_upper_limit="${safety['upper_limit'] - safety['upper_soft_buffer']}"
-                   k_position="${safety['k_position']}"
-                   k_velocity="${safety['k_velocity']}" />
+    <xacro:macro name="safety_limits" params="safety limits">
+        <limit velocity="${safety['max_velocity']}"
+               effort="${safety['max_effort']}"
+               lower="${limits['lower_limit']*pi/180}"
+               upper="${limits['upper_limit']*pi/180}"/>
+        <safety_controller
+                soft_lower_limit="${limits['lower_limit']*pi/180 + safety['lower_soft_buffer']*pi/180}"
+                soft_upper_limit="${limits['upper_limit']*pi/180 - safety['upper_soft_buffer']*pi/180}"
+                k_position="${safety['k_position']}"
+                k_velocity="${safety['k_velocity']}" />
     </xacro:macro>
 </robot>
