Commit message: Large xacro refactor, replacing all joints and pressure soles with macros, moving safety to yaml

File: ros2/src/shared/march_description/urdf/march4.xacro (robot description, xacro)
@@ -25,58 +25,22 @@
         </gazebo>
     </xacro:if>
+    <xacro:arg name="configuration" default="exoskeleton"/>
+    <xacro:property name="configuration" value="$(arg configuration)"/>
 <!-- Include all macro files    -->
+    <xacro:include filename="macros/safety_limits.xacro" />
     <xacro:include filename="macros/pressure_sole.xacro"/>
     <xacro:include filename="macros/frame_part.xacro"/>
-    <xacro:include filename="macros/rotational_joint.xacro"/>
-<!-- Add yaml file with inertia properties -->
-    <xacro:property name="yaml_file" value="properties/inertia_march4.yaml"/>
-    <xacro:property name="all_inertias" value="${load_yaml(yaml_file)}"/>
-    <xacro:property name="hip_aa_Ixx" value="0.013"/>
-    <xacro:property name="hip_aa_Ixy" value="0.008"/>
-    <xacro:property name="hip_aa_Ixz" value="0.005"/>
-    <xacro:property name="hip_aa_Iyy" value="0.023"/>
-    <xacro:property name="hip_aa_Iyz" value="-0.001"/>
-    <xacro:property name="hip_aa_Izz" value="0.028"/>
-    <xacro:property name="upper_leg_Ixx" value="0.127"/>
-    <xacro:property name="upper_leg_Ixy" value="0.0001291"/>
-    <xacro:property name="upper_leg_Ixz" value="-0.0002056"/>
-    <xacro:property name="upper_leg_Iyy" value="0.122"/>
-    <xacro:property name="upper_leg_Iyz" value="0.016"/>
-    <xacro:property name="upper_leg_Izz" value="0.015"/>
-    <xacro:property name="lower_leg_Ixx" value="0.075"/>
-    <xacro:property name="lower_leg_Ixy" value="-0.027"/>
-    <xacro:property name="lower_leg_Ixz" value="-0.008"/>
-    <xacro:property name="lower_leg_Iyy" value="0.11"/>
-    <xacro:property name="lower_leg_Iyz" value="-0.002"/>
-    <xacro:property name="lower_leg_Izz" value="0.071" />
-    <xacro:property name="foot_Ixx" value="0.021"/>
-    <xacro:property name="foot_Ixy" value="-0.002"/>
-    <xacro:property name="foot_Ixz" value="0.02"/>
-    <xacro:property name="foot_Iyy" value="0.027"/>
-    <xacro:property name="foot_Iyz" value="0.004"/>
-    <xacro:property name="foot_Izz" value="0.01" />
-    <!-- The max effort of the rotary joints is lower then the value corresponding to 25A, because short-circuit errors
-    have occured while applying the theoretical max effort for a long time. -->
-    <xacro:arg name="max_effort_rotary" default="18000.0" />
-    <xacro:arg name="max_effort_linear" default="22932.0" />  <!-- = 28 A -->
-    <xacro:property name="max_effort_rotary" value="$(arg max_effort_rotary)" />
-    <xacro:property name="max_effort_linear" value="$(arg max_effort_linear)" />
-    <!-- Values for the safety limits, see https://wiki.ros.org/pr2_controller_manager/safety_limits -->
-    <xacro:arg name="k_velocity_value_hfe" default="20000.0" />
-    <xacro:arg name="k_velocity_value_kfe" default="20000.0" />
-    <xacro:arg name="k_velocity_value_haa" default="20000.0" />
-    <xacro:arg name="k_velocity_value_adpf" default="20000.0" />
-    <xacro:property name="k_velocity_value_hfe" value="$(arg k_velocity_value_hfe)" />
-    <xacro:property name="k_velocity_value_kfe" value="$(arg k_velocity_value_kfe)" />
-    <xacro:property name="k_velocity_value_haa" value="$(arg k_velocity_value_haa)" />
-    <xacro:property name="k_velocity_value_adpf" value="$(arg k_velocity_value_adpf)" />
-    <xacro:arg name="k_position_value_hfe" default="14.88" />
-    <xacro:arg name="k_position_value_kfe" default="14.88" />
-    <xacro:arg name="k_position_value_haa" default="4.0" />
-    <xacro:arg name="k_position_value_adpf" default="5.0" />
-    <xacro:property name="k_position_value_hfe" value="$(arg k_position_value_hfe)" />
-    <xacro:property name="k_position_value_kfe" value="$(arg k_position_value_kfe)" />
-    <xacro:property name="k_position_value_haa" value="$(arg k_position_value_haa)" />
-    <xacro:property name="k_position_value_adpf" value="$(arg k_position_value_adpf)" />
+    <xacro:include filename="macros/joint.xacro"/>
+<!-- Add yaml files with properties -->
+    <xacro:property name="joint_limits_yaml_file" value="properties/march4_joint_limits.yaml"/>
+    <xacro:property name="joint_limits" value="${load_yaml(joint_limits_yaml_file)}"/>
+    <xacro:property name="safety_yaml_file" value="properties/march4_safety_${configuration}.yaml"/>
+    <xacro:property name="safety_values" value="${load_yaml(safety_yaml_file)}"/>
+    <xacro:property name="inertia_yaml_file" value="properties/march4_inertia.yaml"/>
+    <xacro:property name="inertia" value="${load_yaml(inertia_yaml_file)}"/>
+    <xacro:property name="dimensions_yaml_file" value="properties/march4_dimensions.yaml"/>
+    <xacro:property name="dimensions" value="${load_yaml(dimensions_yaml_file)}"/>
+    <xacro:property name="rotary_reduction" value="101"/>
+    <xacro:property name="linear_reduction" value="200"/>
     <!-- Constants for robot dimensions -->
     <!-- Masses determined in Catia, see https://confluence.projectmarch.nl:8443/display/51/URDF+description -->
@@ -122,5 +86,5 @@
 <!-- CHECKED BASED ON LEFT HIP AA< VERIFY RIGHT IS SAME!!    -->
     <xacro:property name="left_hip_aa_com" value="${hip_aa_com_x} ${-hip_aa_com_y} ${hip_aa_com_z}"/>
-    <xacro:property name="right_hip_aa_com" value="${hip_aa_com_x} ${hip_aa_com_y} ${hip_aa_com_z}"/>
+    <xacro:property name="hip_aa_com" value="${hip_aa_com_x} ${hip_aa_com_y} ${hip_aa_com_z}"/>
     <xacro:property name="upper_leg_com_x" value="0.000709"/>
     <xacro:property name="upper_leg_com_y" value="${-hip_base_height/2 - hip_aa_frame_height +
@@ -140,44 +104,4 @@
     <xacro:property name="foot_com_z" value="${upper_leg_height + lower_leg_height + ankle_plate_height - 0.789788}"/>
     <xacro:property name="foot_scale" value="1.35"/>
-    <!-- Inertia of the parts -->
-    <!-- Inertia's have been determined in Catia, see
-         https://confluence.projectmarch.nl:8443/display/51/URDF+description -->
-    <!-- The inertia's were defined around the CoM. Note that in the Catia x axis is the URDF y axis and the Catia y
-         axis is the negative URDF x axis, see confluence for the impact. The given inertia's are for the right leg,
-         Ixy and Iyz will be inverted for the left leg. -->
-    <!-- Joint properties -->
-    <!-- For limit calculations, see https://confluence.projectmarch.nl:8443/pages/viewpage.action?pageId=268697604 -->
-    <xacro:property name="left_hip_fe_rotation_lower_limit" value="${-21.04431152*pi/180}"/> <!-- rad -->
-    <xacro:property name="left_hip_fe_rotation_upper_limit" value="${98.97033691*pi/180}"/> <!-- rad -->
-    <xacro:property name="right_hip_fe_rotation_lower_limit" value="${-20.23406982*pi/180}"/> <!-- rad -->
-    <xacro:property name="right_hip_fe_rotation_upper_limit" value="${99.48120117*pi/180}"/> <!-- rad -->
-    <xacro:property name="hip_fe_soft_buffer" value="${3*pi/180}"/> <!-- rad -->
-    <xacro:property name="hip_fe_effort_limit" value="${max_effort_rotary}"/> <!-- IU -->
-    <xacro:property name="hip_fe_velocity_limit" value="2.0"/> <!-- rad/s -->
-    <xacro:property name="left_hip_aa_rotation_lower_limit" value="${-18.54492188*pi/180}"/> <!-- rad -->
-    <xacro:property name="left_hip_aa_rotation_upper_limit" value="${16.34765625*pi/180}"/> <!-- rad -->
-    <xacro:property name="right_hip_aa_rotation_lower_limit" value="${-18.10546875*pi/180}"/> <!-- rad -->
-    <xacro:property name="right_hip_aa_rotation_upper_limit" value="${15.99609375*pi/180}"/> <!-- rad -->
-    <xacro:property name="hip_aa_soft_buffer" value="${3.5*pi/180}"/> <!-- rad -->
-    <xacro:property name="hip_aa_effort_limit" value="${max_effort_linear}"/> <!-- IU -->
-    <xacro:property name="hip_aa_velocity_limit" value="1.0"/> <!-- rad/s -->
-    <xacro:property name="left_knee_rotation_lower_limit" value="${-5.012512207*pi/180}"/>
-    <xacro:property name="left_knee_rotation_upper_limit" value="${112.4230957*pi/180}"/>
-    <xacro:property name="right_knee_rotation_lower_limit" value="${-4.89440918*pi/180}"/>
-    <xacro:property name="right_knee_rotation_upper_limit" value="${115.3097534*pi/180}"/>
-    <xacro:property name="knee_extension_soft_buffer" value="${3.5*pi/180}"/> <!-- rad -->
-    <xacro:property name="knee_flexion_soft_buffer" value="${3*pi/180}"/> <!-- rad -->
-    <xacro:property name="knee_effort_limit" value="${max_effort_rotary}"/> <!-- IU -->
-    <xacro:property name="knee_velocity_limit" value="2.5"/>
-    <xacro:property name="left_ankle_rotation_lower_limit" value="${-26.30401611*pi/180}"/>
-    <xacro:property name="left_ankle_rotation_upper_limit" value="${15.88348389*pi/180}"/>
-    <xacro:property name="right_ankle_rotation_lower_limit" value="${-23.203125*pi/180}"/>
-    <xacro:property name="right_ankle_rotation_upper_limit" value="${14.23828125*pi/180}"/>
-    <xacro:property name="ankle_dorsalflexion_soft_buffer" value="${5*pi/180}"/> <!-- rad -->
-    <xacro:property name="ankle_plantarflexion_soft_buffer" value="${3*pi/180}"/> <!-- rad -->
-    <xacro:property name="ankle_effort_limit" value="${max_effort_linear}"/> <!-- IU -->
-    <xacro:property name="ankle_velocity_limit" value="1.0"/>
-    <xacro:property name="camera_link" value="0.05"/> <!-- Size of square 'camera' box -->
-    <xacro:property name="axel_offset" value="0.05"/> <!-- Space btw top of beam and the each joint -->
     <!-- Import all Gazebo-customization elements, including Gazebo colors -->
     <xacro:include filename="march.gazebo"/>
@@ -192,5 +116,4 @@
                       side="right"
                       length="${hip_base_height}"
-                      width="${width}"
                       direction="y"
                       visual_origin="${-hip_aa_frame_width} 0 0"
@@ -199,5 +122,5 @@
                       com="${hip_base_com}"
                       mass="${hip_base_mass}"
-                      inertia="${all_inertias['hip_base']}"
+                      inertia="${inertia['hip_base']}"
     />
     <!-- IMU-->
@@ -207,5 +130,4 @@
                       side="left"
                       length="${hip_aa_frame_height}"
-                      width="${width}"
                       direction="y"
                       visual_origin="${-hip_aa_frame_width} ${hip_base_height/2} 0"
@@ -216,15 +138,13 @@
                       side="left"
                       length="${hip_aa_frame_width}"
-                      width="${width}"
                       direction="x"
                       collision_origin="${-hip_aa_frame_width/2} 0 0"
                       com="${left_hip_aa_com}"
                       mass="${hip_aa_mass}"
-                      inertia="${all_inertias['hip_aa']}"
+                      inertia="${inertia['hip_aa']}"
                       />
     <xacro:frame_part name="upper_leg_left"
                       side="left"
                       length="${upper_leg_height}"
-                      width="${width}"
                       direction="z"
                       collision_origin="0 0 ${-upper_leg_height/2}"
@@ -233,10 +153,9 @@
                       com="${left_upper_leg_com}"
                       mass="${upper_leg_mass}"
-                      inertia="${all_inertias['upper_leg']}"
+                      inertia="${inertia['upper_leg']}"
                     />
     <xacro:frame_part name="lower_leg_left"
                       side="left"
                       length="${lower_leg_height}"
-                      width="${width}"
                       direction="z"
                       collision_origin="0 0 ${-lower_leg_height/2}"
@@ -245,10 +164,9 @@
                       com="${left_lower_leg_com}"
                       mass="${lower_leg_mass}"
-                      inertia="${all_inertias['lower_leg']}"
+                      inertia="${inertia['lower_leg']}"
                       />
     <xacro:frame_part name="ankle_plate_left"
                       side="left"
                       length="${ankle_plate_height}"
-                      width="${width}"
                       direction="z"
                       mesh="LeftFoot.stl"
@@ -256,36 +174,15 @@
                                      ${hip_base_height/2 + hip_aa_frame_height - upper_leg_offset - ankle_plate_offset}
                                      ${foot_scale * (upper_leg_height + lower_leg_height)}"
+                      scale="1 1 ${foot_scale}"
                       collision_origin="0 0 ${-ankle_plate_height/2}"
     />
-    <xacro:pressure_sole side="left" parent="ankle_plate_left"/>
     <xacro:frame_part name="foot_left"
                       side="left"
                       length="${foot_height_forward+foot_height_backward}"
-                      width="${width}"
                       direction="x"
-                      inertia="${all_inertias['foot']}"
+                      inertia="${inertia['foot']}"
                       collision_origin="${(-foot_height_forward+foot_height_backward)/2} 0 0"
                       com="${foot_com_x} ${-foot_com_y} ${foot_com_z}"
                       mass="${foot_mass}"/>
-    <link name="pressure_sole_left">
-        <collision>
-            <origin xyz="${(-foot_height_forward+foot_height_backward)/2} 0 0" rpy="0 0 0"/>
-            <geometry>
-                <box size="${foot_height_forward+foot_height_backward} ${width} 0.001"/>
-            </geometry>
-        </collision>
-    </link>
-    <gazebo reference="pressure_sole_left">
-        <sensor name="left_pressure_sole" type="contact">
-            <always_on>true</always_on>
-            <contact>
-                <collision>ankle_plate_left_fixed_joint_lump__pressure_sole_left_collision_2</collision>
-            </contact>
-            <plugin name="left_foot_plugin" filename="libgazebo_ros_bumper.so">
-                <bumperTopicName>march/sensor/left_pressure_sole</bumperTopicName>
-                <frameName>world</frameName>
-            </plugin>
-        </sensor>
-    </gazebo>
     <gazebo reference="foot_left">
         <mu1>${foot_mu1}</mu1>
@@ -294,4 +191,5 @@
         <fdir1>1 0 0</fdir1>
     </gazebo>
+    <xacro:pressure_sole side="left" foot_name="foot_left"/>
     <xacro:frame_part name="hip_aa_frame_right_side"
                       side="right"
@@ -303,15 +201,15 @@
     />
     <xacro:frame_part name="hip_aa_frame_right_front"
-                      width="${width}"
                       length="${hip_aa_frame_width}"
+                      direction="x"
                       collision_origin="${-hip_aa_frame_width/2} 0 0"
                       side="right"
                       com="${hip_aa_com_x} ${hip_aa_com_y} ${hip_aa_com_z}"
                       mass="${hip_aa_mass}"
-                      inertia="${all_inertias['hip_aa']}"
+                      inertia="${inertia['hip_aa']}"
     />
     <xacro:frame_part name="upper_leg_right"
                       side="right"
-                      width="${width}"
+                      direction="z"
                       length="${upper_leg_height}"
                       collision_origin="0 0 ${-upper_leg_height/2}"
@@ -319,5 +217,5 @@
                       mesh="UpperRightLeg.stl"
                       com="${upper_leg_com_x} ${upper_leg_com_y} ${upper_leg_com_z}"
-                      inertia="${all_inertias['upper_leg']}"
+                      inertia="${inertia['upper_leg']}"
                       mass="${upper_leg_mass}"
     />
@@ -325,67 +223,33 @@
                       side="right"
                       length="${lower_leg_height}"
-                      width="${width}"
+                      direction="z"
                       visual_origin="0 ${-hip_base_height/2 - hip_aa_frame_height + upper_leg_offset} ${upper_leg_height}"
                       mesh="LowerRightLeg.stl"
                       com="${lower_leg_com_x} ${lower_leg_com_y} ${lower_leg_com_z}"
                       mass="${lower_leg_mass}"
-                      inertia="${all_inertias['lower_leg']}"
+                      inertia="${inertia['lower_leg']}"
                       collision_origin="0 0 ${-lower_leg_height/2}"
     />
-    <!-- Ankle Plate Right -->
-    <link name="ankle_plate_right">
-        <visual>
-            <origin
-                    xyz="0
-                    ${-hip_base_height/2 - hip_aa_frame_height+ upper_leg_offset + ankle_plate_offset}
-                    ${foot_scale * (upper_leg_height + lower_leg_height)}"
-                    rpy="0 0 ${pi}"/>
-            />
-            <geometry>
-                <mesh filename="package://march_description/urdf/stl-files/RightFoot.stl" scale="1 1 ${foot_scale}"/>
-            </geometry>
-            <material name="blue"/>
-        </visual>
-        <collision>
-            <origin xyz="0 0 ${-ankle_plate_height/2}" rpy="0 0 0"/>
-            <geometry>
-                <box size="${width} ${width} ${ankle_plate_height}"/>
-            </geometry>
-        </collision>
-    </link>
-<<<<<<< HEAD
-    <gazebo reference="ankle_plate_right">
-        <sensor name="ankle_plate_right_contact" type="contact">
-            <plugin name="contact_plugin" filename="libcontact.so"/>
-            <contact>
-                <collision>ankle_plate_right_fixed_joint_lump__foot_right_collision_1</collision>
-            </contact>
-            <update_rate>30</update_rate>
-            <always_on>true</always_on>
-        </sensor>
-    </gazebo>
-=======
-    <xacro:pressure_sole side="right" parent="ankle_plate_right"/>
->>>>>>> ab2ac4d3... Split frame using a macro
+    <xacro:frame_part name="ankle_plate_right"
+                      side="right"
+                      length="${ankle_plate_height}"
+                      direction="z"
+                      mesh="RightFoot.stl"
+                      visual_origin="0
+                                     ${-hip_base_height/2 - hip_aa_frame_height + upper_leg_offset + ankle_plate_offset}
+                                     ${foot_scale * (upper_leg_height + lower_leg_height)}"
+                      collision_origin="0 0 ${-ankle_plate_height/2}"
+                      scale="1 1 ${foot_scale}"
+    />
     <!-- Foot Right -->
-    <link name="foot_right">
-        <inertial>
-            <origin xyz="${foot_com_x} ${foot_com_y} ${foot_com_z}" rpy="0 0 0"/>
-            <mass value="${foot_mass}"/>
-            <inertia
-                    ixx="${foot_Ixx}"
-                    ixy="${foot_Ixy}"
-                    ixz="${foot_Ixz}"
-                    iyy="${foot_Iyy}"
-                    iyz="${foot_Iyz}"
-                    izz="${foot_Izz}" />
-        </inertial>
-        <collision>
-            <origin xyz="${(-foot_height_forward+foot_height_backward)/2} 0 0" rpy="0 0 0"/>
-            <geometry>
-                <box size="${foot_height_forward+foot_height_backward} ${width} ${width}"/>
-            </geometry>
-        </collision>
-    </link>
+    <xacro:pressure_sole side="right" foot_name="foot_right"/>
+    <xacro:frame_part name="foot_right"
+                      side="right"
+                      length="${foot_height_forward+foot_height_backward}"
+                      direction="x"
+                      inertia="${inertia['foot']}"
+                      collision_origin="${(-foot_height_forward+foot_height_backward)/2} 0 0"
+                      com="${foot_com_x} ${foot_com_y} ${foot_com_z}"
+                      mass="${foot_mass}"/>
     <gazebo reference="foot_right">
         <mu1>${foot_mu1}</mu1>
@@ -394,24 +258,4 @@
         <fdir1>1 0 0</fdir1>
     </gazebo>
-    <link name="pressure_sole_right">
-        <collision>
-            <origin xyz="${(-foot_height_forward+foot_height_backward)/2} 0 0" rpy="0 0 0"/>
-            <geometry>
-                <box size="${foot_height_forward+foot_height_backward} ${width} 0.001"/>
-            </geometry>
-        </collision>
-    </link>
-    <gazebo reference="pressure_sole_right">
-        <sensor name="right_pressure_sole" type="contact">
-            <always_on>true</always_on>
-            <contact>
-                <collision>ankle_plate_right_fixed_joint_lump__pressure_sole_right_collision_2</collision>
-            </contact>
-            <plugin name="right_foot_plugin" filename="libgazebo_ros_bumper.so">
-                <bumperTopicName>march/sensor/right_pressure_sole</bumperTopicName>
-                <frameName>world</frameName>
-            </plugin>
-        </sensor>
-    </gazebo>
     <!-- Joints -->
     <joint name="imu_joint" type="fixed">
@@ -424,18 +268,14 @@
         <origin xyz="0 0 ${lower_leg_height+upper_leg_height+ankle_plate_height+width/2.0+hover_height}" rpy="0 0 0"/>
     </joint>
-    <joint name="left_hip_aa" type="revolute">
-        <parent link="hip_base"/>
-        <child link="hip_aa_frame_left_side"/>
-        <origin xyz="0 ${-hip_base_height/2} 0" rpy="0 0 0"/>
-        <axis xyz="-1 0 0"/>
-        <limit velocity="${hip_aa_velocity_limit}"
-               effort="${hip_aa_effort_limit}"
-               lower="${left_hip_aa_rotation_lower_limit}"
-               upper="${left_hip_aa_rotation_upper_limit}"/>
-        <safety_controller soft_lower_limit="${left_hip_aa_rotation_lower_limit + hip_aa_soft_buffer}"
-                           soft_upper_limit="${left_hip_aa_rotation_upper_limit - hip_aa_soft_buffer}"
-                           k_position="${k_position_value_haa}"
-                           k_velocity="${k_velocity_value_haa}" />
-    </joint>
+    <xacro:march_joint
+        name="left_hip_aa"
+        parent="hip_base"
+        child="hip_aa_frame_left_side"
+        origin="0 ${-hip_base_height/2} 0"
+        axis="-1 0 0"
+        safety="${safety_values['haa']}"
+        limits="${joint_limits['left_haa']}"
+        reduction="${linear_reduction}"
+    />
     <joint name="left_hip_angle" type="fixed">
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