Commit message: Large xacro refactor, replacing all joints and pressure soles with macros, moving safety to yaml

File: ros2/src/shared/march_description/urdf/march4_old.xacro (robot description, xacro)
@@ -583,4 +583,13 @@
                            k_velocity="${k_velocity_value_hfe}" />
     </joint>
+    <transmission name="left_hip_fe">
+        <type>transmission_interface/SimpleTransmission</type>
+        <joint name="left_hip_fe">
+            <hardwareInterface>hardware_interface/EffortJointInterface</hardwareInterface>
+        </joint>
+        <actuator name="left_hip_fe_motor">
+            <mechanicalReduction>101</mechanicalReduction>
+        </actuator>
+    </transmission>
     <joint name="left_knee" type="revolute">
         <parent link= "upper_leg_left"/>
@@ -597,4 +606,13 @@
                            k_velocity="${k_velocity_value_kfe}" />
     </joint>
+    <transmission name="left_knee">
+        <type>transmission_interface/SimpleTransmission</type>
+        <joint name="left_knee">
+            <hardwareInterface>hardware_interface/EffortJointInterface</hardwareInterface>
+        </joint>
+        <actuator name="left_knee_motor">
+            <mechanicalReduction>101</mechanicalReduction>
+        </actuator>
+    </transmission>
     <joint name="left_ankle" type="revolute">
         <parent link="lower_leg_left"/>
@@ -659,4 +677,13 @@
                            k_velocity="${k_velocity_value_hfe}" />
     </joint>
+    <transmission name="right_hip_fe">
+        <type>transmission_interface/SimpleTransmission</type>
+        <joint name="right_hip_fe">
+            <hardwareInterface>hardware_interface/EffortJointInterface</hardwareInterface>
+        </joint>
+        <actuator name="right_hip_fe_motor">
+            <mechanicalReduction>101</mechanicalReduction>
+        </actuator>
+    </transmission>
     <joint name="right_knee" type="revolute">
         <parent link="upper_leg_right"/>
@@ -673,4 +700,13 @@
                            k_velocity="${k_velocity_value_kfe}" />
     </joint>
+    <transmission name="right_knee">
+        <type>transmission_interface/SimpleTransmission</type>
+        <joint name="right_knee">
+            <hardwareInterface>hardware_interface/EffortJointInterface</hardwareInterface>
+        </joint>
+        <actuator name="right_knee_motor">
+            <mechanicalReduction>101</mechanicalReduction>
+        </actuator>
+    </transmission>
     <joint name="right_ankle" type="revolute">
         <parent link="lower_leg_right"/>
@@ -700,22 +736,4 @@
         <actuator name="left_hip_aa_motor">
             <mechanicalReduction>200</mechanicalReduction>
-        </actuator>
-    </transmission>
-    <transmission name="left_hip_fe">
-        <type>transmission_interface/SimpleTransmission</type>
-        <joint name="left_hip_fe">
-            <hardwareInterface>hardware_interface/EffortJointInterface</hardwareInterface>
-        </joint>
-        <actuator name="left_hip_fe_motor">
-            <mechanicalReduction>101</mechanicalReduction>
-        </actuator>
-    </transmission>
-    <transmission name="left_knee">
-        <type>transmission_interface/SimpleTransmission</type>
-        <joint name="left_knee">
-            <hardwareInterface>hardware_interface/EffortJointInterface</hardwareInterface>
-        </joint>
-        <actuator name="left_knee_motor">
-            <mechanicalReduction>101</mechanicalReduction>
         </actuator>
     </transmission>
@@ -738,22 +756,4 @@
         </actuator>
     </transmission>
-    <transmission name="right_hip_fe">
-        <type>transmission_interface/SimpleTransmission</type>
-        <joint name="right_hip_fe">
-            <hardwareInterface>hardware_interface/EffortJointInterface</hardwareInterface>
-        </joint>
-        <actuator name="right_hip_fe_motor">
-            <mechanicalReduction>101</mechanicalReduction>
-        </actuator>
-    </transmission>
-    <transmission name="right_knee">
-        <type>transmission_interface/SimpleTransmission</type>
-        <joint name="right_knee">
-            <hardwareInterface>hardware_interface/EffortJointInterface</hardwareInterface>
-        </joint>
-        <actuator name="right_knee_motor">
-            <mechanicalReduction>101</mechanicalReduction>
-        </actuator>
-    </transmission>
     <transmission name="right_ankle">
         <type>transmission_interface/SimpleTransmission</type>

Commit message: Last changes before Christmas break, a start to move dimensions to yaml file and attempt to change collision origin for feet to standard middle

File: ros2/src/shared/march_description/urdf/macros/frame_part.xacro (robot description, xacro)
@@ -2,15 +2,18 @@
 <robot  xmlns:xacro="http://www.ros.org/wiki/xacro">
     <xacro:macro name="frame_part"
-                 params="name side length direction collision_origin visual_origin:=0 mesh:=0 com:=0 mass:=0 inertia:=0 scale:='1 1 1'">
+                 params="name reflect length direction collision_origin visual_origin:=0 mesh:=0 com:=0 mass:=0 inertia:=0 scale:='1 1 1'">
         <xacro:if value="${direction == 'x'}">
             <xacro:property name="size" value="${length} ${width} ${width}"/>
+<!--            <xacro:property name="collision_origin" value="${-length/2} ${width} ${width}"/>-->
             <xacro:property name="rpy" value="0 0 0"/>
         </xacro:if>
         <xacro:if value="${direction == 'y'}">
             <xacro:property name="size" value="${width} ${length} ${width}"/>
+<!--            <xacro:property name="collision_origin" value="${-length/2} ${width} ${width}"/>-->
             <xacro:property name="rpy" value="0 0 ${pi}"/>
         </xacro:if>
         <xacro:if value="${direction == 'z'}">
             <xacro:property name="size" value="${width} ${width} ${length}"/>
+<!--            <xacro:property name="collision_origin" value="${-length/2} ${width} ${width}"/>-->
             <xacro:property name="rpy" value="0 0 ${pi}"/>
         </xacro:if>
@@ -29,22 +32,11 @@
                     <origin xyz="${com}" rpy="0 0 0"/>
                     <mass value="${mass}"/>
-                    <xacro:if value="${side == 'right'}">
-                        <inertia
-                                ixx="${inertia['xx']}"
-                                ixy="${inertia['xy']}"
-                                ixz="${inertia['xz']}"
-                                iyy="${inertia['yy']}"
-                                iyz="${inertia['yz']}"
-                                izz="${inertia['zz']}" />
-                    </xacro:if>
-                    <xacro:if value="${side == 'left'}">
-                        <inertia
-                                ixx="${inertia['xx']}"
-                                ixy="${-inertia['xy']}"
-                                ixz="${inertia['xz']}"
-                                iyy="${inertia['yy']}"
-                                iyz="${-inertia['yz']}"
-                                izz="${inertia['zz']}" />
-                    </xacro:if>
+                    <inertia
+                            ixx="${inertia['xx']}"
+                            ixy="${inertia['xy'] * reflect}"
+                            ixz="${inertia['xz']}"
+                            iyy="${inertia['yy']}"
+                            iyz="${inertia['yz'] * reflect}"
+                            izz="${inertia['zz']}" />
                 </inertial>
             </xacro:unless>
