Commit message: Add new visuals to march6 and use macros
Change colour

Update stl to lfs files

File: ros2/src/shared/march_description/urdf/macros/frame_part.xacro (robot description, xacro)
@@ -2,5 +2,5 @@
 <robot  xmlns:xacro="http://www.ros.org/wiki/xacro">
     <xacro:macro name="frame_part"
-                 params="name reflect length direction collision_origin visual_origin:=0 mesh:=0 com:=0 mass:=0 inertia:=0 scale:='1 1 1'">
+                 params="name reflect length direction collision_origin visual_origin:=0 visual_rpy:=0 mesh:=0 com:=0 mass:=0 inertia:=0 scale:='1 1 1'">
         <xacro:if value="${direction == 'x'}">
             <xacro:property name="size" value="${length} ${width} ${width}"/>
@@ -15,4 +15,7 @@
             <xacro:property name="rpy" value="0 0 ${pi}"/>
         </xacro:if>
+        <xacro:unless value="${visual_rpy == 0}">
+            <xacro:property name="rpy" value="${visual_rpy}"/>
+        </xacro:unless>
         <link name="${name}">
             <xacro:unless value="${visual_origin == 0}">

File: ros2/src/shared/march_description/urdf/march4.xacro (robot description, xacro)
@@ -47,23 +47,35 @@
     <xacro:property name="width"
                     value="0.05"/> <!-- Square dimensions (widthxwidth) of beams -->
-    <xacro:property name="hip_base_height" value="0.160"/>
-    <xacro:property name="hip_base_mass" value="8.686"/>
+    <xacro:property name="hip_base_height" value="${dimensions['hip_base']['length']}"/>
+    <xacro:property name="hip_base_mass" value="${dimensions['hip_base']['mass']}"/>
     <!-- mass = Hip base + HAA actuators -->
-    <xacro:property name="hip_aa_frame_height" value="0.170"/>
-    <xacro:property name="hip_aa_frame_width" value="0.1395"/>
-    <xacro:property name="hip_aa_mass" value="2.982"/>
+    <xacro:property name="hip_aa_frame_height"
+                    value="${dimensions['hip_aa_side']['length']}"/>
+    <xacro:property name="hip_aa_frame_width"
+                    value="${dimensions['hip_aa_base']['length']}"/>
+    <xacro:property name="hip_aa_mass" value="${dimensions['hip_aa_side']['mass']}"/>
     <!-- mass = Moving hip -->
-    <xacro:property name="upper_leg_height" value="0.385"/>
-    <xacro:property name="upper_leg_offset" value="0.04"/>
-    <xacro:property name="upper_leg_mass" value="4.995"/>
+    <xacro:property name="upper_leg_height"
+                    value="${dimensions['upper_leg']['length']}"/>
+    <xacro:property name="upper_leg_offset"
+                    value="${dimensions['upper_leg']['offset']}"/>
+    <xacro:property name="upper_leg_mass"
+                    value="${dimensions['upper_leg']['mass']}"/>
     <!-- mass = KFE joint + HFE joint + Upper leg -->
-    <xacro:property name="lower_leg_height" value="0.385"/>
-    <xacro:property name="lower_leg_mass" value="4.458"/>
+    <xacro:property name="lower_leg_height"
+                    value="${dimensions['lower_leg']['length']}"/>
+    <xacro:property name="lower_leg_mass"
+                    value="${dimensions['lower_leg']['mass']}"/>
     <!-- mass = Ankle actuator + Lower leg -->
-    <xacro:property name="ankle_plate_height" value="0.12"/>
-    <xacro:property name="ankle_plate_offset" value="0.07"/>
-    <xacro:property name="foot_height_forward" value="${0.184}"/>
-    <xacro:property name="foot_height_backward" value="${0.059}"/>
-    <xacro:property name="foot_mass" value="1.821"/>
+    <xacro:property name="ankle_plate_height"
+                    value="${dimensions['ankle_plate']['length']}"/>
+    <xacro:property name="ankle_plate_offset"
+                    value="${dimensions['ankle_plate']['offset']}"/>
+    <xacro:property name="foot_height_forward"
+                    value="${dimensions['foot']['height_forward']}"/>
+    <xacro:property name="foot_height_backward"
+                    value="${dimensions['foot']['height_backward']}"/>
+    <xacro:property name="foot_mass"
+                    value="${dimensions['foot']['mass']}"/>
     <xacro:property name="foot_mu1" value="1"/>
     <xacro:property name="foot_mu2" value="1"/>
@@ -114,7 +126,7 @@
                       visual_origin="${-hip_aa_frame_width} 0 0"
                       collision_origin="0 0 0"
-                      mesh="HipBase.stl"
+                      mesh="march4/HipBase.stl"
                       com="${hip_base_com_x} ${hip_base_com_y} ${hip_base_com_z}"
-                      mass="${hip_base_mass}"
+                      mass="${dimensions['hip_base']['mass']}"
                       inertia="${inertia['hip_base']}"
     />
@@ -128,5 +140,5 @@
                       collision_origin="0 ${-hip_aa_frame_height/2} 0"
                       visual_origin="${-hip_aa_frame_width} ${hip_base_height/2} 0"
-                      mesh="LeftHAA.stl"
+                      mesh="march4/LeftHAA.stl"
     />
     <xacro:frame_part name="hip_aa_frame_left_front"
@@ -145,5 +157,5 @@
                       collision_origin="0 0 ${-upper_leg_height/2}"
                       visual_origin="0 ${hip_base_height/2 + hip_aa_frame_height - upper_leg_offset} 0"
-                      mesh="UpperLeftLeg.stl"
+                      mesh="march4/UpperLeftLeg.stl"
                       com="${upper_leg_com_x} ${-upper_leg_com_y} ${upper_leg_com_z}"
                       mass="${upper_leg_mass}"
@@ -156,5 +168,5 @@
                       collision_origin="0 0 ${-lower_leg_height/2}"
                       visual_origin="0 ${hip_base_height/2 + hip_aa_frame_height - upper_leg_offset} ${upper_leg_height}"
-                      mesh="LowerLeftLeg.stl"
+                      mesh="march4/LowerLeftLeg.stl"
                       com="${lower_leg_com_x} ${-lower_leg_com_y} ${lower_leg_com_z}"
                       mass="${lower_leg_mass}"
@@ -165,5 +177,5 @@
                       length="${ankle_plate_height}"
                       direction="z"
-                      mesh="LeftFoot.stl"
+                      mesh="march4/LeftFoot.stl"
                       visual_origin="0
                                      ${hip_base_height/2 + hip_aa_frame_height - upper_leg_offset - ankle_plate_offset}
@@ -193,5 +205,5 @@
                       visual_origin="${-hip_aa_frame_width} ${-hip_base_height/2} 0"
                       collision_origin="0 ${hip_aa_frame_height/2} 0"
-                      mesh="RightHAA.stl"
+                      mesh="march4/RightHAA.stl"
     />
     <xacro:frame_part name="hip_aa_frame_right_front"
@@ -210,5 +222,5 @@
                       collision_origin="0 0 ${-upper_leg_height/2}"
                       visual_origin="0 ${-hip_base_height/2 - hip_aa_frame_height + upper_leg_offset} 0"
-                      mesh="UpperRightLeg.stl"
+                      mesh="march4/UpperRightLeg.stl"
                       com="${upper_leg_com_x} ${upper_leg_com_y} ${upper_leg_com_z}"
                       inertia="${inertia['upper_leg']}"
@@ -220,5 +232,5 @@
                       direction="z"
                       visual_origin="0 ${-hip_base_height/2 - hip_aa_frame_height + upper_leg_offset} ${upper_leg_height}"
-                      mesh="LowerRightLeg.stl"
+                      mesh="march4/LowerRightLeg.stl"
                       com="${lower_leg_com_x} ${lower_leg_com_y} ${lower_leg_com_z}"
                       mass="${lower_leg_mass}"
@@ -230,5 +242,5 @@
                       length="${ankle_plate_height}"
                       direction="z"
-                      mesh="RightFoot.stl"
+                      mesh="march4/RightFoot.stl"
                       visual_origin="0
                                      ${-hip_base_height/2 - hip_aa_frame_height + upper_leg_offset + ankle_plate_offset}
