Commit message: Add new visuals to march6 and use macros
Change colour

Update stl to lfs files

File: ros2/src/shared/march_description/urdf/march6.xacro (robot description, xacro)
@@ -1,10 +1,3 @@
 <?xml version="1.0"?>
-<!--\________________________________________________________/-->
-<!--                                                          -->
-<!--                Fred Het Exoskelet                        -->
-<!--                                                          -->
-<!--\________________________________________________________/-->
-<!-- Up to date -->
-        <!-- lengths, meshes -->
 <!-- Revolute-Revolute Manipulator -->
 <robot name="march" xmlns:xacro="http://www.ros.org/wiki/xacro">
@@ -14,10 +7,10 @@
     the hover_height to 0.0. Set ground_gait to true to ground gait in simulation.-->
     <xacro:arg name="ground_gait" default="false"/>
-<!--    Switch between using the physical camera and the simulation camera -->
-<!--    If set to 'true', no physical camera is needed -->
-<!--    If this value is set to 'false', the plugin will not be started and the topics -->
-<!--    published by the real camera will be used. -->
-<!--    In both these situations the camera will still be visible and placed in the urdf,-->
-<!--    to be used for the transformations.-->
+    <!--    Switch between using the physical camera and the simulation camera -->
+    <!--    If set to 'true', no physical camera is needed -->
+    <!--    If this value is set to 'false', the plugin will not be started and the topics -->
+    <!--    published by the real camera will be used. -->
+    <!--    In both these situations the camera will still be visible and placed in the urdf,-->
+    <!--    to be used for the transformations.-->
     <xacro:arg name="realsense_simulation" default="false"/>
     <xacro:unless value="$(arg ground_gait)">
@@ -32,59 +25,64 @@
         </gazebo>
     </xacro:if>
-    <!-- TODO Change max efforts and velocity for the MARCH VI -->
-    <!-- The max effort of the rotary joints is lower then the value corresponding to 25A, because short-circuit errors
-    have occured while applying the theoretical max effort for a long time. -->
-    <xacro:arg name="max_effort_rotary" default="18000.0" /> <!-- TODO -->
-    <xacro:arg name="max_effort_linear" default="22932.0" />  <!-- = 28 A --> <!-- TODO -->
-    <xacro:property name="max_effort_rotary" value="$(arg max_effort_rotary)" /> <!-- TODO -->
-    <xacro:property name="max_effort_linear" value="$(arg max_effort_linear)" /> <!-- TODO -->
-    <!-- Values for the safety limits, see https://wiki.ros.org/pr2_controller_manager/safety_limits -->
-    <xacro:arg name="k_velocity_value_hfe" default="20000.0" /> <!-- TODO -->
-    <xacro:arg name="k_velocity_value_kfe" default="20000.0" /> <!-- TODO -->
-    <xacro:arg name="k_velocity_value_haa" default="20000.0" /> <!-- TODO -->
-    <xacro:arg name="k_velocity_value_adpf" default="20000.0" /> <!-- TODO -->
-    <xacro:property name="k_velocity_value_hfe" value="$(arg k_velocity_value_hfe)" /> <!-- TODO -->
-    <xacro:property name="k_velocity_value_kfe" value="$(arg k_velocity_value_kfe)" /> <!-- TODO -->
-    <xacro:property name="k_velocity_value_haa" value="$(arg k_velocity_value_haa)" /> <!-- TODO -->
-    <xacro:property name="k_velocity_value_adpf" value="$(arg k_velocity_value_adpf)" /> <!-- TODO -->
-    <xacro:arg name="k_position_value_hfe" default="14.88" /> <!-- TODO -->
-    <xacro:arg name="k_position_value_kfe" default="14.88" /> <!-- TODO -->
-    <xacro:arg name="k_position_value_haa" default="4.0" /> <!-- TODO -->
-    <xacro:arg name="k_position_value_adpf" default="5.0" /> <!-- TODO -->
-    <xacro:property name="k_position_value_hfe" value="$(arg k_position_value_hfe)" /> <!-- TODO -->
-    <xacro:property name="k_position_value_kfe" value="$(arg k_position_value_kfe)" /> <!-- TODO -->
-    <xacro:property name="k_position_value_haa" value="$(arg k_position_value_haa)" /> <!-- TODO -->
-    <xacro:property name="k_position_value_adpf" value="$(arg k_position_value_adpf)" /> <!-- TODO -->
+    <xacro:arg name="configuration" default="exoskeleton"/>
+    <xacro:property name="configuration" value="$(arg configuration)"/>
+    <!-- Include all macro files    -->
+    <xacro:include filename="macros/safety_limits.xacro"/>
+    <xacro:include filename="macros/pressure_sole.xacro"/>
+    <xacro:include filename="macros/frame_part.xacro"/>
+    <xacro:include filename="macros/joint.xacro"/>
+    <!-- Add yaml files with properties -->
+    <xacro:property name="config_yaml_file"
+                    value="properties/march6.yaml"/>
+    <xacro:property name="properties" value="${load_yaml(config_yaml_file)}"/>
+    <xacro:property name="joint_limits" value="${properties['joint_limits']}"/>
+    <xacro:property name="safety_values"
+                    value="${properties['safety'][configuration]}"/>
+    <xacro:property name="inertia" value="${properties['inertia']}"/>
+    <xacro:property name="dimensions" value="${properties['dimensions']}"/>
+    <xacro:property name="rotary_reduction" value="101"/>
+    <xacro:property name="linear_reduction" value="200"/>
     <!-- Constants for robot dimensions -->
-    <!-- TODO Change masses for the MARCH VI -->
     <!-- Masses determined in Catia, see https://confluence.projectmarch.nl:8443/display/51/URDF+description -->
-    <xacro:property name="width" value="0.05"/> <!-- Square dimensions (widthxwidth) of beams -->
-    <xacro:property name="hip_base_height" value="0.145"/>
-    <xacro:property name="hip_base_mass" value="8.686"/> <!-- TODO -->
+    <xacro:property name="width"
+                    value="0.05"/> <!-- Square dimensions (widthxwidth) of beams -->
+    <xacro:property name="hip_base_height" value="${dimensions['hip_base']['length']}"/>
+    <xacro:property name="hip_base_mass" value="${dimensions['hip_base']['mass']}"/>
     <!-- mass = Hip base + HAA actuators -->
-    <xacro:property name="hip_aa_frame_height" value="0.151"/>
-    <xacro:property name="hip_aa_frame_width" value="0.1605"/>
-    <xacro:property name="hip_aa_mass" value="2.982"/> <!-- TODO -->
+    <xacro:property name="hip_aa_frame_height"
+                    value="${dimensions['hip_aa_side']['length']}"/>
+    <xacro:property name="hip_aa_frame_width"
+                    value="${dimensions['hip_aa_base']['length']}"/>
+    <xacro:property name="hip_aa_mass" value="${dimensions['hip_aa_side']['mass']}"/>
     <!-- mass = Moving hip -->
-    <xacro:property name="upper_leg_height" value="0.410"/>
-    <xacro:property name="upper_leg_offset" value="0.04"/> <!-- TODO -->
-    <xacro:property name="upper_leg_mass" value="4.995"/> <!-- TODO -->
+    <xacro:property name="upper_leg_height"
+                    value="${dimensions['upper_leg']['length']}"/>
+    <xacro:property name="upper_leg_offset"
+                    value="${dimensions['upper_leg']['offset']}"/>
+    <xacro:property name="upper_leg_mass"
+                    value="${dimensions['upper_leg']['mass']}"/>
     <!-- mass = KFE joint + HFE joint + Upper leg -->
-    <xacro:property name="lower_leg_height" value="0.410"/>
-    <xacro:property name="lower_leg_mass" value="4.458"/> <!-- TODO -->
+    <xacro:property name="lower_leg_height"
+                    value="${dimensions['lower_leg']['length']}"/>
+    <xacro:property name="lower_leg_mass"
+                    value="${dimensions['lower_leg']['mass']}"/>
     <!-- mass = Ankle actuator + Lower leg -->
-    <xacro:property name="ankle_plate_height" value="0.14567"/>
-    <xacro:property name="ankle_plate_offset" value="0.07"/>
-    <xacro:property name="foot_height_forward" value="0.184"/>
-    <xacro:property name="foot_height_backward" value="0.059"/>
-    <xacro:property name="foot_mass" value="1.821"/> <!-- TODO -->
-    <xacro:property name="foot_mu1" value="1"/> <!-- TODO -->
-    <xacro:property name="foot_mu2" value="1"/> <!-- TODO -->
+    <xacro:property name="ankle_plate_height"
+                    value="${dimensions['ankle_plate']['length']}"/>
+    <xacro:property name="ankle_plate_offset"
+                    value="${dimensions['ankle_plate']['offset']}"/>
+    <xacro:property name="foot_height_forward"
+                    value="${dimensions['foot']['height_forward']}"/>
+    <xacro:property name="foot_height_backward"
+                    value="${dimensions['foot']['height_backward']}"/>
+    <xacro:property name="foot_mass"
+                    value="${dimensions['foot']['mass']}"/>
+    <xacro:property name="foot_mu1" value="1"/>
+    <xacro:property name="foot_mu2" value="1"/>
     <!-- Minimum allowable depth before contact correction impulse is applied. -->
     <xacro:property name="foot_min_depth" value="0.0005"/>
     <!-- mass = Passive ankle + foot -->
-    <!-- TODO Change center of masses for the MARCH VI -->
     <!-- Center of Mass (CoM) of the parts -->
-    <!-- CoM has been determined in Catia, see https://confluence.projectmarch.nl:8443/display/62tech/Exo+dimensions -->
+    <!-- CoM has been determined in Catia, see https://confluence.projectmarch.nl:8443/display/51/URDF+description -->
     <!-- The Catia locations were defined in a global coordinate system with the origin at the center of the
          rotation axis of the two HFE joints. Here, the joints were all set at zero degrees. Hence, we need some
@@ -92,99 +90,29 @@
          the URDF y axis and the Catia y axis is the negative URDF x axis. The given CoM are for the right leg,
          the y coordinate will be inverted for the left leg. -->
-    <xacro:property name="hip_base_com_x" value="${-hip_aa_frame_width + 0.147989}"/> <!-- TODO -->
-    <xacro:property name="hip_base_com_y" value="0.016341"/> <!-- TODO -->
-    <xacro:property name="hip_base_com_z" value="0.147761"/> <!-- TODO -->
-    <xacro:property name="hip_aa_com_x" value="${-hip_aa_frame_width + 0.108094}"/> <!-- TODO -->
-    <xacro:property name="hip_aa_com_y" value="${-hip_base_height/2 - hip_aa_frame_height + 0.197758}"/> <!-- TODO -->
-    <xacro:property name="hip_aa_com_z" value="0.029507"/> <!-- TODO -->
-    <xacro:property name="upper_leg_com_x" value="0.000709"/> <!-- TODO -->
+    <xacro:property name="hip_base_com_x" value="${-hip_aa_frame_width + 0.147989}"/>
+    <xacro:property name="hip_base_com_y" value="0.016341"/>
+    <xacro:property name="hip_base_com_z" value="0.147761"/>
+    <xacro:property name="hip_aa_com_x" value="${-hip_aa_frame_width + 0.108094}"/>
+    <xacro:property name="hip_aa_com_y"
+                    value="${-hip_base_height/2 - hip_aa_frame_height + 0.197758}"/>
+    <xacro:property name="hip_aa_com_z" value="0.029507"/>
+    <xacro:property name="upper_leg_com_x" value="0.000709"/>
     <xacro:property name="upper_leg_com_y" value="${-hip_base_height/2 - hip_aa_frame_height +
-                                                    upper_leg_offset + 0.215254}"/> <!-- TODO -->
-    <xacro:property name="upper_leg_com_z" value="-0.19205"/> <!-- TODO -->
-    <xacro:property name="lower_leg_com_x" value="-0.00321"/> <!-- TODO -->
+                                                    upper_leg_offset + 0.215254}"/>
+    <xacro:property name="upper_leg_com_z" value="-0.19205"/>
+    <xacro:property name="lower_leg_com_x" value="-0.00321"/>
     <xacro:property name="lower_leg_com_y" value="${-hip_base_height/2 - hip_aa_frame_height +
-                                                    upper_leg_offset + 0.184081}"/> <!-- TODO -->
-    <xacro:property name="lower_leg_com_z" value="${upper_leg_height - 0.527082}"/> <!-- TODO -->
-    <xacro:property name="foot_com_x" value="-0.028926"/> <!-- TODO -->
+                                                    upper_leg_offset + 0.184081}"/>
+    <xacro:property name="lower_leg_com_z" value="${upper_leg_height - 0.527082}"/>
+    <xacro:property name="foot_com_x" value="-0.028926"/>
     <xacro:property name="foot_com_y" value="${-hip_base_height/2 - hip_aa_frame_height +
-                                               upper_leg_offset + ankle_plate_offset + 0.155916}"/> <!-- TODO -->
-    <xacro:property name="foot_com_z" value="${upper_leg_height + lower_leg_height + ankle_plate_height - 0.789788}"/> <!-- TODO -->
-    <xacro:property name="foot_scale" value="1.35"/> <!-- TODO -->
-    <!-- TODO Change Inertia's for the MARCH VI -->
-    <!-- Inertia of the parts -->
-    <!-- Inertia's have been determined in Catia, see
-         https://confluence.projectmarch.nl:8443/display/51/URDF+description -->
-    <!-- The inertia's were defined around the CoM. Note that in the Catia x axis is the URDF y axis and the Catia y
-         axis is the negative URDF x axis, see confluence for the impact. The given inertia's are for the right leg,
-         Ixy and Iyz will be inverted for the left leg. -->
-    <xacro:property name="hip_base_Ixx" value="0.141"/> <!-- TODO -->
-    <xacro:property name="hip_base_Ixy" value="0.0000336"/> <!-- TODO -->
-    <xacro:property name="hip_base_Ixz" value="-0.007"/> <!-- TODO -->
-    <xacro:property name="hip_base_Iyy" value="0.087"/> <!-- TODO -->
-    <xacro:property name="hip_base_Iyz" value="0.0005089"/> <!-- TODO -->
-    <xacro:property name="hip_base_Izz" value="0.091"/> <!-- TODO -->
-    <xacro:property name="hip_aa_Ixx" value="0.013"/> <!-- TODO -->
-    <xacro:property name="hip_aa_Ixy" value="0.008"/> <!-- TODO -->
-    <xacro:property name="hip_aa_Ixz" value="0.005"/> <!-- TODO -->
-    <xacro:property name="hip_aa_Iyy" value="0.023"/> <!-- TODO -->
-    <xacro:property name="hip_aa_Iyz" value="-0.001"/> <!-- TODO -->
-    <xacro:property name="hip_aa_Izz" value="0.028"/> <!-- TODO -->
-    <xacro:property name="upper_leg_Ixx" value="0.127"/> <!-- TODO -->
-    <xacro:property name="upper_leg_Ixy" value="0.0001291"/> <!-- TODO -->
-    <xacro:property name="upper_leg_Ixz" value="-0.0002056"/> <!-- TODO -->
-    <xacro:property name="upper_leg_Iyy" value="0.122"/> <!-- TODO -->
-    <xacro:property name="upper_leg_Iyz" value="0.016"/> <!-- TODO -->
-    <xacro:property name="upper_leg_Izz" value="0.015"/> <!-- TODO -->
-    <xacro:property name="lower_leg_Ixx" value="0.075"/> <!-- TODO -->
-    <xacro:property name="lower_leg_Ixy" value="-0.027"/> <!-- TODO -->
-    <xacro:property name="lower_leg_Ixz" value="-0.008"/> <!-- TODO -->
-    <xacro:property name="lower_leg_Iyy" value="0.11"/> <!-- TODO -->
-    <xacro:property name="lower_leg_Iyz" value="-0.002"/> <!-- TODO -->
-    <xacro:property name="lower_leg_Izz" value="0.071" /> <!-- TODO -->
-    <xacro:property name="foot_Ixx" value="0.021"/> <!-- TODO -->
-    <xacro:property name="foot_Ixy" value="-0.002"/> <!-- TODO -->
-    <xacro:property name="foot_Ixz" value="0.02"/> <!-- TODO -->
-    <xacro:property name="foot_Iyy" value="0.027"/> <!-- TODO -->
-    <xacro:property name="foot_Iyz" value="0.004"/> <!-- TODO -->
-    <xacro:property name="foot_Izz" value="0.01" /> <!-- TODO -->
-    <!-- TODO Change range of motion for the MARCH VI -->
-    <!-- Joint properties -->
-    <!-- For limit calculations, see https://confluence.projectmarch.nl:8443/pages/viewpage.action?pageId=268697604 -->
-    <xacro:property name="left_hip_fe_rotation_lower_limit" value="${-21.04431152*pi/180}"/> <!-- rad --> <!-- TODO -->
-    <xacro:property name="left_hip_fe_rotation_upper_limit" value="${98.97033691*pi/180}"/> <!-- rad --> <!-- TODO -->
-    <xacro:property name="right_hip_fe_rotation_lower_limit" value="${-20.23406982*pi/180}"/> <!-- rad --> <!-- TODO -->
-    <xacro:property name="right_hip_fe_rotation_upper_limit" value="${99.48120117*pi/180}"/> <!-- rad --> <!-- TODO -->
-    <xacro:property name="hip_fe_soft_buffer" value="${3*pi/180}"/> <!-- rad --> <!-- TODO -->
-    <xacro:property name="hip_fe_effort_limit" value="${max_effort_rotary}"/> <!-- IU --> <!-- TODO -->
-    <xacro:property name="hip_fe_velocity_limit" value="2.0"/> <!-- rad/s --> <!-- TODO -->
-    <xacro:property name="left_hip_aa_rotation_lower_limit" value="${-18.54492188*pi/180}"/> <!-- rad --> <!-- TODO -->
-    <xacro:property name="left_hip_aa_rotation_upper_limit" value="${16.34765625*pi/180}"/> <!-- rad --> <!-- TODO -->
-    <xacro:property name="right_hip_aa_rotation_lower_limit" value="${-18.10546875*pi/180}"/> <!-- rad --> <!-- TODO -->
-    <xacro:property name="right_hip_aa_rotation_upper_limit" value="${15.99609375*pi/180}"/> <!-- rad --> <!-- TODO -->
-    <xacro:property name="hip_aa_soft_buffer" value="${3.5*pi/180}"/> <!-- rad --> <!-- TODO -->
-    <xacro:property name="hip_aa_effort_limit" value="${max_effort_linear}"/> <!-- IU --> <!-- TODO -->
-    <xacro:property name="hip_aa_velocity_limit" value="1.0"/> <!-- rad/s --> <!-- TODO -->
-    <xacro:property name="left_knee_rotation_lower_limit" value="${-5.012512207*pi/180}"/> <!-- TODO -->
-    <xacro:property name="left_knee_rotation_upper_limit" value="${112.4230957*pi/180}"/> <!-- TODO -->
-    <xacro:property name="right_knee_rotation_lower_limit" value="${-4.89440918*pi/180}"/> <!-- TODO -->
-    <xacro:property name="right_knee_rotation_upper_limit" value="${115.3097534*pi/180}"/> <!-- TODO -->
-    <xacro:property name="knee_extension_soft_buffer" value="${3.5*pi/180}"/> <!-- rad --> <!-- TODO -->
-    <xacro:property name="knee_flexion_soft_buffer" value="${3*pi/180}"/> <!-- rad --> <!-- TODO -->
-    <xacro:property name="knee_effort_limit" value="${max_effort_rotary}"/> <!-- IU --> <!-- TODO -->
-    <xacro:property name="knee_velocity_limit" value="2.5"/> <!-- TODO -->
-    <xacro:property name="left_ankle_rotation_lower_limit" value="${-26.30401611*pi/180}"/> <!-- TODO -->
-    <xacro:property name="left_ankle_rotation_upper_limit" value="${15.88348389*pi/180}"/> <!-- TODO -->
-    <xacro:property name="right_ankle_rotation_lower_limit" value="${-23.203125*pi/180}"/> <!-- TODO -->
-    <xacro:property name="right_ankle_rotation_upper_limit" value="${14.23828125*pi/180}"/> <!-- TODO -->
-    <xacro:property name="ankle_dorsalflexion_soft_buffer" value="${5*pi/180}"/> <!-- rad --> <!-- TODO -->
-    <xacro:property name="ankle_plantarflexion_soft_buffer" value="${3*pi/180}"/> <!-- rad --> <!-- TODO -->
-    <xacro:property name="ankle_effort_limit" value="${max_effort_linear}"/> <!-- IU --> <!-- TODO -->
-    <xacro:property name="ankle_velocity_limit" value="1.0"/> <!-- TODO -->
-    <xacro:property name="camera_link" value="0.05"/> <!-- Size of square 'camera' box --> <!-- TODO -->
-    <xacro:property name="axel_offset" value="0.05"/> <!-- Space btw top of beam and the each joint --> <!-- TODO -->
+                                               upper_leg_offset + ankle_plate_offset + 0.155916}"/>
+    <xacro:property name="foot_com_z"
+                    value="${upper_leg_height + lower_leg_height + ankle_plate_height - 0.789788}"/>
+    <xacro:property name="foot_scale" value="1.35"/>
     <!-- Import all Gazebo-customization elements, including Gazebo colors -->
     <xacro:include filename="march.gazebo"/>
     <material name="blue">
-        <color rgba="0 0 0.6 1"/> <!-- TODO nieuwe huisstijl -->
+        <color rgba="0.163 0.476 0.718 0.8"/>
     </material>
     <!-- Used for fixing robot to Gazebo 'base_link' -->
@@ -192,196 +120,84 @@
     <!-- Parts -->
     <!-- Hip-->
-    <link name="hip_base">
-        <visual>
-            <origin xyz="${hip_aa_frame_width} ${-hip_base_height/2} ${-width}" rpy="0 0 0"/>
-            <geometry>
-                <mesh filename="package://march_description/urdf/stl-files/march6/HipBase.stl" scale="0.001 0.001 0.001"/>
-            </geometry>
-            <material name="blue"/>
-        </visual>
-        <inertial>
-            <origin xyz="${hip_base_com_x} ${hip_base_com_y} ${hip_base_com_z}" rpy="0 0 0"/>
-            <mass value="${hip_base_mass}"/>
-            <inertia
-                    ixx="${hip_base_Ixx}"
-                    ixy="${hip_base_Ixy}"
-                    ixz="${hip_base_Ixz}"
-                    iyy="${hip_base_Iyy}"
-                    iyz="${hip_base_Iyz}"
-                    izz="${hip_base_Izz}" />
-        </inertial>
-        <collision>
-            <origin xyz="0 0 0" rpy="0 0 0"/>
-            <geometry>
-                <box size="${width} ${hip_base_height} ${width}"/>
-            </geometry>
-        </collision>
-    </link>
+    <xacro:frame_part name="hip_base"
+                      reflect="1"
+                      length="${hip_base_height}"
+                      direction="y"
+                      visual_origin="${hip_aa_frame_width} 0 ${-width}"
+                      collision_origin="0 0 0"
+                      mesh="march6/HipBase.stl"
+                      com="${hip_base_com_x} ${hip_base_com_y} ${hip_base_com_z}"
+                      mass="${dimensions['hip_base']['mass']}"
+                      inertia="${inertia['hip_base']}"
+                      scale="0.001 0.001 0.001"
+                      visual_rpy="0 0 0"
+    />
     <!-- IMU-->
     <link name="imu_link">
     </link>
-    <!-- Left Moving Hip-->
-    <link name="hip_aa_frame_left_side">
-        <visual>
-            <origin xyz="${-hip_aa_frame_width} ${hip_base_height/2} 0" rpy="0 0 ${pi}"/>
-            <geometry>
-                <mesh filename="package://march_description/urdf/stl-files/LeftHAA.stl" scale="1 1 1"/>
-            </geometry>
-            <material name="blue"/>
-        </visual>
-        <collision>
-            <origin xyz="0 ${-hip_aa_frame_height/2} 0" rpy="0 0 0"/>
-            <geometry>
-                <box size="${width} ${hip_aa_frame_height} ${width}"/>
-            </geometry>
-        </collision>
-    </link>
-    <link name="hip_aa_frame_left_front">
-        <inertial>
-            <origin xyz="${hip_aa_com_x} ${-hip_aa_com_y} ${hip_aa_com_z}" rpy="0 0 0"/>
-            <mass value="${hip_aa_mass}"/>
-            <inertia
-                    ixx="${hip_aa_Ixx}"
-                    ixy="${-hip_aa_Ixy}"
-                    ixz="${hip_aa_Ixz}"
-                    iyy="${hip_aa_Iyy}"
-                    iyz="${-hip_aa_Iyz}"
-                    izz="${hip_aa_Izz}" />
-        </inertial>
-        <collision>
-            <origin xyz="${-hip_aa_frame_width/2} 0 0" rpy="0 0 0"/>
-            <geometry>
-                <box size="${hip_aa_frame_width} ${width} ${width}"/>
-            </geometry>
-        </collision>
-    </link>
-    <!-- Upper Leg Left-->
-    <link name="upper_leg_left">
-        <visual>
-            <origin xyz="0 0 0" rpy="0 0 ${pi}"/>
-            <geometry>
-                <mesh filename="package://march_description/urdf/stl-files/UpperLeftLeg.stl" scale="0.001 0.001 0.001"/>
-            </geometry>
-            <material name="blue"/>
-        </visual>
-        <inertial>
-            <origin xyz="${upper_leg_com_x} ${-upper_leg_com_y} ${upper_leg_com_z}" rpy="0 0 0"/>
-            <mass value="${upper_leg_mass}"/>
-            <inertia
-                    ixx="${upper_leg_Ixx}"
-                    ixy="${-upper_leg_Ixy}"
-                    ixz="${upper_leg_Ixz}"
-                    iyy="${upper_leg_Iyy}"
-                    iyz="${-upper_leg_Iyz}"
-                    izz="${upper_leg_Izz}" />
-        </inertial>
-        <collision>
-            <origin xyz="0 0 ${-upper_leg_height/2}" rpy="0 0 0"/>
-            <geometry>
-                <box size="${width} ${width} ${upper_leg_height}"/>
-            </geometry>
-        </collision>
-    </link>
-    <!-- Lower Leg Left -->
-    <link name="lower_leg_left">
-        <visual>
-            <origin
-                xyz="0 ${hip_base_height/2 + hip_aa_frame_height - upper_leg_offset} ${upper_leg_height}"
-                rpy="0 0 ${pi}"
-            />
-            <geometry>
-                <mesh filename="package://march_description/urdf/stl-files/LowerLeftLeg.stl" scale="1 1 1"/>
-            </geometry>
-            <material name="blue"/>
-        </visual>
-        <inertial>
-            <origin xyz="${lower_leg_com_x} ${-lower_leg_com_y} ${lower_leg_com_z}" rpy="0 0 0"/>
-            <mass value="${lower_leg_mass}"/>
-            <inertia
-                    ixx="${lower_leg_Ixx}"
-                    ixy="${-lower_leg_Ixy}"
-                    ixz="${lower_leg_Ixz}"
-                    iyy="${lower_leg_Iyy}"
-                    iyz="${-lower_leg_Iyz}"
-                    izz="${lower_leg_Izz}" />
-        </inertial>
-        <collision>
-            <origin xyz="0 0 ${-lower_leg_height/2}" rpy="0 0 0"/>
-            <geometry>
-                <box size="${width} ${width} ${lower_leg_height}"/>
-            </geometry>
-        </collision>
-    </link>
-    <!-- Ankle plate Left -->
-    <link name="ankle_plate_left">
-        <visual>
-            <origin
-                xyz="0
-                     ${hip_base_height/2 + hip_aa_frame_height - upper_leg_offset - ankle_plate_offset}
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