Commit message: Update xacro to align visuals

File: ros2/src/shared/march_description/urdf/macros/frame_part.xacro (robot description, xacro)
@@ -25,5 +25,5 @@
                         <mesh filename="package://march_description/urdf/stl-files/${mesh}" scale="${scale}"/>
                     </geometry>
-                    <material name="blue"/>
+                    <material name="visuals_material"/>
                 </visual>
             </xacro:unless>

File: ros2/src/shared/march_description/urdf/march4.xacro (robot description, xacro)
@@ -113,5 +113,5 @@
     <!-- Import all Gazebo-customization elements, including Gazebo colors -->
     <xacro:include filename="march.gazebo"/>
-    <material name="blue">
+    <material name="visuals_material">
         <color rgba="0 0 0.6 1"/>
     </material>

File: ros2/src/shared/march_description/urdf/march6.xacro (robot description, xacro)
@@ -63,4 +63,6 @@
     <xacro:property name="upper_leg_offset"
                     value="${dimensions['upper_leg']['offset']}"/>
+    <xacro:property name="knee_offset"
+                    value="${dimensions['lower_leg']['offset']}"/>
     <xacro:property name="upper_leg_mass"
                     value="${dimensions['upper_leg']['mass']}"/>
@@ -72,5 +74,5 @@
     <!-- mass = Ankle actuator + Lower leg -->
     <xacro:property name="ankle_plate_height"
-                    value="${dimensions['ankle_plate']['length']}"/>
+                    value="${dimensions['ankle_plate']['length'] - width}"/>
     <xacro:property name="ankle_plate_offset"
                     value="${dimensions['ankle_plate']['offset']}"/>
@@ -116,6 +118,6 @@
     <!-- Import all Gazebo-customization elements, including Gazebo colors -->
     <xacro:include filename="march.gazebo"/>
-    <material name="blue">
-        <color rgba="0.163 0.476 0.718 0.9"/>
+    <material name="visuals_material">
+        <color rgba="0.163 0.476 0.718 1"/>
     </material>
     <!-- Used for fixing robot to Gazebo 'base_link' -->
@@ -127,5 +129,5 @@
                       length="${hip_base_height}"
                       direction="y"
-                      visual_origin="${hip_aa_frame_width} 0 ${-width}"
+                      visual_origin="${hip_aa_frame_width} ${-width/2} ${-width/2}"
                       collision_origin="0 0 0"
                       mesh="march6/HipBase.stl"
@@ -144,5 +146,5 @@
                       direction="y"
                       collision_origin="0 ${-hip_aa_frame_height/2} 0"
-                      visual_origin="${hip_aa_frame_width-width} ${hip_aa_frame_height/2} ${-width}"
+                      visual_origin="${width/2} ${width/2} ${-width}"
                       mesh="march6/LeftHAA.stl"
                       scale="0.001 0.001 0.001"
@@ -165,5 +167,5 @@
                       direction="z"
                       collision_origin="0 0 ${-upper_leg_height/2}"
-                      visual_origin="0 0 ${-upper_leg_height-width}"
+                      visual_origin="-0.01 ${width/2} ${-upper_leg_height - width - 0.02}"
                       mesh="march6/UpperLeftLeg.stl"
                       com="${upper_leg_com_x} ${-upper_leg_com_y} ${upper_leg_com_z}"
@@ -177,5 +179,5 @@
                       direction="z"
                       collision_origin="0 0 ${-lower_leg_height/2}"
-                      visual_origin="0 ${-width/2} ${-lower_leg_height-width}"
+                      visual_origin="${width/2-0.01} ${-width/2} ${-lower_leg_height-width/2 - 0.01}"
                       mesh="march6/LowerLeftLeg.stl"
                       com="${lower_leg_com_x} ${-lower_leg_com_y} ${lower_leg_com_z}"
@@ -190,10 +192,8 @@
                       direction="z"
                       mesh="march6/LeftFoot.stl"
-                      visual_origin="${foot_height_forward}
-                     ${-width/2}
-                     ${-ankle_plate_height - width/2}"
+                      visual_origin="${-foot_height_forward+0.005} ${-ankle_plate_offset+knee_offset-width/2} ${-ankle_plate_height-width+0.01}"
                       collision_origin="0 0 ${-ankle_plate_height/2}"
                       scale="0.001 0.001 0.001"
-                      visual_rpy="0 0 ${-pi/2}"
+                      visual_rpy="0 0 ${pi}"
     />
     <xacro:frame_part name="foot_left"
@@ -217,5 +217,5 @@
                       direction="y"
                       length="${hip_aa_frame_height}"
-                      visual_origin="${-hip_aa_frame_width-hip_base_height} ${-hip_aa_frame_height/2} ${-width}"
+                      visual_origin="${-width/2-hip_aa_frame_width} ${-width/2} ${-width}"
                       collision_origin="0 ${hip_aa_frame_height/2} 0"
                       mesh="march6/RightHAA.stl"
@@ -238,5 +238,5 @@
                       length="${upper_leg_height}"
                       collision_origin="0 0 ${-upper_leg_height/2}"
-                      visual_origin="0 0 ${-upper_leg_height-width}"
+                      visual_origin="-0.01 ${-width/2} ${-upper_leg_height - width - 0.02}"
                       mesh="march6/UpperRightLeg.stl"
                       com="${upper_leg_com_x} ${upper_leg_com_y} ${upper_leg_com_z}"
@@ -250,5 +250,5 @@
                       length="${lower_leg_height}"
                       direction="z"
-                      visual_origin="0 ${width/2} ${-lower_leg_height-width}"
+                      visual_origin="0 ${knee_offset} ${-lower_leg_height-width/2-0.01}"
                       mesh="march6/LowerRightLeg.stl"
                       com="${lower_leg_com_x} ${lower_leg_com_y} ${lower_leg_com_z}"
@@ -265,8 +265,8 @@
                       direction="z"
                       mesh="march6/RightFoot.stl"
-                      visual_origin="${foot_height_forward} ${width/2} ${-ankle_plate_height-width/2}"
+                      visual_origin="0 ${ankle_plate_offset-knee_offset+width/2} ${-ankle_plate_height-width+0.01}"
                       collision_origin="0 0 ${-ankle_plate_height/2}"
                       scale="0.001 0.001 0.001"
-                      visual_rpy="0 0 ${-pi/2}"
+                      visual_rpy="0 0 0"
     />
     <xacro:pressure_sole side="right" foot_name="foot_right"/>
@@ -325,5 +325,5 @@
             child="lower_leg_left"
             safety="${safety_values['knee']}"
-            origin="0 0 ${-upper_leg_height}"
+            origin="0 ${knee_offset} ${-upper_leg_height}"
             axis="0 -1 0"
             reduction="${rotary_reduction}"
@@ -343,5 +343,5 @@
         <parent link="ankle_plate_left"/>
         <child link="foot_left"/>
-        <origin xyz="0 0 ${-ankle_plate_height}" rpy="0 0 0"/>
+        <origin xyz="0 0 ${-ankle_plate_height-width/2}" rpy="0 0 0"/>
     </joint>
     <xacro:march_joint
@@ -374,5 +374,5 @@
             parent="upper_leg_right"
             child="lower_leg_right"
-            origin="0 0 ${-upper_leg_height}"
+            origin="0 ${-knee_offset} ${-upper_leg_height}"
             axis="0 -1 0"
             safety="${safety_values['knee']}"
@@ -393,5 +393,5 @@
         <parent link="ankle_plate_right"/>
         <child link="foot_right"/>
-        <origin xyz="0 0 ${-ankle_plate_height}" rpy="0 0 0"/>
+        <origin xyz="0 0 ${-ankle_plate_height-width/2}" rpy="0 0 0"/>
     </joint>
     <xacro:include filename="camera/_d435.urdf.xacro"/>
