Commit message: Minor pressure sole xacro change

File: ros2/src/shared/march_description/urdf/macros/pressure_sole.xacro (robot description, xacro)
@@ -2,8 +2,9 @@
 <robot  xmlns:xacro="http://www.ros.org/wiki/xacro">
     <xacro:macro name="pressure_sole"
-                 params="side foot_name">
-        <link name="pressure_sole_${side}">
+                 params="foot_place foot_name *origin">
+        <link name="pressure_sole_${foot_place}">
             <collision>
-                <origin xyz="${(-foot_height_forward+foot_height_backward)/2} 0 0" rpy="0 0 0"/>
+                <xacro:insert_block name="origin"/>
+                <!--<origin xyz="${(-foot_height_forward+foot_height_backward)/2} 0 0" rpy="0 0 0"/>-->
                 <geometry>
                     <box size="${foot_height_forward+foot_height_backward} ${width} 0.001"/>
@@ -11,9 +12,9 @@
             </collision>
         </link>
-        <gazebo reference="pressure_sole_${side}">
-            <sensor name="pressure_sole_${side}" type="contact">
+        <gazebo reference="pressure_sole_${foot_place}">
+            <sensor name="pressure_sole_${foot_place}" type="contact">
                 <always_on>true</always_on>
-                <contact collision="ankle_plate_${side}_fixed_joint_lump__pressure_sole_${side}_collision_2"/>
-                <plugin name="pressure_sole_plugin_${side}" filename="libgazebo_ros_bumper.so">
+                <contact collision="ankle_plate_${foot_place}_fixed_joint_lump__pressure_sole_${foot_place}_collision_2"/>
+                <plugin name="pressure_sole_plugin_${foot_place}" filename="libgazebo_ros_bumper.so">
                     <bumperTopicName>/march/sensor/right_pressure_sole</bumperTopicName>
                     <frameName>world</frameName>
@@ -21,7 +22,7 @@
             </sensor>
         </gazebo>`
-        <joint name="pressure_sole_${side}_joint" type="fixed">
+        <joint name="pressure_sole_${foot_place}_joint" type="fixed">
             <parent link="${foot_name}"/>
-            <child link="pressure_sole_${side}"/>
+            <child link="pressure_sole_${foot_place}"/>
             <origin xyz="0 0 ${-(width/2)}" rpy="0 0 0"/>
         </joint>

File: ros2/src/shared/march_description/urdf/march4.xacro (robot description, xacro)
@@ -186,5 +186,7 @@
         <fdir1>1 0 0</fdir1>
     </gazebo>
-    <xacro:pressure_sole side="left" foot_name="foot_left"/>
+    <xacro:pressure_sole foot_place="left_hallux" foot_name="foot_left">
+        <origin xyz="${(-foot_height_forward+foot_height_backward)/2} 0 0" rpy="0 0 0"/>
+    </xacro:pressure_sole>
     <xacro:frame_part name="hip_aa_frame_right_side"
                       reflect="1"
@@ -238,5 +240,7 @@
     />
     <!-- Foot Right -->
-    <xacro:pressure_sole side="right" foot_name="foot_right"/>
+    <xacro:pressure_sole foot_place="right_toe" foot_name="foot_right">
+        <origin xyz="${(-foot_height_forward+foot_height_backward)/2} 0 0" rpy="0 0 0"/>
+    </xacro:pressure_sole>
     <xacro:frame_part name="foot_right"
                       reflect="1"

Commit message: Pressure sole macro change

File: ros2/src/shared/march_description/urdf/macros/pressure_sole.xacro (robot description, xacro)
@@ -8,5 +8,5 @@
                 <!--<origin xyz="${(-foot_height_forward+foot_height_backward)/2} 0 0" rpy="0 0 0"/>-->
                 <geometry>
-                    <box size="${foot_height_forward+foot_height_backward} ${width} 0.001"/>
+                    <box size="${(foot_height_forward+foot_height_backward)/4} ${width/2} 0.001"/>
                 </geometry>
             </collision>

File: ros2/src/shared/march_description/urdf/march4.xacro (robot description, xacro)
@@ -187,5 +187,5 @@
     </gazebo>
     <xacro:pressure_sole foot_place="left_hallux" foot_name="foot_left">
-        <origin xyz="${(-foot_height_forward+foot_height_backward)/2} 0 0" rpy="0 0 0"/>
+        <origin xyz="${(-foot_height_forward+foot_height_backward)/8} ${width/2} 0" rpy="0 0 0"/>
     </xacro:pressure_sole>
     <xacro:frame_part name="hip_aa_frame_right_side"

Commit message: Pressure sole macro update

File: ros2/src/shared/march_description/urdf/macros/pressure_sole.xacro (robot description, xacro)
@@ -1,10 +1,9 @@
 <?xml version="1.0"?>
 <robot  xmlns:xacro="http://www.ros.org/wiki/xacro">
-    <xacro:macro name="pressure_sole"
+    <xacro:macro name="pressure_sensor"
                  params="foot_place foot_name *origin">
         <link name="pressure_sole_${foot_place}">
             <collision>
                 <xacro:insert_block name="origin"/>
-                <!--<origin xyz="${(-foot_height_forward+foot_height_backward)/2} 0 0" rpy="0 0 0"/>-->
                 <geometry>
                     <box size="${(foot_height_forward+foot_height_backward)/4} ${width/2} 0.001"/>
@@ -28,3 +27,30 @@
         </joint>
     </xacro:macro>
+    <xacro:macro name="pressure_sole"
+                 params="foot_name">
+        <xacro:pressure_sensor foot_place="left_heel_1" foot_name="${foot_name}">
+            <origin xyz="${-(foot_height_forward+foot_height_backward)/8} ${width/4} 0" rpy="0 0 0"/>
+        </xacro:pressure_sensor>
+        <xacro:pressure_sensor foot_place="left_heel_2" foot_name="${foot_name}">
+            <origin xyz="${-(foot_height_forward+foot_height_backward)/8} ${-width/4} 0" rpy="0 0 0"/>
+        </xacro:pressure_sensor>
+        <xacro:pressure_sensor foot_place="left_heel_Arch" foot_name="${foot_name}">
+            <origin xyz="${-(foot_height_forward+foot_height_backward)*3/8} ${width/4} 0" rpy="0 0 0"/>
+        </xacro:pressure_sensor>
+        <xacro:pressure_sensor foot_place="left_heel_MET1" foot_name="${foot_name}">
+            <origin xyz="${-(foot_height_forward+foot_height_backward)*3/8} ${-width/4} 0" rpy="0 0 0"/>
+        </xacro:pressure_sensor>
+        <xacro:pressure_sensor foot_place="left_heel_MET3" foot_name="${foot_name}">
+            <origin xyz="${-(foot_height_forward+foot_height_backward)*5/8} ${-width/4} 0" rpy="0 0 0"/>
+        </xacro:pressure_sensor>
+        <xacro:pressure_sensor foot_place="left_heel_MET5" foot_name="${foot_name}">
+            <origin xyz="${-(foot_height_forward+foot_height_backward)*5/8} ${width/4} 0" rpy="0 0 0"/>
+        </xacro:pressure_sensor>
+        <xacro:pressure_sensor foot_place="left_heel_Toes" foot_name="${foot_name}">
+            <origin xyz="${-(foot_height_forward+foot_height_backward)*7/8} ${width/4} 0" rpy="0 0 0"/>
+        </xacro:pressure_sensor>
+        <xacro:pressure_sensor foot_place="left_heel_Hallux" foot_name="${foot_name}">
+            <origin xyz="${-(foot_height_forward+foot_height_backward)*7/8} ${-width/4} 0" rpy="0 0 0"/>
+        </xacro:pressure_sensor>
+    </xacro:macro>
 </robot>

File: ros2/src/shared/march_description/urdf/march4.xacro (robot description, xacro)
@@ -186,10 +186,6 @@
         <fdir1>1 0 0</fdir1>
     </gazebo>
-    <xacro:pressure_sole foot_place="left_heel_1" foot_name="foot_left">
-        <origin xyz="${(-foot_height_forward+foot_height_backward)/8} ${width/4} 0" rpy="0 0 0"/>
-    </xacro:pressure_sole>
-    <xacro:pressure_sole foot_place="left_heel_2" foot_name="foot_left">
-        <origin xyz="${(-foot_height_forward+foot_height_backward)/8} ${-width/4} 0" rpy="0 0 0"/>
-    </xacro:pressure_sole>
+    <xacro:pressure_sole foot_name="foot_left"
+    />
     <xacro:frame_part name="hip_aa_frame_right_side"
                       reflect="1"
@@ -242,5 +238,5 @@
                       scale="1 1 ${foot_scale}"
     />
-    <!-- Foot Right -->
+    <!-- Foot Right
     <xacro:pressure_sole foot_place="right_heel_1" foot_name="foot_right">
         <origin xyz="${(-foot_height_forward+foot_height_backward)/8} ${width/4} 0" rpy="0 0 0"/>
@@ -248,5 +244,5 @@
     <xacro:pressure_sole foot_place="right_heel_2" foot_name="foot_right">
         <origin xyz="${(-foot_height_forward+foot_height_backward)/8} ${-width/4} 0" rpy="0 0 0"/>
-    </xacro:pressure_sole>
+    </xacro:pressure_sole> -->
     <xacro:frame_part name="foot_right"
                       reflect="1"

Commit message: Sdf inpsection

File: ros2/src/shared/march_description/urdf/macros/pressure_sole.xacro (robot description, xacro)
@@ -2,5 +2,5 @@
 <robot  xmlns:xacro="http://www.ros.org/wiki/xacro">
     <xacro:macro name="pressure_sensor"
-                 params="foot_place foot_name *origin">
+                 params="foot_place foot_name counter *origin">
         <link name="pressure_sole_${foot_place}">
             <collision>
@@ -14,7 +14,8 @@
             <sensor name="pressure_sole_${foot_place}" type="contact">
                 <always_on>true</always_on>
-                <contact collision="ankle_plate_${foot_place}_fixed_joint_lump__pressure_sole_${foot_place}_collision_2"/>
+                <!--<contact collision="ankle_plate_${foot_name}_fixed_joint_lump__pressure_sole_${foot_place}_collision_${counter}"/>-->
+                <contact collision="ankle_plate_left_fixed_joint_lump__pressure_sole_left_heel_Hallux_collision_2"/>
                 <plugin name="pressure_sole_plugin_${foot_place}" filename="libgazebo_ros_bumper.so">
-                    <bumperTopicName>/march/sensor/right_pressure_sole</bumperTopicName>
+                    <bumperTopicName>/march/sensor/${foot_name}_pressure_sole_${foot_place}</bumperTopicName>
                     <frameName>world</frameName>
                 </plugin>
@@ -22,5 +23,5 @@
         </gazebo>`
         <joint name="pressure_sole_${foot_place}_joint" type="fixed">
-            <parent link="${foot_name}"/>
+            <parent link="foot_${foot_name}"/>
             <child link="pressure_sole_${foot_place}"/>
             <origin xyz="0 0 ${-(width/2)}" rpy="0 0 0"/>
@@ -29,26 +30,27 @@
     <xacro:macro name="pressure_sole"
                  params="foot_name">
-        <xacro:pressure_sensor foot_place="left_heel_1" foot_name="${foot_name}">
+        <!--
+        <xacro:pressure_sensor foot_place="left_heel_1" foot_name="${foot_name}" counter="2">
             <origin xyz="${-(foot_height_forward+foot_height_backward)/8} ${width/4} 0" rpy="0 0 0"/>
         </xacro:pressure_sensor>
-        <xacro:pressure_sensor foot_place="left_heel_2" foot_name="${foot_name}">
+        <xacro:pressure_sensor foot_place="left_heel_2" foot_name="${foot_name}" counter="3">
             <origin xyz="${-(foot_height_forward+foot_height_backward)/8} ${-width/4} 0" rpy="0 0 0"/>
         </xacro:pressure_sensor>
-        <xacro:pressure_sensor foot_place="left_heel_Arch" foot_name="${foot_name}">
+        <xacro:pressure_sensor foot_place="left_heel_Arch" foot_name="${foot_name}" counter="4">
             <origin xyz="${-(foot_height_forward+foot_height_backward)*3/8} ${width/4} 0" rpy="0 0 0"/>
         </xacro:pressure_sensor>
-        <xacro:pressure_sensor foot_place="left_heel_MET1" foot_name="${foot_name}">
+        <xacro:pressure_sensor foot_place="left_heel_MET1" foot_name="${foot_name}" counter="6">
             <origin xyz="${-(foot_height_forward+foot_height_backward)*3/8} ${-width/4} 0" rpy="0 0 0"/>
         </xacro:pressure_sensor>
-        <xacro:pressure_sensor foot_place="left_heel_MET3" foot_name="${foot_name}">
+        <xacro:pressure_sensor foot_place="left_heel_MET3" foot_name="${foot_name}" counter="7">
             <origin xyz="${-(foot_height_forward+foot_height_backward)*5/8} ${-width/4} 0" rpy="0 0 0"/>
         </xacro:pressure_sensor>
-        <xacro:pressure_sensor foot_place="left_heel_MET5" foot_name="${foot_name}">
+        <xacro:pressure_sensor foot_place="left_heel_MET5" foot_name="${foot_name}" counter="8">
             <origin xyz="${-(foot_height_forward+foot_height_backward)*5/8} ${width/4} 0" rpy="0 0 0"/>
         </xacro:pressure_sensor>
-        <xacro:pressure_sensor foot_place="left_heel_Toes" foot_name="${foot_name}">
+        <xacro:pressure_sensor foot_place="left_heel_Toes" foot_name="${foot_name}" counter="9">
             <origin xyz="${-(foot_height_forward+foot_height_backward)*7/8} ${width/4} 0" rpy="0 0 0"/>
-        </xacro:pressure_sensor>
-        <xacro:pressure_sensor foot_place="left_heel_Hallux" foot_name="${foot_name}">
+        </xacro:pressure_sensor>-->
+        <xacro:pressure_sensor foot_place="left_heel_Hallux" foot_name="${foot_name}" counter="5">
             <origin xyz="${-(foot_height_forward+foot_height_backward)*7/8} ${-width/4} 0" rpy="0 0 0"/>
         </xacro:pressure_sensor>

File: ros2/src/shared/march_description/urdf/march4.xacro (robot description, xacro)
@@ -186,5 +186,5 @@
         <fdir1>1 0 0</fdir1>
     </gazebo>
-    <xacro:pressure_sole foot_name="foot_left"
+    <xacro:pressure_sole foot_name="left"
     />
     <xacro:frame_part name="hip_aa_frame_right_side"

Commit message: Change sensor name

File: ros2/src/shared/march_description/urdf/macros/pressure_sole.xacro (robot description, xacro)
@@ -12,10 +12,12 @@
         </link>
         <gazebo reference="pressure_sole_${foot_place}">
-            <sensor name="pressure_sole_${foot_place}" type="contact">
+            <sensor name="pressure_sole_${foot_place}_sensor" type="contact">
                 <always_on>true</always_on>
-                <contact collision="ankle_plate_${foot_name}_fixed_joint_lump__pressure_sole_${foot_place}_collision_${counter}"/>
+                <contact>
+                    <collision>ankle_plate_${foot_name}_fixed_joint_lump__pressure_sole_${foot_place}_collision_${counter}</collision>
+                </contact>
                 <!--<contact collision="ankle_plate_left_collision"/>-->
                 <plugin name="pressure_sole_plugin_${foot_place}" filename="libgazebo_ros_bumper.so">
-                    <bumperTopicName>/march/sensor/${foot_name}_pressure_sole_${foot_place}</bumperTopicName>
+                    <bumperTopicName>march/sensor/${foot_name}_pressure_sole_${foot_place}</bumperTopicName>
                     <frameName>world</frameName>
                 </plugin>

Commit message: Fix feet

File: ros2/src/shared/march_description/urdf/macros/pressure_sole.xacro (robot description, xacro)
@@ -5,5 +5,6 @@
         <link name="pressure_sole_${side}">
             <collision>
-                <origin xyz="${(-foot_height_forward+foot_height_backward)/2} 0 0" rpy="0 0 0"/>
+                <origin xyz="${(foot_height_backward-foot_height_forward)/2} 0 0"
+                        rpy="0 0 0"/>
                 <geometry>
                     <box size="${foot_height_forward+foot_height_backward} ${width} 0.001"/>
@@ -26,4 +27,10 @@
             <origin xyz="0 0 ${-(width/2)}" rpy="0 0 0"/>
         </joint>
+        <gazebo reference="pressure_sole_${side}">
+            <mu1>${foot_mu1}</mu1>
+            <mu2>${foot_mu2}</mu2>
+            <minDepth>${foot_min_depth}</minDepth>
+            <fdir1>1 0 0</fdir1>
+        </gazebo>
     </xacro:macro>
 </robot>

File: ros2/src/shared/march_description/urdf/march6.xacro (robot description, xacro)
@@ -191,5 +191,5 @@
                       mesh="march6/LeftFoot.stl"
                       visual_origin="${foot_height_forward}
-                     0
+                     ${-ankle_plate_offset/2}
                      ${-ankle_plate_height - width/2}"
                       collision_origin="0 0 ${-ankle_plate_height/2}"
@@ -202,5 +202,5 @@
                       direction="x"
                       inertia="${inertia['foot']}"
-                      collision_origin="${-(foot_height_forward+foot_height_backward)/2} 0 0"
+                      collision_origin="${(foot_height_backward-foot_height_forward)/2} 0 0"
                       com="${foot_com_x} ${-foot_com_y} ${foot_com_z}"
                       mass="${foot_mass}"/>
@@ -265,5 +265,5 @@
                       direction="z"
                       mesh="march6/RightFoot.stl"
-                      visual_origin="${foot_height_forward} 0 ${-ankle_plate_height-width/2}"
+                      visual_origin="${foot_height_forward} ${ankle_plate_offset/2} ${-ankle_plate_height-width/2}"
                       collision_origin="0 0 ${-ankle_plate_height/2}"
                       scale="0.001 0.001 0.001"
@@ -276,5 +276,5 @@
                       direction="x"
                       inertia="${inertia['foot']}"
-                      collision_origin="${-(foot_height_forward+foot_height_backward)/2} 0 0"
+                      collision_origin="${(foot_height_backward-foot_height_forward)/2} 0 0"
                       com="${foot_com_x} ${foot_com_y} ${foot_com_z}"
                       mass="${foot_mass}"/>
