Commit message: Rename moving to actuating

File: ros2/src/shared/march_description/urdf/macros/configurable_joint.xacro (robot description, xacro)
@@ -4,5 +4,5 @@
     <xacro:macro name="march_configurable_joint"
                  params="name parent child safety origin axis reduction limits">
-        <xacro:if value="${name in moving_joints}">
+        <xacro:if value="${name in actuating_joints}">
             <xacro:march_joint
                 name="${name}"
@@ -16,5 +16,5 @@
                 />
         </xacro:if>
-        <xacro:unless value="${name in moving_joints}">
+        <xacro:unless value="${name in actuating_joints}">
             <joint name="${name}" type="fixed">
                 <parent link="${parent}"/>

File: ros2/src/shared/march_description/urdf/march6.xacro (robot description, xacro)
@@ -47,5 +47,5 @@
     <xacro:property name="linear_reduction_hip" value="240"/>
     <xacro:property name="linear_reduction_ankle" value="236"/>
-    <xacro:property name="moving_joints" value="${(properties['moving_joints'])}"/>
+    <xacro:property name="actuating_joints" value="${(properties['actuating_joints'])}"/>
     <!-- Constants for robot dimensions -->
     <!-- Masses determined in Catia, see https://confluence.projectmarch.nl:8443/display/51/URDF+description -->
