Commit message: Fix the problem of angle directions that were different defined in M6 URDF vs LR/RL URDF

File: ros1/src/dynamic_gait/march7_description/march7_description_lr/urdf/march7_description_lr.urdf (robot description, URDF)
Before this commit: robot march7_description_lr, 9 links, 8 joints
Links:
- link base_link: mass 0.5 -> 0.61034
- link hip: mass 0.375 -> 0.58567
- link left_hip: mass 0.27454 -> 0.98442
- link left_lower_leg: mass 0.72546 -> 1.1232
- link left_upper_leg: mass 0.72546 -> 1.1232
- link right_foot: mass 0.5 -> 0.61034
- link right_hip: mass 0.27454 -> 0.98442
- link right_lower_leg: mass 0.72546 -> 1.1232
- link right_upper_leg: mass 0.72546 -> 1.1232
Joints:
- joint left_ankle: axis 1 0 0 -> -1 0 0; limit lower=-0.7854 upper=0.7854 effort=0 velocity=0 -> lower=-1.2217 upper=0.087266 effort=0 velocity=0; origin xyz=0.025 -0.2 0.025 rpy=1.5708 0 0 -> xyz=0 -0.258 0.108 rpy=1.5708 0 0
- joint left_hip_aa: limit lower=-0.34907 upper=0.34907 effort=0 velocity=0 -> lower=-0.34907 upper=0.5236 effort=0 velocity=0; origin xyz=-0.1 0.025 -0.025 rpy=3.1416 0 3.1416 -> xyz=-0.1545 0 -0.175 rpy=3.1416 0 3.1416
- joint left_hip_fe: limit lower=-0.7854 upper=0.7854 effort=0 velocity=0 -> lower=-0.2618 upper=2.0071 effort=0 velocity=0; origin xyz=0 0.275 -0.025 rpy=3.1416 0 3.1416 -> xyz=0 0.41 0 rpy=3.1416 0 3.1416
- joint left_knee: limit lower=0 upper=1.5708 effort=0 velocity=0 -> lower=0 upper=2.3562 effort=0 velocity=0; origin xyz=0 0.3 0.05 rpy=0 0 0 -> xyz=0 0.41 0 rpy=0 0 0
- joint right_ankle: axis 1 0 0 -> -1 0 0; limit lower=-0.7854 upper=0.7854 effort=0 velocity=0 -> lower=-1.2217 upper=0.087266 effort=0 velocity=0; origin xyz=0 -0.3 -0.05 rpy=0 0 0 -> xyz=0 -0.41 0 rpy=3.1416 0 3.1416
- joint right_hip_aa: axis 0 0 1 -> 0 0 -1; limit lower=-0.34907 upper=0.34907 effort=0 velocity=0 -> lower=-0.34907 upper=0.5236 effort=0 velocity=0; origin xyz=0.15 0 0 rpy=0 0 0 -> xyz=0.145 0 0 rpy=-3.1416 0 0
- joint right_hip_fe: limit lower=-0.7854 upper=0.7854 effort=0 velocity=0 -> lower=-0.2618 upper=2.0071 effort=0 velocity=0; origin xyz=0.1 -0.025 -0.025 rpy=0 0 0 -> xyz=0.1295 0 0.175 rpy=3.1416 0 0
- joint right_knee: axis 1 0 0 -> -1 0 0; limit lower=-1.5708 upper=0 effort=0 velocity=0 -> lower=0 upper=2.3562 effort=0 velocity=0; origin xyz=0 -0.275 0.025 rpy=0 0 0 -> xyz=0 -0.41 0 rpy=0 0 0

File: ros1/src/dynamic_gait/march7_description/march7_description_rl/urdf/march7_description_rl.urdf (robot description, URDF)
Before this commit: robot march7_description_rl, 9 links, 8 joints
Links:
- link base_link: mass 0.5 -> 0.61034
- link hip: mass 0.375 -> 0.58567
- link left_foot: mass 0.5 -> 0.61034
- link left_hip: mass 0.27454 -> 0.98442
- link left_lower_leg: mass 0.72546 -> 1.1232
- link left_upper_leg: mass 0.72546 -> 1.1232
- link right_hip: mass 0.27454 -> 0.98442
- link right_lower_leg: mass 0.72546 -> 1.1232
- link right_upper_leg: mass 0.72546 -> 1.1232
Joints:
- joint left_ankle: axis 1 0 0 -> -1 0 0; limit lower=-0.7854 upper=0.7854 effort=0 velocity=0 -> lower=-1.2217 upper=0.087266 effort=0 velocity=0; origin xyz=0 -0.3 -0.05 rpy=0 0 0 -> xyz=0 -0.41 0 rpy=3.1416 0 3.1416
- joint left_hip_aa: limit lower=-0.34907 upper=0.34907 effort=0 velocity=0 -> lower=-0.34907 upper=0.5236 effort=0 velocity=0; origin xyz=-0.15 0 0 rpy=-3.1416 0 3.1416 -> xyz=-0.145 0 0 rpy=3.1416 0 3.1416
- joint left_hip_fe: limit lower=-0.7854 upper=0.7854 effort=0 velocity=0 -> lower=-0.2618 upper=2.0071 effort=0 velocity=0; origin xyz=0.1 -0.025 -0.025 rpy=-3.1416 0 3.1416 -> xyz=0.1295 0 0.175 rpy=3.1416 0 3.1416
- joint left_knee: axis 1 0 0 -> -1 0 0; limit lower=-1.5708 upper=0 effort=0 velocity=0 -> lower=0 upper=2.3562 effort=0 velocity=0; origin xyz=0 -0.275 0.025 rpy=0 0 0 -> xyz=0 -0.41 0 rpy=0 0 0
- joint right_ankle: axis 1 0 0 -> -1 0 0; limit lower=-0.7854 upper=0.7854 effort=0 velocity=0 -> lower=-1.2217 upper=0.087266 effort=0 velocity=0; origin xyz=-0.025 -0.2 0.025 rpy=1.5708 0 0 -> xyz=0 -0.258 0.108 rpy=1.5708 0 0
- joint right_hip_aa: axis 0 0 1 -> 0 0 -1; limit lower=-0.34907 upper=0.34907 effort=0 velocity=0 -> lower=-0.34907 upper=0.5236 effort=0 velocity=0; origin xyz=-0.1 0.025 -0.025 rpy=0 0 0 -> xyz=-0.1545 0 -0.175 rpy=3.1416 0 0
- joint right_hip_fe: axis 1 0 0 -> -1 0 0; limit lower=-0.7854 upper=0.7854 effort=0 velocity=0 -> lower=-0.2618 upper=2.0071 effort=0 velocity=0; origin xyz=0 0.275 -0.025 rpy=0 0 0 -> xyz=0 0.41 0 rpy=-3.1416 0 0
- joint right_knee: limit lower=0 upper=1.5708 effort=0 velocity=0 -> lower=0 upper=2.3562 effort=0 velocity=0; origin xyz=0 0.3 0.05 rpy=0 0 0 -> xyz=0 0.41 0 rpy=0 0 0

Commit message: Change the dorsiflexion limit in URDF to 10 degrees

File: ros1/src/dynamic_gait/march7_description/march7_description_lr/urdf/march7_description_lr.urdf (robot description, URDF)
Before this commit: robot march7_description_lr, 9 links, 8 joints
Joints:
- joint left_ankle: limit lower=-1.2217 upper=0.087266 effort=0 velocity=0 -> lower=-1.2217 upper=0.174533 effort=0 velocity=0
- joint right_ankle: limit lower=-1.2217 upper=0.087266 effort=0 velocity=0 -> lower=-1.2217 upper=0.174533 effort=0 velocity=0

File: ros1/src/dynamic_gait/march7_description/march7_description_rl/urdf/march7_description_rl.urdf (robot description, URDF)
Before this commit: robot march7_description_rl, 9 links, 8 joints
Joints:
- joint left_ankle: limit lower=-1.2217 upper=0.087266 effort=0 velocity=0 -> lower=-1.2217 upper=0.174533 effort=0 velocity=0
- joint right_ankle: limit lower=-1.2217 upper=0.087266 effort=0 velocity=0 -> lower=-1.2217 upper=0.174533 effort=0 velocity=0
