Commit message: Add camera to march4, wrong location

File: ros2/src/shared/march_description/urdf/camera/_d435.urdf.xacro (robot description, xacro)
@@ -1,12 +1,18 @@
 <?xml version="1.0"?>
 <!--
-License: Apache 2.0. See LICENSE file in root directory.
-Copyright(c) 2017 Intel Corporation. All Rights Reserved
-This is the URDF model for the Intel RealSense 430 camera, in it's
-aluminum peripherial evaluation case.
+Copyright 2017 Intel Corporation
+Licensed under the Apache License, Version 2.0 (the "License");
+you may not use this file except in compliance with the License.
+You may obtain a copy of the License at
+    http://www.apache.org/licenses/LICENSE-2.0
+Unless required by applicable law or agreed to in writing, software
+distributed under the License is distributed on an "AS IS" BASIS,
+WITHOUT WARRANTIES OR CONDITIONS OF ANY KIND, either express or implied.
+See the License for the specific language governing permissions and
+limitations under the License.
 -->
 <robot name="sensor_d435" xmlns:xacro="http://ros.org/wiki/xacro">
   <!--File includes-->
-  <xacro:include filename="$(find realsense2_description)/urdf/_d435.gazebo.xacro"/>
+  <xacro:include filename="_d435.gazebo.xacro"/>
   <xacro:macro name="sensor_d435" params="name:=camera topics_ns:=camera parent *origin publish_pointcloud:=true">
     <xacro:property name="M_PI" value="3.1415926535897931" />
@@ -48,6 +54,5 @@
         <geometry>
           <!-- <box size="${d435_cam_width} ${d435_cam_height} ${d435_cam_depth}"/> -->
-          <mesh filename="package://realsense2_description/meshes/d435.dae" />
-          <!--<mesh filename="package://realsense2_description/meshes/d435/d435.dae" />-->
+          <mesh filename="package://march_description/urdf/camera/_d435.dae" />
         </geometry>
         <material name="${name}_aluminum"/>

File: ros2/src/shared/march_description/urdf/march4.xacro (robot description, xacro)
@@ -692,5 +692,4 @@
         <origin xyz="0 0 ${-ankle_plate_height}" rpy="0 0 0"/>
     </joint>
-    <xa
     <xacro:include filename="camera/_d435.urdf.xacro" />
     <xacro:sensor_d435 parent="upper_leg_left">

File: ros2/src/shared/march_description/urdf/march4_with_koen_lengths.xacro (robot description, xacro)
@@ -644,5 +644,5 @@
         <origin xyz="0 0 ${-ankle_plate_height}" rpy="0 0 0"/>
     </joint>
-    <xacro:include filename="$(find realsense2_description)/urdf/_d435.urdf.xacro" />
+    <xacro:include filename="camera/_d435.urdf.xacro" />
     <xacro:sensor_d435 parent="upper_leg_left">
         <origin xyz="0 0 0" rpy="0 0 3.1416"/>

Commit message: Add possibility to turn off simulation camera to test with physical camera

File: ros2/src/shared/march_description/urdf/camera/_d435.urdf.xacro (robot description, xacro)
@@ -15,5 +15,6 @@
   <!--File includes-->
   <xacro:include filename="_d435.gazebo.xacro"/>
-  <xacro:macro name="sensor_d435" params="name:=camera topics_ns:=camera parent *origin publish_pointcloud:=true">
+  <xacro:macro name="sensor_d435"
+               params="name:=camera topics_ns:=camera parent plugin *origin publish_pointcloud:=true">
     <xacro:property name="M_PI" value="3.1415926535897931" />
     <!-- The following values are approximate, and the camera node
@@ -124,5 +125,7 @@
     <link name="${name}_color_optical_frame"/>
     <!-- Realsense Gazebo Plugin -->
-    <xacro:gazebo_d435 camera_name="${name}" reference_link="${name}_link" topics_ns="${topics_ns}" depth_optical_frame="${name}_depth_optical_frame" color_optical_frame="${name}_color_optical_frame" infrared1_optical_frame="${name}_left_ir_optical_frame" infrared2_optical_frame="${name}_right_ir_optical_frame" publish_pointcloud="${publish_pointcloud}"/>
+    <xacro:if value="${plugin}">
+      <xacro:gazebo_d435 camera_name="${name}" reference_link="${name}_link" topics_ns="${topics_ns}" depth_optical_frame="${name}_depth_optical_frame" color_optical_frame="${name}_color_optical_frame" infrared1_optical_frame="${name}_left_ir_optical_frame" infrared2_optical_frame="${name}_right_ir_optical_frame" publish_pointcloud="${publish_pointcloud}"/>
+    </xacro:if>
   </xacro:macro>
 </robot>

File: ros2/src/shared/march_description/urdf/march4.xacro (robot description, xacro)
@@ -7,4 +7,11 @@
     the hover_height to 0.0. Set ground_gait to true to ground gait in simulation.-->
     <xacro:arg name="ground_gait" default="false"/>
+<!--    Switch between using the physical camera and the simulation camera -->
+<!--    If set to 'true', no physical camera is needed -->
+<!--    If this value is set to 'false', the plugin will not be started and the topics -->
+<!--    published by the real camera will be used. -->
+<!--    In both these situations the camera will still be visible and placed in the urdf,-->
+<!--    to be used for the transformations.-->
+    <xacro:arg name="realsense_simulation" default="false"/>
     <xacro:unless value="$(arg ground_gait)">
         <xacro:property name="parent_name" value="world"/>
@@ -693,5 +700,5 @@
     </joint>
     <xacro:include filename="camera/_d435.urdf.xacro" />
-    <xacro:sensor_d435 parent="hip_base">
+    <xacro:sensor_d435 parent="hip_base" plugin="$(arg realsense_simulation)">
 <!--    Attached to the hip_base, since this is most comparable to the backpack -->
 <!--    in amount of movement, the distance from hip base is based on first design.-->

File: ros2/src/shared/march_description/urdf/march4_with_koen_lengths.xacro (robot description, xacro)
@@ -7,4 +7,11 @@
     the hover_height to 0.0. Set ground_gait to true to ground gait in simulation.-->
     <xacro:arg name="ground_gait" default="false"/>
+    <!--    Switch between using the physical camera and the simulation camera -->
+    <!--    If set to 'true', no physical camera is needed -->
+    <!--    If this value is set to 'false', the plugin will not be started and the topics -->
+    <!--    published by the real camera will be used. -->
+    <!--    In both these situations the camera will still be visible and placed in the urdf,-->
+    <!--    to be used for the transformations.-->
+    <xacro:arg name="realsense_simulation" default="false"/>
     <xacro:unless value="$(arg ground_gait)">
         <xacro:property name="parent_name" value="world"/>
@@ -644,6 +651,6 @@
         <origin xyz="0 0 ${-ankle_plate_height}" rpy="0 0 0"/>
     </joint>
-    <xacro:include filename="camera/_d435.urdf.xacro" />
-    <xacro:sensor_d435 parent="hip_base">
+    <xacro:include filename="camera/_d435.urdf.xacro"/>
+    <xacro:sensor_d435 parent="hip_base" plugin="$(arg realsense_simulation)">
         <!--    Attached to the hip_base, since this is most comparable to the backpack -->
         <!--    in amount of movement, the distance from hip base is based on first design.-->

Commit message: Launch realsense from ROS2 and process IMU data with plugins

File: ros2/src/shared/march_description/urdf/camera/_d435.urdf.xacro (robot description, xacro)
@@ -124,10 +124,21 @@
     </joint>
     <link name="${name}_color_optical_frame"/>
-    <link name="${name}_imu_optical_frame"/>
-    <joint name="${name}_imu_optical_joint" type="fixed">
-      <origin xyz="0 0 0" rpy="${-M_PI/2} 0 ${-M_PI/2}"/>
-      <parent link="${name}_depth_frame" />
-      <child link="${name}_imu_optical_frame"/>
-    </joint>
+    <!-- This block is needed as the realsense ROS2 wrapper uses the frame 'camera_imu_optical_frame' for IMU data -->
+    <xacro:if value="${name == 'camera_back'}">
+      <link name="camera_imu_optical_frame"/>
+      <joint name="${name}_imu_optical_joint" type="fixed">
+        <origin xyz="0 0 0" rpy="${-M_PI/2} 0 ${-M_PI/2}"/>
+        <parent link="${name}_depth_frame" />
+        <child link="camera_imu_optical_frame"/>
+      </joint>
+    </xacro:if>
+    <xacro:unless value="${name == 'camera_back'}">
+      <link name="${name}_imu_optical_frame"/>
+      <joint name="${name}_imu_optical_joint" type="fixed">
+        <origin xyz="0 0 0" rpy="${-M_PI/2} 0 ${-M_PI/2}"/>
+        <parent link="${name}_depth_frame" />
+        <child link="${name}_imu_optical_frame"/>
+      </joint>
+    </xacro:unless>
     <!-- Realsense Gazebo Plugin -->
     <xacro:if value="${plugin}">

Commit message: Fix rviz2 visualization in ROS2

File: ros2/src/shared/march_description/urdf/camera/_d435.urdf.xacro (robot description, xacro)
@@ -124,21 +124,18 @@
     </joint>
     <link name="${name}_color_optical_frame"/>
-    <!-- This block is needed as the realsense ROS2 wrapper uses the frame 'camera_imu_optical_frame' for IMU data -->
+    <link name="${name}_imu_optical_frame"/>
+    <joint name="${name}_imu_optical_joint" type="fixed">
+      <origin xyz="0 0 0" rpy="${-M_PI/2} 0 ${-M_PI/2}"/>
+      <parent link="${name}_depth_frame" />
+      <child link="${name}_imu_optical_frame"/>
+    </joint>
     <xacro:if value="${name == 'camera_back'}">
       <link name="camera_imu_optical_frame"/>
-      <joint name="${name}_imu_optical_joint" type="fixed">
-        <origin xyz="0 0 0" rpy="${-M_PI/2} 0 ${-M_PI/2}"/>
-        <parent link="${name}_depth_frame" />
+      <joint name="camera_imu_optical_joint" type="fixed">
+        <origin xyz="0 0 0" rpy="0 0 0"/>
+        <parent link="camera_back_depth_frame" />
         <child link="camera_imu_optical_frame"/>
       </joint>
     </xacro:if>
-    <xacro:unless value="${name == 'camera_back'}">
-      <link name="${name}_imu_optical_frame"/>
-      <joint name="${name}_imu_optical_joint" type="fixed">
-        <origin xyz="0 0 0" rpy="${-M_PI/2} 0 ${-M_PI/2}"/>
-        <parent link="${name}_depth_frame" />
-        <child link="${name}_imu_optical_frame"/>
-      </joint>
-    </xacro:unless>
     <!-- Realsense Gazebo Plugin -->
     <xacro:if value="${plugin}">

Commit message: Fix weird orientation with world

File: ros2/src/shared/march_description/urdf/camera/_d435.urdf.xacro (robot description, xacro)
@@ -134,5 +134,5 @@
       <joint name="camera_imu_optical_joint" type="fixed">
         <origin xyz="0 0 0" rpy="0 0 0"/>
-        <parent link="camera_back_depth_frame" />
+        <parent link="camera_back_imu_optical_frame" />
         <child link="camera_imu_optical_frame"/>
       </joint>
