Commit message: Add ability to disable kill when outside hard limits for certain joints and change msg update speed.

File: ros2/src/control/march_control/xacro/ros2_control.xacro (robot description, xacro)
@@ -2,5 +2,6 @@
 <robot xmlns:xacro="http://www.ros.org/wiki/xacro">
   <!-- Defines a normal effort joint used for within a ros2_control tag. Used in the exo and for gazebo. -->
-  <xacro:macro name="effort_joint" params="name">
+    <xacro:macro name="effort_joint"
+                 params="name stop_when_outside_hard_limits:=^ msec_until_error_when_in_error_soft_limits:=^">
     <joint name="${name}">
       <command_interface name="effort"/>
@@ -8,4 +9,6 @@
       <state_interface name="velocity"/>
       <state_interface name="effort"/>
+        <param name="stop_when_outside_hard_limits">${stop_when_outside_hard_limits}</param>
+        <param name="msec_until_error_when_in_error_soft_limits">${msec_until_error_when_in_error_soft_limits}</param>
     </joint>
   </xacro:macro>
@@ -18,5 +21,7 @@
   </xacro:macro>
   <xacro:macro name="march_joint"
-               params="name type:=^|effort">
+               params="name type:=^|effort
+               stop_when_outside_hard_limits:=^|true
+               msec_until_error_when_in_error_soft_limits:=^|1000">
     <xacro:if value="${type == 'effort'}">
       <xacro:effort_joint name="${name}"/>
@@ -37,9 +42,9 @@
     <hardware>
       <xacro:if value="${type == 'rviz'}">
-        <plugin>fake_components/GenericSystem</plugin>
+<!--        <plugin>fake_components/GenericSystem</plugin>-->
         <!-- Switch the 'fake_components/GenericSystem' with 'march_hardware_interface/MarchRvizSystemInterface' -->
         <!-- If you whish to debug and play around with a very simple hardware interface, -->
         <!-- They practically work the same -->
-<!--        <plugin>march_hardware_interface/MarchRvizSystemInterface</plugin>-->
+        <plugin>march_hardware_interface/MarchRvizSystemInterface</plugin>
       </xacro:if>
       <xacro:if value="${type == 'effort'}">
@@ -53,9 +58,9 @@
       </xacro:if>
     </hardware>
-    <xacro:march_joint name="left_ankle"/>
+    <xacro:march_joint name="left_ankle" stop_when_outside_hard_limits="false" msec_until_error_when_in_error_soft_limits="0"/>
     <xacro:march_joint name="left_hip_aa"/>
     <xacro:march_joint name="left_hip_fe"/>
     <xacro:march_joint name="left_knee"/>
-    <xacro:march_joint name="right_ankle"/>
+    <xacro:march_joint name="right_ankle" stop_when_outside_hard_limits="false" msec_until_error_when_in_error_soft_limits="0"/>
     <xacro:march_joint name="right_hip_aa"/>
     <xacro:march_joint name="right_hip_fe"/>
