Commit message: Update repo, remove some old functions and update other things

File: ros2/src/march_control/xacro/ros2_control.xacro (robot description, xacro)
@@ -1,7 +1,7 @@
 <?xml version="1.0"?>
 <robot xmlns:xacro="http://www.ros.org/wiki/xacro">
-  <!-- Defines a normal effort joint used for within a ros2_control tag. Used in the exo. -->
-    <xacro:macro name="effort_joint"
-                 params="name stop_when_outside_hard_limits:=^ msec_until_error_when_in_error_soft_limits:=^">
+  <!-- Defines a normal effort joint used for within a ros2_control tag. Used in the exo and for gazebo. -->
+  <xacro:macro name="effort_joint"
+               params="name stop_when_outside_hard_limits:=^ msec_until_error_when_in_error_soft_limits:=^">
     <joint name="${name}">
       <command_interface name="position"/>
@@ -10,10 +10,10 @@
       <state_interface name="velocity"/>
       <state_interface name="effort"/>
-        <param name="stop_when_outside_hard_limits">${stop_when_outside_hard_limits}</param>
-        <param name="msec_until_error_when_in_error_soft_limits">${msec_until_error_when_in_error_soft_limits}</param>
+      <param name="stop_when_outside_hard_limits">${stop_when_outside_hard_limits}</param>
+      <param name="msec_until_error_when_in_error_soft_limits">${msec_until_error_when_in_error_soft_limits}</param>
     </joint>
   </xacro:macro>
-  <!-- Defines a basic position joint used for within a ros2_control tag. Used when running simulation only. -->
-  <xacro:macro name="simulation_joint" params="name">
+  <!-- Defines a basic position joint used for within a ros2_control tag. Used when running rviz only. -->
+  <xacro:macro name="rviz_joint" params="name">
     <joint name="${name}">
       <command_interface name="position"/>
@@ -28,26 +28,30 @@
       <xacro:effort_joint name="${name}"/>
     </xacro:if>
-    <xacro:if value="${type == 'simulation'}">
-      <xacro:simulation_joint name="${name}"/>
+    <xacro:if value="${type == 'rviz'}">
+      <xacro:rviz_joint name="${name}"/>
     </xacro:if>
   </xacro:macro>
-  <!-- You have 2 types 'effort' or 'simulation' if you do simulation you should only open simulation. -->
+  <!-- You have 2 types 'effort' or 'rviz' if you do rviz you should only open rviz. -->
   <!-- Default is 'effort' because this makes easier bc gazebo control is activated through the urdf on published on the '/robot_description' -->
   <xacro:arg name="type" default='effort'/>
   <xacro:property name="type" value="$(arg type)"/>
-  <!-- You have 2 types 'effort' or 'simulation' if you do simulation you should only open simulation (not gazebo!). -->
-  <!-- Has no effect if type is simulation.-->
-  <xacro:arg name="simulation" default="true"/>
+  <!-- You have 2 types 'effort' or 'rviz' if you do rviz you should only open rviz (not gazebo!). -->
+  <!-- Has no effect if type is rviz.-->
+  <!-- Default is 'true' because this makes easier bc gazebo control is activated through the urdf on published on the '/robot_description' -->
+  <xacro:arg name="mujoco" default="true"/>
   <ros2_control name="march" type="system">
     <hardware>
-      <xacro:if value="${type == 'simulation'}">
+      <xacro:if value="${type == 'rviz'}">
+        <!--        <plugin>fake_components/GenericSystem</plugin>-->
+        <!-- Switch the 'march_hardware_interface/MarchMockSystemInterface' with 'fake_components/GenericSystem' -->
+        <!-- If you wish to debug and play around with RVIZ, otherwise use the mock interface for mujoco-->
         <plugin>march_hardware_interface/MarchMockSystemInterface</plugin>
       </xacro:if>
       <xacro:if value="${type == 'effort'}">
-          <plugin>march_hardware_interface/MarchExoSystemInterface</plugin>
-          <param name="robot">pressure_soles</param>
+        <plugin>march_hardware_interface/MarchExoSystemInterface</plugin>
+        <param name="robot">pressure_soles</param>
       </xacro:if>
     </hardware>
-    <xacro:march_joint name="left_ankle" stop_when_outside_hard_limits="false" msec_until_error_when_in_error_soft_limits="0"/>
+    <!-- <xacro:march_joint name="left_ankle" stop_when_outside_hard_limits="false" msec_until_error_when_in_error_soft_limits="0"/>
     <xacro:march_joint name="left_hip_aa" stop_when_outside_hard_limits="false"  msec_until_error_when_in_error_soft_limits="0"/>
     <xacro:march_joint name="left_hip_fe"/>
@@ -56,5 +60,13 @@
     <xacro:march_joint name="right_hip_aa" stop_when_outside_hard_limits="false" msec_until_error_when_in_error_soft_limits="0"/>
     <xacro:march_joint name="right_hip_fe"/>
-    <xacro:march_joint name="right_knee"/>
+    <xacro:march_joint name="right_knee"/> -->
   </ros2_control>
+  <!-- These tags are only used when gazebo control is used -->
+  <xacro:arg name="gazebo_control_file" default="NO FILE SPECIFIED"/>
+  <gazebo>
+    <plugin name="gazebo_ros2_control" filename="libgazebo_ros2_control.so">
+      <robot_sim_type>gazebo_ros2_control/GazeboSystem</robot_sim_type>
+      <parameters>$(arg gazebo_control_file)</parameters>
+    </plugin>
+  </gazebo>
 </robot>
