Commit message: Eliminate unnecessary error soft limit margins and improve logging and checks for hard and soft limits.

File: ros2/src/march_control/xacro/ros2_control_m9.xacro (robot description, xacro)
@@ -1,58 +1,53 @@
 <?xml version="1.0"?>
 <robot xmlns:xacro="http://www.ros.org/wiki/xacro">
-<!-- Defines a normal effort joint used for within a ros2_control tag. Used in the exo. -->
-<xacro:macro name="effort_joint"
-             params="name stop_when_outside_hard_limits:=^ msec_until_error_when_in_error_soft_limits:=^">
-  <joint name="${name}">
-    <command_interface name="position"/>
-    <state_interface name="position"/>
-    <state_interface name="velocity"/>
-    <state_interface name="effort"/>
-    <param name="stop_when_outside_hard_limits">${stop_when_outside_hard_limits}</param>
-    <param name="msec_until_error_when_in_error_soft_limits">${msec_until_error_when_in_error_soft_limits}</param>
-  </joint>
-</xacro:macro>
-<!-- Defines a basic position joint used for within a ros2_control tag. Used when running simulation only. -->
-<xacro:macro name="simulation_joint" params="name">
-  <joint name="${name}">
-    <command_interface name="position"/>
-    <state_interface name="position"/>
-  </joint>
-</xacro:macro>
-<xacro:macro name="march_joint"
-             params="name type:=^|effort
-               stop_when_outside_hard_limits:=^|true
-               msec_until_error_when_in_error_soft_limits:=^|100">
-  <xacro:if value="${type != 'simulation'}">
-    <xacro:effort_joint name="${name}"/>
-  </xacro:if>
-  <xacro:if value="${type == 'simulation'}">
-    <xacro:simulation_joint name="${name}"/>
-  </xacro:if>
-</xacro:macro>
-<!-- You have 2 types 'effort' or 'simulation' if you do simulation you should only open simulation. -->
-<xacro:arg name="type" default='effort'/>
-<xacro:property name="type" value="$(arg type)"/>
-<!-- You have 2 types 'effort' or 'simulation' if you do simulation you should only open simulation (not gazebo!). -->
-<!-- Has no effect if type is simulation.-->
-<xacro:arg name="simulation" default="true"/>
-<ros2_control name="march" type="system">
-  <hardware>
+  <!-- Defines a normal effort joint used for within a ros2_control tag. Used in the exo. -->
+  <xacro:macro name="effort_joint" params="name stop_when_outside_hard_limits:=True">
+    <joint name="${name}">
+      <command_interface name="position"/>
+      <state_interface name="position"/>
+      <state_interface name="velocity"/>
+      <state_interface name="effort"/>
+      <param name="stop_when_outside_hard_limits">${stop_when_outside_hard_limits}</param>
+    </joint>
+  </xacro:macro>
+  <!-- Defines a basic position joint used for within a ros2_control tag. Used when running simulation only. -->
+  <xacro:macro name="simulation_joint" params="name">
+    <joint name="${name}">
+      <command_interface name="position"/>
+      <state_interface name="position"/>
+    </joint>
+  </xacro:macro>
+  <xacro:macro name="march_joint" params="name type:=effort stop_when_outside_hard_limits:=True">
+    <xacro:if value="${type != 'simulation'}">
+      <xacro:effort_joint name="${name}" stop_when_outside_hard_limits="${stop_when_outside_hard_limits}"/>
+    </xacro:if>
     <xacro:if value="${type == 'simulation'}">
-      <plugin>march_system_interface/MarchMockSystemInterface</plugin>
+      <xacro:simulation_joint name="${name}"/>
     </xacro:if>
-    <xacro:if value="${type == 'effort'}">
-      <plugin>march_system_interface/MarchExoSystemInterface</plugin>
-      <param name="robot">hardware_izzy</param>
-    </xacro:if>
-  </hardware>
-  <xacro:march_joint name="left_ankle_dpf"/>
-  <xacro:march_joint name="left_hip_aa"/>
-  <xacro:march_joint name="left_hip_fe"/>
-  <xacro:march_joint name="left_knee"/>
-  <xacro:march_joint name="right_ankle_dpf"/>
-  <xacro:march_joint name="right_hip_aa"/>
-  <xacro:march_joint name="right_hip_fe"/>
-  <xacro:march_joint name="right_knee"/>
-</ros2_control>
+  </xacro:macro>
+  <!-- You have 2 types 'effort' or 'simulation'. If you do simulation, only use simulation. -->
+  <xacro:arg name="type" default="effort"/>
+  <xacro:property name="type" value="$(arg type)"/>
+  <!-- You have 2 types 'effort' or 'simulation'. -->
+  <!-- Has no effect if type is simulation. -->
+  <xacro:arg name="simulation" default="True"/>
+  <ros2_control name="march" type="system">
+    <hardware>
+      <xacro:if value="${type == 'simulation'}">
+        <plugin>march_system_interface/MarchMockSystemInterface</plugin>
+      </xacro:if>
+      <xacro:if value="${type == 'effort'}">
+        <plugin>march_system_interface/MarchExoSystemInterface</plugin>
+        <param name="robot">hardware_izzy</param>
+      </xacro:if>
+    </hardware>
+    <xacro:march_joint name="left_ankle_dpf" type="${type}" stop_when_outside_hard_limits="True"/>
+    <xacro:march_joint name="left_hip_aa" type="${type}" stop_when_outside_hard_limits="True"/>
+    <xacro:march_joint name="left_hip_fe" type="${type}" stop_when_outside_hard_limits="True"/>
+    <xacro:march_joint name="left_knee" type="${type}" stop_when_outside_hard_limits="True"/>
+    <xacro:march_joint name="right_ankle_dpf" type="${type}" stop_when_outside_hard_limits="True"/>
+    <xacro:march_joint name="right_hip_aa" type="${type}" stop_when_outside_hard_limits="True"/>
+    <xacro:march_joint name="right_hip_fe" type="${type}" stop_when_outside_hard_limits="True"/>
+    <xacro:march_joint name="right_knee" type="${type}" stop_when_outside_hard_limits="True"/>
+  </ros2_control>
 </robot>

File: ros2/src/march_control/xacro/ros2_control_test_linear.xacro (robot description, xacro)
@@ -1,52 +1,46 @@
 <?xml version="1.0"?>
 <robot xmlns:xacro="http://www.ros.org/wiki/xacro">
-<!-- Defines a normal effort joint used for within a ros2_control tag. Used in the exo. -->
-<xacro:macro name="effort_joint"
-             params="name stop_when_outside_hard_limits:=^ msec_until_error_when_in_error_soft_limits:=^">
-  <joint name="${name}">
-    <command_interface name="position"/>
-    <state_interface name="position"/>
-    <state_interface name="velocity"/>
-    <state_interface name="effort"/>
-    <param name="stop_when_outside_hard_limits">${stop_when_outside_hard_limits}</param>
-    <param name="msec_until_error_when_in_error_soft_limits">${msec_until_error_when_in_error_soft_limits}</param>
-  </joint>
-</xacro:macro>
-<!-- Defines a basic position joint used for within a ros2_control tag. Used when running simulation only. -->
-<xacro:macro name="simulation_joint" params="name">
-  <joint name="${name}">
-    <command_interface name="position"/>
-    <state_interface name="position"/>
-  </joint>
-</xacro:macro>
-<xacro:macro name="march_joint"
-             params="name type:=^|effort
-               stop_when_outside_hard_limits:=^|true
-               msec_until_error_when_in_error_soft_limits:=^|1000">
-  <xacro:if value="${type != 'simulation'}">
-    <xacro:effort_joint name="${name}"/>
-  </xacro:if>
-  <xacro:if value="${type == 'simulation'}">
-    <xacro:simulation_joint name="${name}"/>
-  </xacro:if>
-</xacro:macro>
-<!-- You have 2 types 'effort' or 'simulation' if you do simulation you should only open simulation. -->
-<!-- Default is 'effort' because this makes easier bc gazebo control is activated through the urdf on published on the '/robot_description' -->
-<xacro:arg name="type" default='effort'/>
-<xacro:property name="type" value="$(arg type)"/>
-<!-- You have 2 types 'effort' or 'simulation' if you do simulation you should only open simulation (not gazebo!). -->
-<!-- Has no effect if type is simulation.-->
-<xacro:arg name="simulation" default="true"/>
-<ros2_control name="march" type="system">
-  <hardware>
+  <!-- Defines a normal effort joint used for within a ros2_control tag. Used in the exo. -->
+  <xacro:macro name="effort_joint" params="name stop_when_outside_hard_limits:=True">
+    <joint name="${name}">
+      <command_interface name="position"/>
+      <state_interface name="position"/>
+      <state_interface name="velocity"/>
+      <state_interface name="effort"/>
+      <param name="stop_when_outside_hard_limits">${stop_when_outside_hard_limits}</param>
+    </joint>
+  </xacro:macro>
+  <!-- Defines a basic position joint used for within a ros2_control tag. Used when running simulation only. -->
+  <xacro:macro name="simulation_joint" params="name">
+    <joint name="${name}">
+      <command_interface name="position"/>
+      <state_interface name="position"/>
+    </joint>
+  </xacro:macro>
+  <xacro:macro name="march_joint" params="name type:=effort stop_when_outside_hard_limits:=True">
+    <xacro:if value="${type != 'simulation'}">
+      <xacro:effort_joint name="${name}" stop_when_outside_hard_limits="${stop_when_outside_hard_limits}"/>
+    </xacro:if>
     <xacro:if value="${type == 'simulation'}">
-      <plugin>march_system_interface/MarchMockSystemInterface</plugin>
+      <xacro:simulation_joint name="${name}"/>
     </xacro:if>
-    <xacro:if value="${type == 'effort'}">
-      <plugin>march_system_interface/MarchExoSystemInterface</plugin>
-      <param name="robot">hardware_test_setup</param>
-    </xacro:if>
-  </hardware>
-  <xacro:march_joint name="linear_joint"/>
-</ros2_control>
+  </xacro:macro>
+  <!-- You have 2 types 'effort' or 'simulation'. If you do simulation, only use simulation. -->
+  <xacro:arg name="type" default="effort"/>
+  <xacro:property name="type" value="$(arg type)"/>
+  <!-- You have 2 types 'effort' or 'simulation'. -->
+  <!-- Has no effect if type is simulation. -->
+  <xacro:arg name="simulation" default="True"/>
+  <ros2_control name="march" type="system">
+    <hardware>
+      <xacro:if value="${type == 'simulation'}">
+        <plugin>march_system_interface/MarchMockSystemInterface</plugin>
+      </xacro:if>
+      <xacro:if value="${type == 'effort'}">
+        <plugin>march_system_interface/MarchExoSystemInterface</plugin>
+        <param name="robot">hardware_test_setup</param>
+      </xacro:if>
+    </hardware>
+    <xacro:march_joint name="linear_joint" type="${type}" stop_when_outside_hard_limits="True"/>
+  </ros2_control>
 </robot>

File: ros2/src/march_control/xacro/ros2_control_test_rotational.xacro (robot description, xacro)
@@ -1,52 +1,46 @@
 <?xml version="1.0"?>
 <robot xmlns:xacro="http://www.ros.org/wiki/xacro">
-<!-- Defines a normal effort joint used for within a ros2_control tag. Used in the exo. -->
-<xacro:macro name="effort_joint"
-             params="name stop_when_outside_hard_limits:=^ msec_until_error_when_in_error_soft_limits:=^">
-  <joint name="${name}">
-    <command_interface name="position"/>
-    <state_interface name="position"/>
-    <state_interface name="velocity"/>
-    <state_interface name="effort"/>
-    <param name="stop_when_outside_hard_limits">${stop_when_outside_hard_limits}</param>
-    <param name="msec_until_error_when_in_error_soft_limits">${msec_until_error_when_in_error_soft_limits}</param>
-  </joint>
-</xacro:macro>
-<!-- Defines a basic position joint used for within a ros2_control tag. Used when running simulation only. -->
-<xacro:macro name="simulation_joint" params="name">
-  <joint name="${name}">
-    <command_interface name="position"/>
-    <state_interface name="position"/>
-  </joint>
-</xacro:macro>
-<xacro:macro name="march_joint"
-             params="name type:=^|effort
-               stop_when_outside_hard_limits:=^|true
-               msec_until_error_when_in_error_soft_limits:=^|1000">
-  <xacro:if value="${type != 'simulation'}">
-    <xacro:effort_joint name="${name}"/>
-  </xacro:if>
-  <xacro:if value="${type == 'simulation'}">
-    <xacro:simulation_joint name="${name}"/>
-  </xacro:if>
-</xacro:macro>
-<!-- You have 2 types 'effort' or 'simulation' if you do simulation you should only open simulation. -->
-<!-- Default is 'effort' because this makes easier bc gazebo control is activated through the urdf on published on the '/robot_description' -->
-<xacro:arg name="type" default='effort'/>
-<xacro:property name="type" value="$(arg type)"/>
-<!-- You have 2 types 'effort' or 'simulation' if you do simulation you should only open simulation (not gazebo!). -->
-<!-- Has no effect if type is simulation.-->
-<xacro:arg name="simulation" default="true"/>
-<ros2_control name="march" type="system">
-  <hardware>
+  <!-- Defines a normal effort joint used for within a ros2_control tag. Used in the exo. -->
+  <xacro:macro name="effort_joint" params="name stop_when_outside_hard_limits:=True">
+    <joint name="${name}">
+      <command_interface name="position"/>
+      <state_interface name="position"/>
+      <state_interface name="velocity"/>
+      <state_interface name="effort"/>
+      <param name="stop_when_outside_hard_limits">${stop_when_outside_hard_limits}</param>
+    </joint>
+  </xacro:macro>
+  <!-- Defines a basic position joint used for within a ros2_control tag. Used when running simulation only. -->
+  <xacro:macro name="simulation_joint" params="name">
+    <joint name="${name}">
+      <command_interface name="position"/>
+      <state_interface name="position"/>
+    </joint>
+  </xacro:macro>
+  <xacro:macro name="march_joint" params="name type:=effort stop_when_outside_hard_limits:=True">
+    <xacro:if value="${type != 'simulation'}">
+      <xacro:effort_joint name="${name}" stop_when_outside_hard_limits="${stop_when_outside_hard_limits}"/>
+    </xacro:if>
     <xacro:if value="${type == 'simulation'}">
-      <plugin>march_system_interface/MarchMockSystemInterface</plugin>
+      <xacro:simulation_joint name="${name}"/>
     </xacro:if>
-    <xacro:if value="${type == 'effort'}">
-      <plugin>march_system_interface/MarchExoSystemInterface</plugin>
-      <param name="robot">hardware_test_setup</param>
-    </xacro:if>
-  </hardware>
-  <xacro:march_joint name="rotational_joint"/>
-</ros2_control>
+  </xacro:macro>
+  <!-- You have 2 types 'effort' or 'simulation'. If you do simulation, only use simulation. -->
+  <xacro:arg name="type" default="effort"/>
+  <xacro:property name="type" value="$(arg type)"/>
+  <!-- You have 2 types 'effort' or 'simulation'. -->
+  <!-- Has no effect if type is simulation. -->
+  <xacro:arg name="simulation" default="True"/>
+  <ros2_control name="march" type="system">
+    <hardware>
+      <xacro:if value="${type == 'simulation'}">
+        <plugin>march_system_interface/MarchMockSystemInterface</plugin>
+      </xacro:if>
+      <xacro:if value="${type == 'effort'}">
+        <plugin>march_system_interface/MarchExoSystemInterface</plugin>
+        <param name="robot">hardware_test_setup</param>
+      </xacro:if>
+    </hardware>
+    <xacro:march_joint name="rotational_joint" type="${type}" stop_when_outside_hard_limits="True"/>
+  </ros2_control>
 </robot>

File: ros2/src/march_control/xacro/ros2_control_test_setup.xacro (robot description, xacro)
@@ -1,51 +1,47 @@
 <?xml version="1.0"?>
 <robot xmlns:xacro="http://www.ros.org/wiki/xacro">
-<!-- Defines a normal effort joint used for within a ros2_control tag. Used in the exo. -->
-<xacro:macro name="effort_joint"
-             params="name stop_when_outside_hard_limits:=^ msec_until_error_when_in_error_soft_limits:=^">
-  <joint name="${name}">
-    <command_interface name="position"/>
-    <state_interface name="position"/>
-    <state_interface name="velocity"/>
-    <state_interface name="effort"/>
-    <param name="stop_when_outside_hard_limits">${stop_when_outside_hard_limits}</param>
-    <param name="msec_until_error_when_in_error_soft_limits">${msec_until_error_when_in_error_soft_limits}</param>
-  </joint>
-</xacro:macro>
-<!-- Defines a basic position joint used for within a ros2_control tag. Used when running simulation only. -->
-<xacro:macro name="simulation_joint" params="name">
-  <joint name="${name}">
-    <command_interface name="position"/>
-    <state_interface name="position"/>
-  </joint>
-</xacro:macro>
-<xacro:macro name="march_joint"
-             params="name type:=^|effort
-               stop_when_outside_hard_limits:=^|true
-               msec_until_error_when_in_error_soft_limits:=^|1000">
-  <xacro:if value="${type != 'simulation'}">
-    <xacro:effort_joint name="${name}"/>
-  </xacro:if>
-  <xacro:if value="${type == 'simulation'}">
-    <xacro:simulation_joint name="${name}"/>
-  </xacro:if>
-</xacro:macro>
-<!-- You have 2 types 'effort' or 'simulation' if you do simulation you should only open simulation. -->
-<!-- Default is 'effort' because this makes easier bc gazebo control is activated through the urdf on published on the '/robot_description' -->
-<xacro:arg name="type" default='effort'/>
-<xacro:property name="type" value="$(arg type)"/>
-<!-- You have 2 types 'effort' or 'simulation' if you do simulation you should only open simulation (not gazebo!). -->
-<!-- Has no effect if type is simulation.-->
-<xacro:arg name="simulation" default="true"/>
-<ros2_control name="march" type="system">
-  <hardware>
+  <!-- Defines a normal effort joint used for within a ros2_control tag. Used in the exo. -->
+  <xacro:macro name="effort_joint" params="name stop_when_outside_hard_limits:=True">
+    <joint name="${name}">
+      <command_interface name="position"/>
+      <state_interface name="position"/>
+      <state_interface name="velocity"/>
+      <state_interface name="effort"/>
+      <param name="stop_when_outside_hard_limits">${stop_when_outside_hard_limits}</param>
+    </joint>
+  </xacro:macro>
+  <!-- Defines a basic position joint used for within a ros2_control tag. Used when running simulation only. -->
+  <xacro:macro name="simulation_joint" params="name">
+    <joint name="${name}">
+      <command_interface name="position"/>
+      <state_interface name="position"/>
+    </joint>
+  </xacro:macro>
+  <xacro:macro name="march_joint" params="name type:=effort stop_when_outside_hard_limits:=True">
+    <xacro:if value="${type != 'simulation'}">
+      <xacro:effort_joint name="${name}" stop_when_outside_hard_limits="${stop_when_outside_hard_limits}"/>
+    </xacro:if>
     <xacro:if value="${type == 'simulation'}">
-      <plugin>march_system_interface/MarchMockSystemInterface</plugin>
+      <xacro:simulation_joint name="${name}"/>
     </xacro:if>
-    <xacro:if value="${type == 'effort'}">
-      <plugin>march_system_interface/MarchExoSystemInterface</plugin>
-      <param name="robot">hardware_test_setup</param>
-    </xacro:if>
-  </hardware>
-</ros2_control>
+  </xacro:macro>
+  <!-- You have 2 types 'effort' or 'simulation'. If you do simulation, only use simulation. -->
+  <xacro:arg name="type" default="effort"/>
+  <xacro:property name="type" value="$(arg type)"/>
+  <!-- You have 2 types 'effort' or 'simulation'. -->
+  <!-- Has no effect if type is simulation. -->
+  <xacro:arg name="simulation" default="True"/>
+  <ros2_control name="march" type="system">
+    <hardware>
+      <xacro:if value="${type == 'simulation'}">
+        <plugin>march_system_interface/MarchMockSystemInterface</plugin>
+      </xacro:if>
+      <xacro:if value="${type == 'effort'}">
+        <plugin>march_system_interface/MarchExoSystemInterface</plugin>
+        <param name="robot">hardware_test_setup</param>
+      </xacro:if>
+    </hardware>
+    <xacro:march_joint name="linear_joint" type="${type}" stop_when_outside_hard_limits="True"/>
+    <xacro:march_joint name="rotational_joint" type="${type}" stop_when_outside_hard_limits="True"/>
+  </ros2_control>
 </robot>
