Commit message: add first ik_solver tests

File: ros2/src/ik_solver/test/urdf/march_test_urdf.urdf (robot description, URDF)
Before this commit: robot march, 65 links, 64 joints
Links:
- removed link ankle_plate_left
- removed link ankle_plate_right
- removed link camera_back_bottom_screw_frame
- removed link camera_back_color_frame
- removed link camera_back_color_optical_frame
- removed link camera_back_depth_frame
- removed link camera_back_depth_optical_frame
- removed link camera_back_imu_optical_frame
- removed link camera_back_left_ir_frame
- removed link camera_back_left_ir_optical_frame
- removed link camera_back_link
- removed link camera_back_right_ir_frame
- removed link camera_back_right_ir_optical_frame
- removed link camera_front_left_bottom_screw_frame
- removed link camera_front_left_color_frame
- removed link camera_front_left_color_optical_frame
- removed link camera_front_left_depth_frame
- removed link camera_front_left_depth_optical_frame
- removed link camera_front_left_imu_optical_frame
- removed link camera_front_left_left_ir_frame
- removed link camera_front_left_left_ir_optical_frame
- removed link camera_front_left_link
- removed link camera_front_left_right_ir_frame
- removed link camera_front_left_right_ir_optical_frame
- removed link camera_front_right_bottom_screw_frame
- removed link camera_front_right_color_frame
- removed link camera_front_right_color_optical_frame
- removed link camera_front_right_depth_frame
- removed link camera_front_right_depth_optical_frame
- removed link camera_front_right_imu_optical_frame
- removed link camera_front_right_left_ir_frame
- removed link camera_front_right_left_ir_optical_frame
- removed link camera_front_right_link
- removed link camera_front_right_right_ir_frame
- removed link camera_front_right_right_ir_optical_frame
- removed link camera_imu_optical_frame
- removed link foot_left
- removed link foot_right
- removed link hip_aa_frame_left_front
- removed link hip_aa_frame_left_side
- removed link hip_aa_frame_right_front
- removed link hip_aa_frame_right_side
- removed link hip_base
- removed link imu_link
- removed link lower_leg_left
- removed link lower_leg_right
- removed link pressure_sole_left_arch
- removed link pressure_sole_left_hallux
- removed link pressure_sole_left_heel_1
- removed link pressure_sole_left_heel_2
- removed link pressure_sole_left_met1
- removed link pressure_sole_left_met3
- removed link pressure_sole_left_met5
- removed link pressure_sole_left_toes
- removed link pressure_sole_right_arch
- removed link pressure_sole_right_hallux
- removed link pressure_sole_right_heel_1
- removed link pressure_sole_right_heel_2
- removed link pressure_sole_right_met1
- removed link pressure_sole_right_met3
- removed link pressure_sole_right_met5
- removed link pressure_sole_right_toes
- removed link upper_leg_left
- removed link upper_leg_right
- removed link world
- added link L_LL, mass 4.159; collision mesh filename=package://march_gym/march_gym/envs/assets/meshes/LowerLegLe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 scale=1 1 1; visual mesh filename=package://march_gym/march_gym/envs/assets/meshes/LowerLegLe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 scale=1 1 1
- added link L_UL, mass 8.566; collision mesh filename=package://march_gym/march_gym/envs/assets/meshes/UpperLegLe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 scale=1 1 1; visual mesh filename=package://march_gym/march_gym/envs/assets/meshes/UpperLegLe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 scale=1 1 1
- added link L_foot, mass 1.22; collision mesh filename=package://march_gym/march_gym/envs/assets/meshes/FootLeft.o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 scale=1 1 1; visual mesh filename=package://march_gym/march_gym/envs/assets/meshes/FootLeft.o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 scale=1 1 1
- added link L_ground
- added link L_hip, mass 1.277; collision mesh filename=package://march_gym/march_gym/envs/assets/meshes/HipLeft.obj scale=1 1 1; visual mesh filename=package://march_gym/march_gym/envs/assets/meshes/HipLeft.obj scale=1 1 1
- added link R_LL, mass 4.159; collision mesh filename=package://march_gym/march_gym/envs/assets/meshes/LowerLegLe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 scale=1 -1 1; visual mesh filename=package://march_gym/march_gym/envs/assets/meshes/LowerLegLe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 scale=1 -1 1
- added link R_UL, mass 8.566; collision mesh filename=package://march_gym/march_gym/envs/assets/meshes/UpperLegLe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 scale=1 -1 1; visual mesh filename=package://march_gym/march_gym/envs/assets/meshes/UpperLegLe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 scale=1 -1 1
- added link R_foot, mass 1.22; collision mesh filename=package://march_gym/march_gym/envs/assets/meshes/FootLeft.o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 scale=1 -1 1; visual mesh filename=package://march_gym/march_gym/envs/assets/meshes/FootLeft.o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 scale=1 -1 1
- added link R_ground
- added link R_hip, mass 1.277; collision mesh filename=package://march_gym/march_gym/envs/assets/meshes/HipLeft.obj scale=1 -1 1; visual mesh filename=package://march_gym/march_gym/envs/assets/meshes/HipLeft.obj scale=1 -1 1
- added link backpack, mass 11.02; collision mesh filename=package://march_gym/march_gym/envs/assets/meshes/Backpack.o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 scale=1 1 1; visual mesh filename=package://march_gym/march_gym/envs/assets/meshes/Backpack.o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 scale=1 1 1
Joints:
- removed joint camera_back_color_joint
- removed joint camera_back_color_optical_joint
- removed joint camera_back_depth_joint
- removed joint camera_back_depth_optical_joint
- removed joint camera_back_imu_optical_joint
- removed joint camera_back_joint
- removed joint camera_back_left_ir_joint
- removed joint camera_back_left_ir_optical_joint
- removed joint camera_back_link_joint
- removed joint camera_back_right_ir_joint
- removed joint camera_back_right_ir_optical_joint
- removed joint camera_front_left_color_joint
- removed joint camera_front_left_color_optical_joint
- removed joint camera_front_left_depth_joint
- removed joint camera_front_left_depth_optical_joint
- removed joint camera_front_left_imu_optical_joint
- removed joint camera_front_left_joint
- removed joint camera_front_left_left_ir_joint
- removed joint camera_front_left_left_ir_optical_joint
- removed joint camera_front_left_link_joint
- removed joint camera_front_left_right_ir_joint
- removed joint camera_front_left_right_ir_optical_joint
- removed joint camera_front_right_color_joint
- removed joint camera_front_right_color_optical_joint
- removed joint camera_front_right_depth_joint
- removed joint camera_front_right_depth_optical_joint
- removed joint camera_front_right_imu_optical_joint
- removed joint camera_front_right_joint
- removed joint camera_front_right_left_ir_joint
- removed joint camera_front_right_left_ir_optical_joint
- removed joint camera_front_right_link_joint
- removed joint camera_front_right_right_ir_joint
- removed joint camera_front_right_right_ir_optical_joint
- removed joint camera_imu_optical_joint
- removed joint hip
- removed joint imu_joint
- removed joint left_foot_angle
- removed joint left_hip_angle
- removed joint pressure_sole_left_arch_joint
- removed joint pressure_sole_left_hallux_joint
- removed joint pressure_sole_left_heel_1_joint
- removed joint pressure_sole_left_heel_2_joint
- removed joint pressure_sole_left_met1_joint
- removed joint pressure_sole_left_met3_joint
- removed joint pressure_sole_left_met5_joint
- removed joint pressure_sole_left_toes_joint
- removed joint pressure_sole_right_arch_joint
- removed joint pressure_sole_right_hallux_joint
- removed joint pressure_sole_right_heel_1_joint
- removed joint pressure_sole_right_heel_2_joint
- removed joint pressure_sole_right_met1_joint
- removed joint pressure_sole_right_met3_joint
- removed joint pressure_sole_right_met5_joint
- removed joint pressure_sole_right_toes_joint
- removed joint right_foot_angle
- removed joint right_hip_angle
- added joint L_ground: type fixed, parent L_foot, child L_ground, origin xyz=0 0 -0.126
- added joint R_ground: type fixed, parent R_foot, child R_ground, origin xyz=0 0 -0.126
- joint left_ankle: axis 0 1 0 -> 0 -1 0; child ankle_plate_left -> L_foot; limit lower=-0.4996942416537476 upper=0.40151947122906656 effort=30.0 velocity=2.5 -> lower=-0.0174533 upper=0.436332 effort=0.9 velocity=4.1; origin xyz=0 0.01 -0.4 rpy=0 0 0 -> xyz=0 -0.037 -0.414 rpy=0 0 0; parent lower_leg_left -> L_LL
- joint left_hip_aa: child hip_aa_frame_left_side -> L_hip; limit lower=-0.1564660403643354 upper=0.23661653653136014 effort=30.0 velocity=2.5 -> lower=-0.2618 upper=0.174533 effort=280 velocity=2.6; origin xyz=0 -0.065 0 rpy=0 0 0 -> xyz=-0.021 0.08 0.025 rpy=0 0 0; parent hip_base -> backpack
- joint left_hip_fe: axis 0 1 0 -> 0 -1 0; child upper_leg_left -> L_UL; limit lower=-0.37755102141835345 upper=1.8026191733641141 effort=30.0 velocity=3.0 -> lower=-2.00713 upper=0.20944 effort=250 velocity=3.94; origin xyz=-0.19 0.0 0 rpy=0 0 0 -> xyz=0.182 0.182 0 rpy=0 0 0.0; parent hip_aa_frame_left_front -> L_hip
- joint left_knee: axis 0 -1 0 -> 0 1 0; child lower_leg_left -> L_LL; limit lower=-0.10258496518985226 upper=1.9959966264369478 effort=30.0 velocity=3.5 -> lower=-0.017453 upper=1.9548 effort=250 velocity=3.94; origin xyz=0 0.07 -0.41 rpy=0 0 0 -> xyz=0 -0.06 -0.413 rpy=0 0 0; parent upper_leg_left -> L_UL
- joint right_ankle: axis 0 1 0 -> 0 -1 0; child ankle_plate_right -> R_foot; limit lower=-0.5062136600022615 upper=0.3436116964863836 effort=30.0 velocity=2.5 -> lower=-0.0174533 upper=0.436332 effort=0.9 velocity=4.1; origin xyz=0 -0.01 -0.4 rpy=0 0 0 -> xyz=0 0.037 -0.414 rpy=0 0 0; parent lower_leg_right -> R_LL
- joint right_hip_aa: child hip_aa_frame_right_side -> R_hip; limit lower=-0.1856116753341626 upper=0.21514080550096118 effort=30.0 velocity=2.5 -> lower=-0.174533 upper=0.0872665 effort=4.5 velocity=2.6; origin xyz=0 0.065 0 rpy=0 0 0 -> xyz=-0.021 -0.08 0.025 rpy=0 0 0; parent hip_base -> backpack
- joint right_hip_fe: axis 0 1 0 -> 0 -1 0; child upper_leg_right -> R_UL; limit lower=-0.42663840663069397 upper=1.8019480567694142 effort=30.0 velocity=3.0 -> lower=-2.00713 upper=0.20944 effort=12.2 velocity=3.94; origin xyz=-0.19 -0.0 0 rpy=0 0 0 -> xyz=0.182 -0.182 0 rpy=0 0 0.0; parent hip_aa_frame_right_front -> R_hip
- joint right_knee: axis 0 -1 0 -> 0 1 0; child lower_leg_right -> R_LL; limit lower=-0.09951700361408097 upper=2.002899539982433 effort=30.0 velocity=3.5 -> lower=-0.017453 upper=1.9548 effort=12.2 velocity=3.94; origin xyz=0 -0.07 -0.41 rpy=0 0 0 -> xyz=0 0.06 -0.413 rpy=0 0 0; parent upper_leg_right -> R_UL
