Commit message: june 20 changes:

File: ros2/src/shared/march_description/urdf/march8/hennie_v0.urdf (robot description, URDF)
Before this commit: robot Hennie, 13 links, 12 joints
Joints:
- joint left_ankle: limit lower=-0.436332313 upper=0.1745329252 effort=179 velocity=4.1 -> lower=-0.436332313 upper=0.1645329252 effort=179 velocity=4.1
- joint right_ankle: limit lower=-0.436332313 upper=0.1745329252 effort=179 velocity=4.1 -> lower=-0.436332313 upper=0.1645329252 effort=179 velocity=4.1

Commit message: set the hard limits for the ankles to 8.8 deg

File: ros2/src/shared/march_description/urdf/march8/hennie_v0.urdf (robot description, URDF)
Before this commit: robot Hennie, 13 links, 12 joints
Joints:
- joint left_ankle: limit lower=-0.436332313 upper=0.1645329252 effort=179 velocity=4.1 -> lower=-0.436332313 upper=0.155000 effort=179 velocity=4.1
- joint right_ankle: limit lower=-0.436332313 upper=0.1645329252 effort=179 velocity=4.1 -> lower=-0.436332313 upper=0.155000 effort=179 velocity=4.1

Commit message: make the constraints in the urdf more strict

File: ros2/src/shared/march_description/urdf/march8/hennie_v0.urdf (robot description, URDF)
Before this commit: robot Hennie, 13 links, 12 joints
Joints:
- joint left_knee: limit lower=0 upper=2.181661565 effort=250 velocity=3.94 -> lower=0.05 upper=2.131661565 effort=250 velocity=3.94
- joint right_knee: limit lower=0 upper=2.181661565 effort=250 velocity=3.94 -> lower=0.05 upper=2.131661565 effort=250 velocity=3.94

Commit message: make the knee constraints harder

File: ros2/src/shared/march_description/urdf/march8/hennie_v0.urdf (robot description, URDF)
Before this commit: robot Hennie, 13 links, 12 joints
Joints:
- joint left_knee: limit lower=0.05 upper=2.131661565 effort=250 velocity=3.94 -> lower=0.08 upper=2.131661565 effort=250 velocity=3.94
- joint right_knee: limit lower=0.05 upper=2.131661565 effort=250 velocity=3.94 -> lower=0.08 upper=2.131661565 effort=250 velocity=3.94

Commit message: increase the plantar limits

File: ros2/src/shared/march_description/urdf/march8/hennie_v0.urdf (robot description, URDF)
Before this commit: robot Hennie, 13 links, 12 joints
Joints:
- joint left_ankle: limit lower=-0.436332313 upper=0.155000 effort=179 velocity=4.1 -> lower=-0.336332313 upper=0.155000 effort=179 velocity=4.1
- joint right_ankle: limit lower=-0.436332313 upper=0.155000 effort=179 velocity=4.1 -> lower=-0.336332313 upper=0.155000 effort=179 velocity=4.1
