Commit message: add new m9_sim_models and add dummy base link to hennie model

File: ros2/src/shared/march_description/urdf/march8/hennie_with_koen.urdf (robot description, URDF)
Before this commit: robot HennieKoen, 13 links, 12 joints
Links:
- added link base_link
Joints:
- added joint base_link_to_backpack: type fixed, parent base_link, child backpack, origin xyz=0 0 0 rpy=0 0 0

File: ros2/src/shared/march_description/urdf/march9/march9.urdf (robot description, URDF)
Before this commit: robot Hennie, 13 links, 12 joints
Links:
- removed link L_ground
- removed link L_toe
- removed link R_ground
- removed link R_toe
- added link L_ankle, mass 0.683; collision mesh filename=package://march_description/meshes/march9/L_Ankle.stl scale=1 1 1; visual mesh filename=package://march_description/meshes/march9/L_Ankle.stl scale=1 1 1
- added link R_ankle, mass 0.683; collision mesh filename=package://march_description/meshes/march9/L_Ankle.stl scale=1 -1 1; visual mesh filename=package://march_description/meshes/march9/L_Ankle.stl scale=1 -1 1
- added link base_link
- link L_LL: mass 4.159 -> 1.895; geometry collision mesh filename=package://march_description/meshes/march9/L_LowerLeg.stl scale=1 1 1; visual mesh filename=package://march_description/meshes/march9/L_LowerLeg.stl scale=1 1 1
- link L_UL: mass 8.566 -> 1.520; geometry collision mesh filename=package://march_description/meshes/march9/L_UpperLeg.stl scale=1 1 1; visual mesh filename=package://march_description/meshes/march9/L_UpperLeg.stl scale=1 1 1
- link L_foot: mass 1.22 -> 0.589; geometry collision mesh filename=package://march_description/meshes/march9/L_Sole.stl scale=1 1 1; visual mesh filename=package://march_description/meshes/march9/L_Sole.stl scale=1 1 1
- link L_hip: mass 1.277 -> 3.684; geometry collision mesh filename=package://march_description/meshes/march9/L_Hip.stl scale=1 1 1; visual mesh filename=package://march_description/meshes/march9/L_Hip.stl scale=1 1 1
- link R_LL: mass 4.159 -> 1.895; geometry collision mesh filename=package://march_description/meshes/march9/L_LowerLeg.stl scale=1 -1 1; visual mesh filename=package://march_description/meshes/march9/L_LowerLeg.stl scale=1 -1 1
- link R_UL: mass 8.566 -> 1.520; geometry collision mesh filename=package://march_description/meshes/march9/L_UpperLeg.stl scale=1 -1 1; visual mesh filename=package://march_description/meshes/march9/L_UpperLeg.stl scale=1 -1 1
- link R_foot: mass 1.22 -> 0.589; geometry collision mesh filename=package://march_description/meshes/march9/L_Sole.stl scale=1 -1 1; visual mesh filename=package://march_description/meshes/march9/L_Sole.stl scale=1 -1 1
- link R_hip: mass 1.277 -> 3.684; geometry collision mesh filename=package://march_description/meshes/march9/L_Hip.stl scale=1 -1 1; visual mesh filename=package://march_description/meshes/march9/L_Hip.stl scale=1 -1 1
- link backpack: mass 11.02 -> 3.548; geometry collision mesh filename=package://march_description/meshes/march9/backpack.stl scale=1 1 1; visual mesh filename=package://march_description/meshes/march9/backpack.stl scale=1 1 1
Joints:
- removed joint L_ground
- removed joint R_ground
- removed joint left_ankle
- removed joint left_toe
- removed joint right_ankle
- removed joint right_toe
- added joint base_link_to_backpack: type fixed, parent base_link, child backpack, origin xyz=0 0 0 rpy=0 0 0
- added joint left_ankle_dpf: type revolute, parent L_LL, child L_ankle, origin xyz=0.000 -0.016 -0.474 rpy=0 0 0, axis 0 -1 0, limit lower=-0.488692 upper=0.349066 effort=179 velocity=4.1
- added joint left_ankle_ie: type revolute, parent L_ankle, child L_foot, origin xyz=-0.093 -0.061 -0.025 rpy=0 0 0, axis 1 0 0, limit lower=-0.1396263 upper=0.1396263 effort=179 velocity=4.1
- added joint right_ankle_dpf: type revolute, parent R_LL, child R_ankle, origin xyz=0.000 0.016 -0.474 rpy=0 0 0, axis 0 -1 0, limit lower=-0.488692 upper=0.349066 effort=179 velocity=4.1
- added joint right_foot_ie: type revolute, parent R_ankle, child R_foot, origin xyz=-0.093 0.061 -0.025 rpy=0 0 0, axis 1 0 0, limit lower=-0.1396263 upper=0.1396263 effort=179 velocity=4.1
- joint left_hip_aa: limit lower=-0.2617993878 upper=0.1745329252 effort=280 velocity=2.6 -> lower=-0.349066 upper=0.174533 effort=280 velocity=2.6; origin xyz=-0.021 0.08 0.025 rpy=0 0 0 -> xyz=0.021 0.092 0.028 rpy=0 0 0
- joint left_hip_fe: limit lower=-0.1745329252 upper=1.9634954085 effort=250 velocity=3.94 -> lower=-0.349066 upper=2.00713 effort=250 velocity=3.94; origin xyz=0.182 0.182 0 rpy=0 0 0.0 -> xyz=0.169 0.173 0.000 rpy=0 0 0.0
- joint left_knee: limit lower=0.08 upper=2.131661565 effort=250 velocity=3.94 -> lower=0 upper=2.18166 effort=250 velocity=3.94; origin xyz=0 -0.06 -0.413 rpy=0 0 0 -> xyz=0.000 -0.077 -0.478 rpy=0 0 0
- joint right_hip_aa: limit lower=-0.2617993878 upper=0.1745329252 effort=280 velocity=2.6 -> lower=-0.349066 upper=0.174533 effort=280 velocity=2.6; origin xyz=-0.021 -0.08 0.025 rpy=0 0 0 -> xyz=0.021 -0.092 0.028 rpy=0 0 0
- joint right_hip_fe: limit lower=-0.1745329252 upper=1.9634954085 effort=250 velocity=3.94 -> lower=-0.349066 upper=2.00713 effort=250 velocity=3.94; origin xyz=0.182 -0.182 0 rpy=0 0 0.0 -> xyz=0.169 -0.173 0.000 rpy=0 0 0.0
- joint right_knee: limit lower=0.08 upper=2.131661565 effort=250 velocity=3.94 -> lower=0 upper=2.18166 effort=250 velocity=3.94; origin xyz=0 0.06 -0.413 rpy=0 0 0 -> xyz=0.000 0.077 -0.478 rpy=0 0 0

Commit message: remove base link from hennie koen urdf

File: ros2/src/shared/march_description/urdf/march8/hennie_with_koen.urdf (robot description, URDF)
Before this commit: robot HennieKoen, 14 links, 13 joints
Links:
- removed link base_link
Joints:
- removed joint base_link_to_backpack
