Commit message: Implement torque converter in state estimator including dynamical joint acceleration, and test script

File: ros2/src/shared/march_description/urdf/march9/rotational_test_setup.urdf (robot description, URDF)
Before this commit: robot rotational_test_setup, 2 links, 1 joints
Links:
- removed link endpoint
- removed link world
- added link base_link, mass 0.3743; visual cylinder length=0.1 radius=0.1
- added link weight, mass 0.7073; visual cylinder length=1.0 radius=0.05
Joints:
- joint bar: axis 0 -1 0 -> 0 1 0; child endpoint -> weight; limit lower=-0.1745329252 upper=1.9634954085 effort=250 velocity=3.94 -> lower=-0.78539816339 upper=0.78539816339 effort=250 velocity=3.94; parent world -> base_link
