Commit message: add foot transforms ankle to heel, sole, and toe

File: ros2/src/shared/march_description/urdf/march9/march9.urdf (robot description, URDF)
Before this commit: robot Izzy, 12 links, 11 joints
Links:
- added link L_heel
- added link L_sole
- added link L_toe
- added link R_heel
- added link R_sole
- added link R_toe
Joints:
- added joint L_foot_to_L_heel: type fixed, parent L_foot, child L_heel, origin xyz=-0.015 0.0 -0.08 rpy=0 0 0
- added joint L_foot_to_L_sole: type fixed, parent L_foot, child L_sole, origin xyz=0.151 0.0 -0.080 rpy=0 0 0
- added joint L_foot_to_L_toe: type fixed, parent L_foot, child L_toe, origin xyz=0.317 0.0 -0.080 rpy=0 0 0
- added joint R_foot_to_R_heel: type fixed, parent R_foot, child R_heel, origin xyz=-0.015 0.0 -0.08 rpy=0 0 0
- added joint R_foot_to_R_sole: type fixed, parent R_foot, child R_sole, origin xyz=0.151 0.0 -0.080 rpy=0 0 0
- added joint R_foot_to_R_toe: type fixed, parent R_foot, child R_toe, origin xyz=0.317 0.0 -0.080 rpy=0 0 0

Commit message: Fix Izzy URDF

File: ros2/src/shared/march_description/urdf/march9/march9.urdf (robot description, URDF)
Before this commit: robot Izzy, 18 links, 17 joints
Joints:
- removed joint right_foot_ie
- added joint right_ankle_ie: type revolute, parent R_ankle, child R_foot, origin xyz=-0.093 0.061 -0.025 rpy=0 0 0, axis 1 0 0, limit lower=-0.1396263 upper=0.1396263 effort=179 velocity=4.1

Commit message: fix aie_force with added damping coeff

File: ros2/src/shared/march_description/urdf/march9/march9.urdf (robot description, URDF)
Before this commit: robot Izzy, 18 links, 17 joints
Joints:
- joint left_ankle_ie: limit lower=-0.1396263 upper=0.1396263 effort=179 velocity=4.1 -> lower=-0.157079633 upper=0.157079633 effort=179 velocity=4.1
- joint right_ankle_ie: axis 1 0 0 -> -1 0 0; limit lower=-0.1396263 upper=0.1396263 effort=179 velocity=4.1 -> lower=-0.157079633 upper=0.157079633 effort=179 velocity=4.1

Commit message: Add working m9 sim with izzy, synchronize hardware errors, fix AIE

File: ros2/src/shared/march_description/urdf/march9/march9.urdf (robot description, URDF)
Before this commit: robot Izzy, 18 links, 17 joints
Joints:
- removed joint right_foot_ie
- added joint right_ankle_ie: type revolute, parent R_ankle, child R_foot, origin xyz=-0.093 0.061 -0.025 rpy=0 0 0, axis -1 0 0, limit lower=-0.157079633 upper=0.157079633 effort=179 velocity=4.1
- joint left_ankle_ie: limit lower=-0.1396263 upper=0.1396263 effort=179 velocity=4.1 -> lower=-0.157079633 upper=0.157079633 effort=179 velocity=4.1

Commit message: M9 sim add URDF link and joint for camera

File: ros2/src/shared/march_description/urdf/march9/march9.urdf (robot description, URDF)
Before this commit: robot Izzy, 18 links, 17 joints
Links:
- added link L_camera
- added link R_camera
Joints:
- added joint L_UL_to_L_camera: type fixed, parent L_UL, child L_camera, origin xyz=0.050 0.000 -0.050 rpy=0 0 0
- added joint R_UL_to_R_camera: type fixed, parent R_UL, child R_camera, origin xyz=0.050 0.000 -0.050 rpy=0 0 0

Commit message: Update alignment in simulation model

File: ros2/src/shared/march_description/urdf/march9/march9.urdf (robot description, URDF)
Before this commit: robot Izzy, 20 links, 19 joints
Joints:
- joint left_ankle_dpf: origin xyz=0.000 -0.016 -0.474 rpy=0 0 0 -> xyz=0.000 -0.016 -0.469 rpy=0 0 0
- joint left_hip_aa: origin xyz=0.021 0.092 0.028 rpy=0 0 0 -> xyz=0.021 0.081 0.028 rpy=0 0 0
- joint left_hip_fe: origin xyz=0.169 0.173 0.000 rpy=0 0 0.0 -> xyz=0.169 0.176 0.000 rpy=0 0 0.0
- joint left_knee: origin xyz=0.000 -0.077 -0.478 rpy=0 0 0 -> xyz=0.000 -0.077 -0.463 rpy=0 0 0
- joint right_ankle_dpf: origin xyz=0.000 0.016 -0.474 rpy=0 0 0 -> xyz=0.000 0.016 -0.469 rpy=0 0 0
- joint right_hip_aa: origin xyz=0.021 -0.092 0.028 rpy=0 0 0 -> xyz=0.021 -0.081 0.028 rpy=0 0 0
- joint right_hip_fe: origin xyz=0.169 -0.173 0.000 rpy=0 0 0.0 -> xyz=0.169 -0.176 0.000 rpy=0 0 0.0
- joint right_knee: origin xyz=0.000 0.077 -0.478 rpy=0 0 0 -> xyz=0.000 0.077 -0.463 rpy=0 0 0

Commit message: First release of March IX with our exoskeleton Izzy

File: ros2/src/shared/march_description/urdf/march9/march9.urdf (robot description, URDF)
Before this commit: robot Izzy, 12 links, 11 joints
Links:
- added link L_camera
- added link L_heel
- added link L_sole
- added link L_toe
- added link R_camera
- added link R_heel
- added link R_sole
- added link R_toe
Joints:
- removed joint right_foot_ie
- added joint L_UL_to_L_camera: type fixed, parent L_UL, child L_camera, origin xyz=0.050 0.000 -0.050 rpy=0 0 0
- added joint L_foot_to_L_heel: type fixed, parent L_foot, child L_heel, origin xyz=-0.015 0.0 -0.08 rpy=0 0 0
- added joint L_foot_to_L_sole: type fixed, parent L_foot, child L_sole, origin xyz=0.151 0.0 -0.080 rpy=0 0 0
- added joint L_foot_to_L_toe: type fixed, parent L_foot, child L_toe, origin xyz=0.317 0.0 -0.080 rpy=0 0 0
- added joint R_UL_to_R_camera: type fixed, parent R_UL, child R_camera, origin xyz=0.050 0.000 -0.050 rpy=0 0 0
- added joint R_foot_to_R_heel: type fixed, parent R_foot, child R_heel, origin xyz=-0.015 0.0 -0.08 rpy=0 0 0
- added joint R_foot_to_R_sole: type fixed, parent R_foot, child R_sole, origin xyz=0.151 0.0 -0.080 rpy=0 0 0
- added joint R_foot_to_R_toe: type fixed, parent R_foot, child R_toe, origin xyz=0.317 0.0 -0.080 rpy=0 0 0
- added joint right_ankle_ie: type revolute, parent R_ankle, child R_foot, origin xyz=-0.093 0.061 -0.025 rpy=0 0 0, axis -1 0 0, limit lower=-0.157079633 upper=0.157079633 effort=179 velocity=4.1
- joint left_ankle_ie: limit lower=-0.1396263 upper=0.1396263 effort=179 velocity=4.1 -> lower=-0.157079633 upper=0.157079633 effort=179 velocity=4.1

Commit message: add new camera frames to URDF

File: ros2/src/shared/march_description/urdf/march9/march9.urdf (robot description, URDF)
Before this commit: robot Izzy, 20 links, 19 joints
Joints:
- joint L_UL_to_L_camera: origin xyz=0.050 0.000 -0.050 rpy=0 0 0 -> xyz=0.0801 0.0019 -0.1424 rpy=0 0.6970 0
- joint R_UL_to_R_camera: origin xyz=0.050 0.000 -0.050 rpy=0 0 0 -> xyz=0.0801 -0.0019 -0.1424 rpy=0 0.6970 0

File: ros2/src/shared/march_description/urdf/march9/march9_with_person.urdf (robot description, URDF)
Before this commit: robot Izzy, 20 links, 19 joints
Joints:
- joint L_UL_to_L_camera: origin xyz=0.050 0.000 -0.050 rpy=0 0 0 -> xyz=0.0801 0.0019 -0.1424 rpy=0 0.6970 0
- joint R_UL_to_R_camera: origin xyz=0.050 0.000 -0.050 rpy=0 0 0 -> xyz=0.0801 -0.0019 -0.1424 rpy=0 0.6970 0
