Commit message: refactor urdf and xml folder

File: ros2/src/shared/march_description/models/march9.urdf (robot description, URDF)
Before this commit: robot Izzy, 20 links, 19 joints
Links:
- link L_LL: geometry collision mesh filename=package://march_description/models/assets/L_LowerLeg.stl scale=1 1 1; visual mesh filename=package://march_description/models/assets/L_LowerLeg.stl scale=1 1 1
- link L_UL: geometry collision mesh filename=package://march_description/models/assets/L_UpperLeg.stl scale=1 1 1; visual mesh filename=package://march_description/models/assets/L_UpperLeg.stl scale=1 1 1
- link L_ankle: geometry collision mesh filename=package://march_description/models/assets/L_Ankle.stl scale=1 1 1; visual mesh filename=package://march_description/models/assets/L_Ankle.stl scale=1 1 1
- link L_foot: geometry collision mesh filename=package://march_description/models/assets/L_Sole.stl scale=1 1 1; visual mesh filename=package://march_description/models/assets/L_Sole.stl scale=1 1 1
- link L_hip: geometry collision mesh filename=package://march_description/models/assets/L_Hip.stl scale=1 1 1; visual mesh filename=package://march_description/models/assets/L_Hip.stl scale=1 1 1
- link R_LL: geometry collision mesh filename=package://march_description/models/assets/L_LowerLeg.stl scale=1 -1 1; visual mesh filename=package://march_description/models/assets/L_LowerLeg.stl scale=1 -1 1
- link R_UL: geometry collision mesh filename=package://march_description/models/assets/L_UpperLeg.stl scale=1 -1 1; visual mesh filename=package://march_description/models/assets/L_UpperLeg.stl scale=1 -1 1
- link R_ankle: geometry collision mesh filename=package://march_description/models/assets/L_Ankle.stl scale=1 -1 1; visual mesh filename=package://march_description/models/assets/L_Ankle.stl scale=1 -1 1
- link R_foot: geometry collision mesh filename=package://march_description/models/assets/L_Sole.stl scale=1 -1 1; visual mesh filename=package://march_description/models/assets/L_Sole.stl scale=1 -1 1
- link R_hip: geometry collision mesh filename=package://march_description/models/assets/L_Hip.stl scale=1 -1 1; visual mesh filename=package://march_description/models/assets/L_Hip.stl scale=1 -1 1
- link backpack: geometry collision mesh filename=package://march_description/models/assets/backpack.stl scale=1 1 1; visual mesh filename=package://march_description/models/assets/backpack.stl scale=1 1 1

File: ros2/src/shared/march_description/models/march9_with_person.urdf (robot description, URDF)
Before this commit: robot Izzy, 20 links, 19 joints
Links:
- link L_LL: geometry collision mesh filename=package://march_description/models/assets/L_LowerLeg.stl scale=1 1 1; visual mesh filename=package://march_description/models/assets/L_LowerLeg.stl scale=1 1 1
- link L_UL: geometry collision mesh filename=package://march_description/models/assets/L_UpperLeg.stl scale=1 1 1; visual mesh filename=package://march_description/models/assets/L_UpperLeg.stl scale=1 1 1
- link L_ankle: geometry collision mesh filename=package://march_description/models/assets/L_Ankle.stl scale=1 1 1; visual mesh filename=package://march_description/models/assets/L_Ankle.stl scale=1 1 1
- link L_foot: geometry collision mesh filename=package://march_description/models/assets/L_Sole.stl scale=1 1 1; visual mesh filename=package://march_description/models/assets/L_Sole.stl scale=1 1 1
- link L_hip: geometry collision mesh filename=package://march_description/models/assets/L_Hip.stl scale=1 1 1; visual mesh filename=package://march_description/models/assets/L_Hip.stl scale=1 1 1
- link R_LL: geometry collision mesh filename=package://march_description/models/assets/L_LowerLeg.stl scale=1 -1 1; visual mesh filename=package://march_description/models/assets/L_LowerLeg.stl scale=1 -1 1
- link R_UL: geometry collision mesh filename=package://march_description/models/assets/L_UpperLeg.stl scale=1 -1 1; visual mesh filename=package://march_description/models/assets/L_UpperLeg.stl scale=1 -1 1
- link R_ankle: geometry collision mesh filename=package://march_description/models/assets/L_Ankle.stl scale=1 -1 1; visual mesh filename=package://march_description/models/assets/L_Ankle.stl scale=1 -1 1
- link R_foot: geometry collision mesh filename=package://march_description/models/assets/L_Sole.stl scale=1 -1 1; visual mesh filename=package://march_description/models/assets/L_Sole.stl scale=1 -1 1
- link R_hip: geometry collision mesh filename=package://march_description/models/assets/L_Hip.stl scale=1 -1 1; visual mesh filename=package://march_description/models/assets/L_Hip.stl scale=1 -1 1
- link backpack: geometry collision mesh filename=package://march_description/models/assets/backpack.stl scale=1 1 1; visual mesh filename=package://march_description/models/assets/backpack.stl scale=1 1 1
